Commit message: refs #84 add a gazebo plugins (controller manager) for ROS to publish joint_states
git-svn-id: svn+ssh://marvin.3it.usherbrooke.ca/svn/introlab/johnny0/svn/branches/M6/ros-pkgs/johnny_0_model/johnny_0_description@559 23a761d4-b60a-4777-9503-f06a07968eac

File: gazebo/gazebo.urdf.xacro (robot description, xacro)
@@ -10,9 +10,9 @@
     </controller:gazebo_ros_controller_manager>
 		<!-- Inutile pour l'instant -->
-    <controller:gazebo_ros_battery name="gazebo_ros_battery_controller" plugin="libgazebo_ros_battery.so">
+    <controller:gazebo_ros_power_monitor name="gazebo_ros_power_monitor_controller" plugin="libgazebo_ros_power_monitor.so">
       <alwaysOn>true</alwaysOn>
       <updateRate>1.0</updateRate>
       <timeout>5</timeout>
-      <interface:audio name="battery_dummy_interface" />
+      <interface:audio name="power_monitor_dummy_interface" />
       <powerStateTopic>power_state</powerStateTopic>
       <powerStateRate>10.0</powerStateRate>
@@ -22,5 +22,5 @@
       <dischargeVoltage>15.52</dischargeVoltage>
       <chargeVoltage>16.41</chargeVoltage>
-    </controller:gazebo_ros_battery>
+    </controller:gazebo_ros_power_monitor>
   </gazebo>
 </robot>

File: robots/johnny_0.urdf.xacro (robot description, xacro)
@@ -16,5 +16,5 @@
 	<include filename="$(find johnny_0_description)/urdf/camera/camera.urdf.xacro" />
 	<!-- generic simulator_gazebo plugins for starting mechanism control, ros time, ros battery -->
-	<!--include filename="$(find johnny_0_description)/gazebo/gazebo.urdf.xacro" /-->
+	<include filename="$(find johnny_0_description)/gazebo/gazebo.urdf.xacro" />
 	<!-- materials for visualization -->
 	<include filename="$(find johnny_0_description)/urdf/materials.urdf.xacro" />
@@ -37,4 +37,4 @@
 	<xacro:arm side="L" reflect="1" parent="torso_link"/>
 	<xacro:head name="head" parent="torso_link"/>
-	<xacro:camera name="camera" parent="head_head_link"/>
+	<!--xacro:camera name="camera" parent="head_head_link"/-->
 </robot>

File: urdf/arm/ADE_pitch_elbow/ADE_pitch_elbow.urdf.xacro (robot description, xacro)
@@ -4,4 +4,5 @@
        xmlns:interface="http://playerstage.sourceforge.net/gazebo/xmlschema/#interface"
        xmlns:xacro="http://ros.org/wiki/xacro">
+	<include filename="$(find johnny_0_description)/urdf/arm/arm.transmission.xacro" />
 	<xacro:macro name="ADE_pitch_elbow" params="side reflect parent">
 		<link name="ADE_pitch_elbow${side}_box">
@@ -86,4 +87,6 @@
 			<origin xyz="0.0235 0 0" rpy="0 0 0" />
 		</joint>
+		<!-- extensions -->
+		<xacro:johnny_0_ADE_pitch_elbow_transmission side="${side}" />
 		<gazebo reference="ADE_pitch_elbow${side}_box">
 			<material>Gazebo/Green</material>

File: urdf/arm/ADE_pitch_shoulder/ADE_pitch_shoulder.urdf.xacro (robot description, xacro)
@@ -4,4 +4,5 @@
        xmlns:interface="http://playerstage.sourceforge.net/gazebo/xmlschema/#interface"
        xmlns:xacro="http://ros.org/wiki/xacro">
+	<include filename="$(find johnny_0_description)/urdf/arm/arm.transmission.xacro" />
 	<xacro:macro name="ADE_pitch_shoulder" params="side reflect parent">
 		<joint name="ADE_pitch_shoulder${side}_fixed_1_joint" type="fixed">
@@ -86,4 +87,6 @@
 			</collision>
 		</link>
+		<!-- extensions -->
+		<xacro:johnny_0_ADE_pitch_shoulder_transmission side="${side}" />
 		<gazebo reference="ADE_pitch_shoulder${side}_link">
 			<material>Gazebo/Red</material>

File: urdf/arm/ADE_roll/ADE_roll.urdf.xacro (robot description, xacro)
@@ -4,4 +4,5 @@
        xmlns:interface="http://playerstage.sourceforge.net/gazebo/xmlschema/#interface"
        xmlns:xacro="http://ros.org/wiki/xacro">
+	<include filename="$(find johnny_0_description)/urdf/arm/arm.transmission.xacro" />
 	<xacro:macro name="ADE_roll" params="side reflect parent">
 		<joint name="ADE_roll${side}_fixed_origine_joint" type="fixed">
@@ -87,4 +88,6 @@
 			</collision>
 		</link>
+		<!-- extensions -->
+		<xacro:johnny_0_ADE_roll_shoulder_transmission side="${side}" />
 		<gazebo reference="ADE_roll${side}_box">
 			<material>Gazebo/Blue</material>

File: urdf/base/base.urdf.xacro (robot description, xacro)
@@ -4,5 +4,7 @@
        xmlns:interface="http://playerstage.sourceforge.net/gazebo/xmlschema/#interface"
        xmlns:xacro="http://ros.org/wiki/xacro">
-  <property name="base_collision_size_z" value="0.04" />
+	<!-- Include files for extansions -->
+	<include filename="$(find johnny_0_description)/urdf/base/base.gazebo.xacro" />
+	<property name="base_collision_size_z" value="0.04" />
 	<xacro:macro name="base" params="name">
 		<!-- Suppression of the link between the world and the base -->
@@ -32,4 +34,9 @@
 		  </collision>
 		</link>
+		<joint name="${name}_footprint_joint" type="fixed">
+		  <origin xyz="0 0 0.251" rpy="0 0 0" />
+		  <child link="${name}_link" />
+		  <parent link="${name}_footprint"/>
+		</joint>
 		<!-- base_footprint is a fictitious link(frame) that is on the ground right below base_link origin,
 			navigation stack dedpends on this frame -->
@@ -57,9 +64,6 @@
 		  </collision>
 		</link>
-		<joint name="${name}_footprint_joint" type="fixed">
-		  <origin xyz="0 0 0.251" rpy="0 0 0" />
-		  <child link="${name}_link" />
-		  <parent link="${name}_footprint"/>
-		</joint>
+		<!-- gazebo extensions -->
+		<xacro:johnny_0_base_gazebo name="${name}" />
 		<gazebo reference="${name}_link">
 			<material>Gazebo/Blue</material>

File: urdf/head/head.urdf.xacro (robot description, xacro)
@@ -4,4 +4,5 @@
        xmlns:interface="http://playerstage.sourceforge.net/gazebo/xmlschema/#interface"
        xmlns:xacro="http://ros.org/wiki/xacro">
+	<include filename="$(find johnny_0_description)/urdf/head/head.transmission.xacro" />
 	<xacro:macro name="head" params="name parent">
 		<joint name="${name}_fixed_joint" type="fixed">
@@ -30,5 +31,5 @@
 			</collision>
 		</link>
-		<joint name="${name}_revolute_joint_tmp" type="revolute">
+		<joint name="${name}_tilt_joint" type="revolute">
 			<parent link="${name}_link"/>
 			<child link="${name}_head_link_tmp"/>
@@ -58,5 +59,5 @@
 			</collision>
 		</link>
-		<joint name="${name}_revolute_joint" type="revolute">
+		<joint name="${name}_pan_joint" type="revolute">
 			<parent link="${name}_head_link_tmp"/>
 			<child link="${name}_head_link"/>
@@ -86,4 +87,7 @@
 			</collision>
 		</link>
+		<!-- extansions -->
+		<xacro:johnny_0_head_tilt_transmission />
+		<xacro:johnny_0_head_pan_transmission />
 		<gazebo reference="${name}_link">
 			<material>Gazebo/Green</material>

File: urdf/wheel/wheel.urdf.xacro (robot description, xacro)
@@ -4,4 +4,7 @@
        xmlns:interface="http://playerstage.sourceforge.net/gazebo/xmlschema/#interface"
        xmlns:xacro="http://ros.org/wiki/xacro">
+	<!-- Include files for extansions -->
+	<include filename="$(find johnny_0_description)/urdf/wheel/wheel.gazebo.xacro" />
+	<include filename="$(find johnny_0_description)/urdf/wheel/wheel.transmission.xacro" />
 	<xacro:macro name="wheel" params="side reflectSide face reflectFace parent">
 		<joint name="wheel${side}${face}_fixed_joint" type="fixed">
@@ -109,4 +112,8 @@
 			</collision>
 		</link>
+		<!-- extensions -->
+		<xacro:johnny_0_wheel_gazebo side="${side}" face="${face}" />
+		<xacro:johnny_0_wheel_transmission side="${side}" face="${face}" />
+		<xacro:johnny_0_ADE_transmission side="${side}" face="${face}" />
 		<gazebo reference="wheel${side}${face}_link">
 			<material>Gazebo/Red</material>
