Commit message: refs #85 get the robot urdf model to have the upper torso oriented in the X direction of the base instead of Y
git-svn-id: svn+ssh://marvin.3it.usherbrooke.ca/svn/introlab/johnny0/svn/branches/M6/ros-pkgs/johnny_0_model/johnny_0_description@568 23a761d4-b60a-4777-9503-f06a07968eac

File: urdf/arm/ADE_roll/ADE_roll.urdf.xacro (robot description, xacro)
@@ -9,5 +9,5 @@
 			<parent link="${parent}"/>
 			<child link="ADE_roll${side}_box"/>
-			<origin xyz="${reflect*0.1} 0 0.1" rpy="0 0 ${(reflect-1)*M_PI/2}" />
+			<origin xyz="0 ${reflect*0.09} 0.1" rpy="0 0 ${(reflect-1)*M_PI/2+M_PI/2}" />
 		</joint>
 		<link name="ADE_roll${side}_box">
@@ -15,12 +15,12 @@
 				<mass value="1.105" />
 				<origin xyz="0 0 0" rpy="0 0 0"/>
-        <inertia  ixx="0.002790566518" ixy="0.00"  ixz="0.00"
-                  iyy="0.002862829183" iyz="0.00"
-                  izz="0.001375984901" />
+				<inertia  ixx="0.002790566518" ixy="0.00"  ixz="0.00"
+						  iyy="0.002862829183" iyz="0.00"
+						  izz="0.001375984901" />
 			</inertial>
 			<visual>
 				<origin xyz="0 0 0" rpy="0 0 0" />
 				<geometry name="ADE_roll${side}_box_visual_geom">
-					<box size="0.088678 0.084137 0.1524" />
+					<box size="0.084137 0.088678 0.1524" />
 				</geometry>
 			</visual>
@@ -28,5 +28,5 @@
 				<origin xyz="0 0 0" rpy="0 0 0 " />
 				<geometry name="ADE_roll${side}_box_collision_geom">
-					<box size="0.088678 0.084137 0.1524" />
+					<box size="0.084137 0.088678 0.1524" />
 				</geometry>
 			</collision>

File: urdf/head/head.urdf.xacro (robot description, xacro)
@@ -9,5 +9,5 @@
 			<parent link="${parent}"/>
 			<child link="${name}_link"/>
-			<origin xyz="0 0.02 0.2228115" rpy="0 0 0" />
+			<origin xyz="0.02 0 0.2228115" rpy="0 0 0" />
 		</joint>
 		<link name="${name}_link">
@@ -34,6 +34,6 @@
 			<parent link="${name}_link"/>
 			<child link="${name}_head_link_tmp"/>
-			<origin xyz="0 -0.02 0.0966715" rpy="0 0 0" />
-			<axis xyz="1 0 0" rpy="0 0 0"/>
+			<origin xyz="-0.02 0 0.0966715" rpy="0 0 0" />
+			<axis xyz="0 1 0" rpy="0 0 0"/>
 			<limit effort="100" velocity="0.1" lower="-0.7" upper="0.7" />
 			<calibration reference_position="0.0"/>
@@ -77,5 +77,5 @@
 				<origin xyz="0 0 0" rpy="0 0 0" />
 				<geometry name="${name}_head_visual_geom">
-					<box size="0.17418 0.16268 0.12693" />
+					<box size="0.16268 0.17418 0.12693" />
 				</geometry>
 			</visual>
@@ -83,5 +83,5 @@
 				<origin xyz="0 0 0" rpy="0 0 0" />
 				<geometry name="${name}_head_collision_geom">
-					<box size="0.17418 0.16268 0.12693" />
+					<box size="0.16268 0.17418 0.12693" />
 				</geometry>
 			</collision>

File: urdf/torso/torso.urdf.xacro (robot description, xacro)
@@ -20,5 +20,5 @@
 				<origin xyz="0 0 0" rpy="0 0 0" />
 				<geometry name="${name}_visual_geom">
-					<box size="0.270 0.21583 0.37921" />
+					<box size="0.21583 0.270 0.37921" />
 				</geometry>
 			</visual>
@@ -26,5 +26,5 @@
 				<origin xyz="0 0 0" rpy="0 0 0" />
 				<geometry name="${name}_collision_geom">
-					<box size="0.270 0.21583 0.37921" />
+					<box size="0.21583 0.270 0.37921" />
 				</geometry>
 			</collision>
