Commit message: Closes #117, #132, #135. Merging back M7.
git-svn-id: svn+ssh://marvin.3it.usherbrooke.ca/svn/introlab/johnny0/svn/trunk/ros-pkgs/johnny_0_model/johnny_0_description@914 23a761d4-b60a-4777-9503-f06a07968eac

File: robots/azimut_3.urdf.xacro (robot description, xacro)
@@ -11,9 +11,4 @@
 	<include filename="$(find johnny_0_description)/urdf/base/base.urdf.xacro" />
 	<include filename="$(find johnny_0_description)/urdf/wheel/wheel.urdf.xacro" />
-	<include filename="$(find johnny_0_description)/urdf/baseTorsoLink/baseTorsoLink.urdf.xacro" />
-	<include filename="$(find johnny_0_description)/urdf/torso/torso.urdf.xacro" />
-	<include filename="$(find johnny_0_description)/urdf/arm/arm.urdf.xacro" />
-	<include filename="$(find johnny_0_description)/urdf/head/head.urdf.xacro" />
-	<include filename="$(find johnny_0_description)/urdf/camera/bumblebee.urdf.xacro" />
 	<!-- generic simulator_gazebo plugins for starting mechanism control, ros time, ros battery -->
 	<include filename="$(find johnny_0_description)/gazebo/gazebo.urdf.xacro" />
@@ -33,11 +28,4 @@
 	<xacro:wheel side="L" reflectSide="1" face="B" reflectFace="-1" parent="base_link"/>
 	<xacro:wheel side="L" reflectSide="1" face="F" reflectFace="1" parent="base_link"/>
-	<xacro:baseTorsoLink name="baseTorsoLink" parent="base_link"/>
-	<xacro:torso name="torso" parent="baseTorsoLink_link"/>
-	<xacro:arm side="R" reflect="-1" parent="torso_link"/>
-	<xacro:arm side="L" reflect="1" parent="torso_link"/>
-	<xacro:head name="head" parent="torso_link">
-		<origin xyz="0.04 0 ${torso_size_z/2}" />
-	</xacro:head>
 	<!--xacro:bumblebee name="bumblebee" parent="head_head_link">
 		<origin xyz="0.06 0 ${head_size_z/2 + bumblebee_size_z/2}" />

File: urdf/arm/ADE_pitch_elbow/ADE_pitch_elbow.urdf.xacro (robot description, xacro)
@@ -80,5 +80,5 @@
 			<axis xyz="0 1 0" rpy="0 0 0"/>
 			<limit effort="100" velocity="0.1" lower="0" upper="1.5708" />
-			<calibration reference_position="0.0"/>
+			<!-- calibration reference_position="0.0"/ -->
 		</joint>
 		<joint name="ADE_pitch_elbow${side}_fixed_2_joint" type="fixed">

File: urdf/arm/ADE_pitch_shoulder/ADE_pitch_shoulder.urdf.xacro (robot description, xacro)
@@ -38,5 +38,5 @@
 			<axis xyz="0 1 0" rpy="0 0 0"/>
 			<limit effort="100" velocity="0.1" lower="-0.7854" upper="0.7854" />
-			<calibration reference_position="0.0"/>
+			<!-- calibration reference_position="0.0"/ -->
 		</joint>
 		<link name="ADE_pitch_shoulder${side}_fixation">

File: urdf/arm/ADE_roll/ADE_roll.urdf.xacro (robot description, xacro)
@@ -65,5 +65,5 @@
 			<axis xyz="0 0 1" rpy="0 0 0"/>
 			<limit effort="30" velocity="0.1" lower="-2.8" upper="2.8" />
-			<calibration reference_position="0.0"/>
+			<!-- calibration reference_position="0.0"/ -->
 		</joint>
 		<link name="ADE_roll${side}_link">

File: urdf/arm/arm.transmission.xacro (robot description, xacro)
@@ -7,5 +7,5 @@
   <!-- ADE roll shoulder -->
   <xacro:macro name="johnny_0_ADE_roll_shoulder_transmission" params="side" >
-    <transmission type="SimpleTransmission" name="${side}_ADE_roll_shoulder_trans">
+    <transmission type="pr2_mechanism_model/SimpleTransmission" name="${side}_ADE_roll_shoulder_trans">
       <actuator name="${side}_ADE_roll_shoulder_motor" />
       <joint name="ADE_roll${side}_revolute_joint" />
@@ -15,5 +15,5 @@
   <!-- ADE pitch shoulder -->
   <xacro:macro name="johnny_0_ADE_pitch_shoulder_transmission" params="side" >
-    <transmission type="SimpleTransmission" name="${side}_ADE_pitch_shoulder_trans">
+    <transmission type="pr2_mechanism_model/SimpleTransmission" name="${side}_ADE_pitch_shoulder_trans">
       <actuator name="${side}_ADE_pitch_shoulder_motor" />
       <joint name="ADE_pitch_shoulder${side}_revolute_joint" />
@@ -23,5 +23,5 @@
   <!--  ADE pitch elbow -->
   <xacro:macro name="johnny_0_ADE_pitch_elbow_transmission" params="side" >
-    <transmission type="SimpleTransmission" name="${side}_ADE_pitch_elbow_trans">
+    <transmission type="pr2_mechanism_model/SimpleTransmission" name="${side}_ADE_pitch_elbow_trans">
       <actuator name="${side}_ADE_pitch_elbow_motor" />
       <joint name="ADE_pitch_elbow${side}_revolute_joint" />

File: urdf/base/base.urdf.xacro (robot description, xacro)
@@ -8,7 +8,7 @@
 	<property name="base_collision_size_z" value="0.04" />
 	<!-- Warning: eye-balled values for the laser position. -->
-	<property name="base_laser_x" value="0.15" />
-	<property name="base_laser_y" value="0.0" />
-	<property name="base_laser_z" value="0.4" />
+	<property name="base_laser_x" value="0.150" />
+	<property name="base_laser_y" value="0.055" />
+	<property name="base_laser_z" value="0.200" />
 	<property name="base_laser_size_x" value="0.06" />
 	<property name="base_laser_size_y" value="0.06" />
@@ -16,10 +16,9 @@
 	<property name="base_laser_collision_offset_z" value="0.023" />
 	<xacro:macro name="base" params="name">
-		<!-- Suppression of the link between the world and the base -->
-		<!--joint name="${name}_fixed_joint" type="fixed">
-				<parent link="${parent}"/>
+		<joint name="${name}_fixed_joint" type="fixed">
+				<parent link="${name}_footprint"/>
 				<child link="${name}_link"/>
 				<origin xyz="0 0 0.22" rpy="0 0 0" />
-		</joint-->
+		</joint>
 		<link name="${name}_link">
 		  <inertial>
@@ -42,9 +41,9 @@
 		  </collision>
 		</link>
-		<joint name="${name}_footprint_joint" type="fixed">
+		<!-- joint name="${name}_footprint_joint" type="fixed">
 		  <origin xyz="0 0 0.251" rpy="0 0 0" />
 		  <child link="${name}_link" />
 		  <parent link="${name}_footprint"/>
-		</joint>
+		</joint -->
 		<!-- base_footprint is a fictitious link(frame) that is on the ground right below base_link origin,
 			navigation stack dedpends on this frame -->

File: urdf/camera/omnivision.urdf.xacro (robot description, xacro)
@@ -4,9 +4,10 @@
        xmlns:interface="http://playerstage.sourceforge.net/gazebo/xmlschema/#interface"
        xmlns:xacro="http://ros.org/wiki/xacro">
-<xacro:macro name="camera" params="name parent">
+<xacro:macro name="omnivision" params="name parent *origin">
 		<joint name="${name}_fixed_joint" type="fixed">
 				<parent link="${parent}"/>
 				<child link="${name}_link"/>
-				<origin xyz="0 -0.06009 0.078965" rpy="0 0 0" />
+				<insert_block name="origin" />
+				<!--origin xyz="0.13 0 0.38" rpy="0 0 0" /-->
 		</joint>
 		<link name="${name}_link">
@@ -20,5 +21,5 @@
 			<origin xyz="0 0 0" rpy="0 0 0" />
 			<geometry name="${name}_visual_geom">
-				<box size="0.152 0.0425 0.031" />
+				<box size="0.10 0.055 0.06" />
 			</geometry>
 		  </visual>
@@ -26,5 +27,5 @@
 			<origin xyz="0 0 0" rpy="0 0 0" />
 			<geometry name="${name}_collision_geom">
-				<box size="0.152 0.0425 0.031" />
+				<box size="0.10 0.055 0.06" />
 			</geometry>
 		  </collision>

File: urdf/head/head.transmission.xacro (robot description, xacro)
@@ -7,5 +7,5 @@
   <!-- Head pan (or yaw) -->
   <xacro:macro name="johnny_0_head_pan_transmission" >
-    <transmission type="SimpleTransmission" name="head_pan_trans">
+    <transmission type="pr2_mechanism_model/SimpleTransmission" name="head_pan_trans">
       <actuator name="head_pan_motor" />
       <joint name="head_pan_joint" />
@@ -15,5 +15,5 @@
   <!-- Head tilt (or roll) -->
   <xacro:macro name="johnny_0_head_tilt_transmission" >
-    <transmission type="SimpleTransmission" name="head_tilt_trans">
+    <transmission type="pr2_mechanism_model/SimpleTransmission" name="head_tilt_trans">
       <actuator name="head_tilt_motor" />
       <joint name="head_tilt_joint" />

File: urdf/head/head.urdf.xacro (robot description, xacro)
@@ -5,65 +5,96 @@
        xmlns:xacro="http://ros.org/wiki/xacro">
 	<include filename="$(find johnny_0_description)/urdf/head/head.transmission.xacro" />
-	<xacro:macro name="head" params="name parent">
+	<property name="pan_size_z" value="0.05" />
+	<property name="head_size_z" value="0.17" />
+	<xacro:macro name="head" params="name parent *origin">
 		<joint name="${name}_fixed_joint" type="fixed">
 			<parent link="${parent}"/>
-			<child link="${name}_link"/>
-			<origin xyz="0.02 0 0.2228115" rpy="0 0 0" />
+			<child link="${name}_pan_link"/>
+			<insert_block name="origin" />
+			<!--origin xyz="0.02 0 0.2228115" rpy="0 0 0" /-->
 		</joint>
-		<link name="${name}_link">
+		<link name="${name}_pan_link">
 			<inertial>
 				<mass value="0.5" />
-				<origin xyz="0 0 0" />
+				<origin xyz="0 0 ${pan_size_z/2}" />
 				<inertia ixx="0" ixy="0" ixz="0"
 						 iyy="0" iyz="0" izz="0" />
 			</inertial>
-			<visual name="${name}_visual">
-				<origin xyz="0 0 0" rpy="0 0 0" />
-				<geometry name="${name}_visual_geom">
-					<box size="0.04 0.04 0.066413" />
+			<visual name="${name}_pan_visual">
+				<origin xyz="0 0 ${pan_size_z/2}" rpy="0 0 0" />
+				<geometry name="${name}_pan_visual_geom">
+					<box size="0.04 0.04 ${pan_size_z}" />
 				</geometry>
 			</visual>
-			<collision name="${name}_collision">
-				<origin xyz="0 0 0" rpy="0 0 0" />
-				<geometry name="${name}_collision_geom">
-					<box size="0.04 0.04 0.066413" />
+			<collision name="${name}_pan_collision">
+				<origin xyz="0 0 ${pan_size_z/2}" rpy="0 0 0" />
+				<geometry name="${name}_pan_collision_geom">
+					<box size="0.04 0.04 ${pan_size_z}" />
+				</geometry>
+			</collision>
+		</link>
+		<joint name="${name}_pan_joint" type="revolute">
+			<parent link="${name}_pan_link"/>
+			<child link="${name}_tilt_link"/>
+			<origin xyz="0 0 ${pan_size_z}" rpy="0 0 0" />
+			<axis xyz="0 0 1" rpy="0 0 0"/>
+			<limit effort="100" velocity="0.1" lower="-0.7854" upper="0.7854" />
+			<!-- calibration reference_position="0.0"/ -->
+		</joint>
+		<link name="${name}_tilt_link">
+			<inertial>
+				<mass value="0.001" />
+				<origin xyz="0 0 0.023" />
+				<inertia ixx="0" ixy="0" ixz="0"
+						 iyy="0" iyz="0" izz="0" />
+			</inertial>
+			<visual name="${name}_tilt_visual">
+				<origin xyz="0 0 0.023" rpy="0 0 0" />
+				<geometry name="${name}_tilt_visual_geom">
+					<box size="0.04 0.04 0.046" />
+				</geometry>
+			</visual>
+			<collision name="${name}_tilt_collision">
+				<origin xyz="0 0 0.023" rpy="0 0 0" />
+				<geometry name="${name}_tilt_collision_geom">
+					<box size="0.04 0.04 0.046" />
 				</geometry>
 			</collision>
 		</link>
 		<joint name="${name}_tilt_joint" type="revolute">
-			<parent link="${name}_link"/>
-			<child link="${name}_head_link_tmp"/>
-			<origin xyz="-0.02 0 0.0966715" rpy="0 0 0" />
+			<parent link="${name}_tilt_link"/>
+			<child link="${name}_neck_link"/>
+			<!-- distance between tilt axis and beginning of the head plus the half of the head height-->
+			<origin xyz="0 0 0.046" rpy="0 0 0" />
 			<axis xyz="0 1 0" rpy="0 0 0"/>
 			<limit effort="100" velocity="0.1" lower="-0.7" upper="0.7" />
-			<calibration reference_position="0.0"/>
+			<!-- calibration reference_position="0.0"/ -->
 		</joint>
-		<link name="${name}_head_link_tmp">
+		<link name="${name}_neck_link">
 			<inertial>
 				<mass value="0.001" />
-				<origin xyz="0 0 0" />
+				<origin xyz="0 0 0.04" />
 				<inertia ixx="0" ixy="0" ixz="0"
 						 iyy="0" iyz="0" izz="0" />
 			</inertial>
-			<visual name="${name}_head_tmp_visual">
-				<origin xyz="0 0 0" rpy="0 0 0" />
-				<geometry name="${name}_head_tmp_visual_geom">
-					<sphere radius="0.001" />
+			<visual name="${name}_neck_visual">
+				<origin xyz="0 0 0.04" rpy="0 0 0" />
+				<geometry name="${name}_neck_visual_geom">
+					<box size="0.04 0.04 0.08" />
 				</geometry>
 			</visual>
-			<collision name="${name}_head_tmp_collision">
-				<origin xyz="0 0 0" rpy="0 0 0" />
-				<geometry name="${name}_head_tmp_collision_geom">
-					<sphere radius="0.001" />
+			<collision name="${name}_neck_collision">
+				<origin xyz="0 0 0.04" rpy="0 0 0" />
+				<geometry name="${name}_neck_collision_geom">
+					<box size="0.04 0.04 0.08" />
 				</geometry>
 			</collision>
 		</link>
-		<joint name="${name}_pan_joint" type="revolute">
-			<parent link="${name}_head_link_tmp"/>
+		<joint name="${name}_neck_joint" type="fixed">
+			<parent link="${name}_neck_link"/>
 			<child link="${name}_head_link"/>
-			<origin xyz="0 0 0" rpy="0 0 0" />
-			<axis xyz="0 0 1" rpy="0 0 0"/>
-			<limit effort="100" velocity="0.1" lower="-0.7854" upper="0.7854" />
-			<calibration reference_position="0.0"/>
+			<!-- distance between tilt axis and beginning of the head plus the half of the head height-->
+			<origin xyz="0 0 ${0.06 + head_size_z/2}" rpy="0 0 0" />
+			<!-- calibration reference_position="0.0"/ -->
 		</joint>
 		<link name="${name}_head_link">
@@ -77,5 +108,5 @@
 				<origin xyz="0 0 0" rpy="0 0 0" />
 				<geometry name="${name}_head_visual_geom">
-					<box size="0.16268 0.17418 0.12693" />
+					<box size="0.17 0.19 ${head_size_z}" />
 				</geometry>
 			</visual>
@@ -83,5 +114,5 @@
 				<origin xyz="0 0 0" rpy="0 0 0" />
 				<geometry name="${name}_head_collision_geom">
-					<box size="0.16268 0.17418 0.12693" />
+					<box size="0.17 0.19 ${head_size_z}" />
 				</geometry>
 			</collision>

File: urdf/torso/torso.urdf.xacro (robot description, xacro)
@@ -4,4 +4,5 @@
        xmlns:interface="http://playerstage.sourceforge.net/gazebo/xmlschema/#interface"
        xmlns:xacro="http://ros.org/wiki/xacro">
+	<property name="torso_size_z" value="0.37921" />
 	<xacro:macro name="torso" params="name parent">
 		<joint name="${name}_fixed_joint" type="fixed">
@@ -20,5 +21,5 @@
 				<origin xyz="0 0 0" rpy="0 0 0" />
 				<geometry name="${name}_visual_geom">
-					<box size="0.21583 0.270 0.37921" />
+					<box size="0.21583 0.270 ${torso_size_z}" />
 				</geometry>
 			</visual>
@@ -26,5 +27,5 @@
 				<origin xyz="0 0 0" rpy="0 0 0" />
 				<geometry name="${name}_collision_geom">
-					<box size="0.21583 0.270 0.37921" />
+					<box size="0.21583 0.270 ${torso_size_z}" />
 				</geometry>
 			</collision>

File: urdf/wheel/wheel.transmission.xacro (robot description, xacro)
@@ -6,5 +6,5 @@
   <!--  wheel transmission   -->
   <xacro:macro name="johnny_0_wheel_transmission" params="side face">
-    <transmission type="SimpleTransmission" name="${side}_${face}_wheel_trans">
+    <transmission type="pr2_mechanism_model/SimpleTransmission" name="${side}_${face}_wheel_trans">
       <actuator name="${side}_${face}_wheel_motor" />
       <joint name="wheel${side}${face}_wheel_continuous_joint" />
@@ -14,5 +14,5 @@
   <!-- ADE transmission only -->
   <xacro:macro name="johnny_0_ADE_transmission" params="side face">
-    <transmission type="SimpleTransmission" name="${side}_${face}_rotation_trans">
+    <transmission type="pr2_mechanism_model/SimpleTransmission" name="${side}_${face}_rotation_trans">
       <actuator name="ADE_${side}_${face}_revolute_motor" />
       <joint name="wheel${side}${face}_revolute_joint" />

File: urdf/wheel/wheel.urdf.xacro (robot description, xacro)
@@ -64,5 +64,5 @@
 			<axis xyz="0 0 1" rpy="0 0 0"/>
 			<limit effort="100" velocity="0.1" lower="-0.7854" upper="0.7854" />
-			<calibration reference_position="0.0"/>
+			<!-- calibration reference_position="0.0"/ -->
 		</joint>
 		<link name="wheel${side}${face}_ADE2_link">
