Commit message: Refs #156. Better AZ2 obstacle avoidance through corrected URDF.
git-svn-id: svn+ssh://marvin.3it.usherbrooke.ca/svn/introlab/johnny0/svn/branches/M8/ros-pkgs/johnny_0_model/johnny_0_description@1132 23a761d4-b60a-4777-9503-f06a07968eac

File: robots/azimut_2.urdf.xacro (robot description, xacro)
@@ -11,10 +11,4 @@
 	<include filename="$(find johnny_0_description)/urdf/base/base.urdf.xacro" />
 	<include filename="$(find johnny_0_description)/urdf/wheel/wheel.urdf.xacro" />
-	<include filename="$(find johnny_0_description)/urdf/baseTorsoLink/baseTorsoLink.urdf.xacro" />
-	<include filename="$(find johnny_0_description)/urdf/torso/torso.urdf.xacro" />
-	<include filename="$(find johnny_0_description)/urdf/arm/arm.urdf.xacro" />
-	<include filename="$(find johnny_0_description)/urdf/head/head.urdf.xacro" />
-	<include filename="$(find johnny_0_description)/urdf/camera/bumblebee.urdf.xacro" />
-	<include filename="$(find johnny_0_description)/urdf/camera/kinect.urdf.xacro" />
 	<!-- generic simulator_gazebo plugins for starting mechanism control, ros time, ros battery -->
 	<include filename="$(find johnny_0_description)/gazebo/gazebo.urdf.xacro" />
@@ -30,7 +24,7 @@
        is the world frame). For more, see http://www.ros.org/wiki/xacro -->
 	<!-- Warning: eye-balled values for the laser position. -->
-	<property name="base_laser_x" value="0.150" />
-	<property name="base_laser_y" value="0.055" />
-	<property name="base_laser_z" value="0.200" />
+	<property name="base_laser_x" value="0.045" />
+	<property name="base_laser_y" value="0.000" />
+	<property name="base_laser_z" value="0.150" />
 	<property name="base_laser_size_x" value="0.06" />
 	<property name="base_laser_size_y" value="0.06" />
@@ -42,16 +36,6 @@
 	<xacro:wheel side="L" reflectSide="1" face="B" reflectFace="-1" parent="base_link"/>
 	<xacro:wheel side="L" reflectSide="1" face="F" reflectFace="1" parent="base_link"/>
-	<xacro:baseTorsoLink name="baseTorsoLink" parent="base_link"/>
-	<xacro:torso name="torso" parent="baseTorsoLink_link"/>
-	<xacro:arm side="R" reflect="-1" parent="torso_link"/>
-	<xacro:arm side="L" reflect="1" parent="torso_link"/>
-	<xacro:head name="head" parent="torso_link">
-		<origin xyz="0.04 0 ${torso_size_z/2}" />
-	</xacro:head>
-	<xacro:bumblebee name="head_camera" parent="head_head_link">
+	<!--xacro:bumblebee name="bumblebee" parent="head_head_link">
 		<origin xyz="0.06 0 ${head_size_z/2 + bumblebee_size_z/2}" />
-	</xacro:bumblebee>
-	<xacro:kinect name="openni_camera" parent="torso_link">
-		<origin xyz="0.17 0 ${torso_size_z/2 + kinect_size_z/2}" rpy="0 -0.35 0"/>
-	</xacro:kinect>
+	</xacro:bumblebee-->
 </robot>

File: robots/azimut_3.urdf.xacro (robot description, xacro)
@@ -23,4 +23,12 @@
        the origin block defines where the component is w.r.t its parent (in this case the parent
        is the world frame). For more, see http://www.ros.org/wiki/xacro -->
+	<!-- Warning: eye-balled values for the laser position. -->
+	<property name="base_laser_x" value="0.150" />
+	<property name="base_laser_y" value="0.055" />
+	<property name="base_laser_z" value="0.200" />
+	<property name="base_laser_size_x" value="0.06" />
+	<property name="base_laser_size_y" value="0.06" />
+	<property name="base_laser_size_z" value="0.03" />
+	<property name="base_laser_collision_offset_z" value="0.023" />
 	<xacro:base name="base" />
 	<xacro:wheel side="R" reflectSide="-1" face="B" reflectFace="-1" parent="base_link"/>

File: urdf/base/base.urdf.xacro (robot description, xacro)
@@ -7,12 +7,4 @@
 	<include filename="$(find johnny_0_description)/urdf/base/base.gazebo.xacro" />
 	<property name="base_collision_size_z" value="0.04" />
-	<!-- Warning: eye-balled values for the laser position. -->
-	<property name="base_laser_x" value="0.150" />
-	<property name="base_laser_y" value="0.055" />
-	<property name="base_laser_z" value="0.200" />
-	<property name="base_laser_size_x" value="0.06" />
-	<property name="base_laser_size_y" value="0.06" />
-	<property name="base_laser_size_z" value="0.03" />
-	<property name="base_laser_collision_offset_z" value="0.023" />
 	<xacro:macro name="base" params="name">
 		<joint name="${name}_fixed_joint" type="fixed">
