Commit message: Refs #175. Some work done for the UniDrive and interactive arm configuration. Possible timing problem with the driver: can't reliably get a full state or conversion ratios.
git-svn-id: svn+ssh://marvin.3it.usherbrooke.ca/svn/introlab/johnny0/svn/branches/M9/ros-pkgs/irl_robots/jn0_description@1324 23a761d4-b60a-4777-9503-f06a07968eac

File: robots/junior.urdf.xacro (robot description, xacro)
@@ -26,5 +26,6 @@
 		 -->
 	<!-- Base Azimut 3 + Laser -->
-	<include filename="$(find az3_description)/robots/azimut_3.urdf.xacro" />
+	<!-- include filename="$(find az3_description)/robots/azimut_3.urdf.xacro" /-->
+    <link name="base_link"/>
 	<property name="base_height"  value="0.17" />
 	<xacro:box_torso

Commit message: Refs #176. Added laser to junior
git-svn-id: svn+ssh://marvin.3it.usherbrooke.ca/svn/introlab/johnny0/svn/branches/M9/ros-pkgs/irl_robots/jn0_description@1424 23a761d4-b60a-4777-9503-f06a07968eac

File: robots/junior.urdf.xacro (robot description, xacro)
@@ -13,9 +13,10 @@
 	<include filename="$(find irl_common_description)/urdf/jn0_head/head.urdf.xacro" />
 	<include filename="$(find irl_common_description)/urdf/sensors/kinect.urdf.xacro" />
+	<include filename="$(find irl_common_description)/urdf/sensors/hokuyo_lx04_laser.urdf.xacro" />
 	<!-- generic simulator_gazebo plugins for starting mechanism control, ros time, ros battery -->
 	<include filename="$(find jn0_description)/gazebo/gazebo.urdf.xacro" />
 	<!-- materials for visualization -->
 	<!-- FIXME  Materials from azimut -->
-	<!--include filename="$(find jn0_description)/urdf/materials.urdf.xacro" /-->
+	<include filename="$(find irl_common_description)/urdf/materials.urdf.xacro" />
 	<!-- TODO screenshots in irl_common_description ? -->
 	<!-- TODO ticket wg like robot package
@@ -53,10 +54,4 @@
 		offset_z = "0.02"
 		/>
-	<xacro:kinect_static
-		name="openni"
-		parent="torso_top_frame"
-		xyz="0.17 0 0" rpy="0 0 0"
-		angle="-0.35"
-		/>
 	<xacro:interactive_arm
 		name="arm"
@@ -66,3 +61,18 @@
 		offset_z="0"
 		/>
+	<xacro:kinect_static
+		name="openni"
+		parent="torso_top_frame"
+		xyz="0.17 0 0" rpy="0 0 0"
+		angle="-0.35"
+		/>
+	<xacro:hokuyo_lx04_laser_v0
+		name="base_laser"
+		parent="base"
+		ros_topic="/sensors/base_scan"
+		update_rate="20"
+		min_angle="-2.2689"
+		max_angle="2.2689" >
+		<origin xyz="1 0 0" rpy="0 0 0" />
+	</xacro:hokuyo_lx04_laser_v0>
 </robot>

Commit message: Refs #189, #190. A few fixes to the base and laser relative positions, topic name mappings for face commands, and leg detection settings.
git-svn-id: svn+ssh://marvin.3it.usherbrooke.ca/svn/introlab/johnny0/svn/branches/M9/ros-pkgs/irl_robots/jn0_description@1523 23a761d4-b60a-4777-9503-f06a07968eac

File: robots/junior.urdf.xacro (robot description, xacro)
@@ -26,8 +26,7 @@
 		   {xxx}_msgs
 		 -->
-	<!-- Base Azimut 3 + Laser -->
-	<!-- include filename="$(find az3_description)/robots/azimut_3.urdf.xacro" /-->
+	<!-- Junior torso with U2S base and separate laser -->
     <link name="base_link"/>
-	<property name="base_height"  value="0.17" />
+	<property name="base_height"  value="0.45" />
 	<xacro:box_torso
 		name="torso"
@@ -72,7 +71,7 @@
 		ros_topic="/sensors/base_scan"
 		update_rate="20"
-		min_angle="-2.2689"
-		max_angle="2.2689" >
-		<origin xyz="1 0 0" rpy="0 0 0" />
+		min_angle="-1.57"
+		max_angle="1.57" >
+		<origin xyz="0.4 1 ${base_height}" rpy="0 0 0" />
 	</xacro:hokuyo_lx04_laser_v0>
 </robot>

Commit message: Refs #189. Laser position.
git-svn-id: svn+ssh://marvin.3it.usherbrooke.ca/svn/introlab/johnny0/svn/branches/M9/ros-pkgs/irl_robots/jn0_description@1550 23a761d4-b60a-4777-9503-f06a07968eac

File: robots/junior.urdf.xacro (robot description, xacro)
@@ -73,5 +73,5 @@
 		min_angle="-1.57"
 		max_angle="1.57" >
-		<origin xyz="0.4 1 ${base_height}" rpy="0 0 0" />
+		<origin xyz="0.3 -0.5 ${base_height}" rpy="0 0 0" />
 	</xacro:hokuyo_lx04_laser_v0>
 </robot>
