Commit message: Refs #111. #378. Splitting Johnny-0 URDF into its own macro to avoid repetitions between jn0_full and jn0_standalone, adding link for IMV camera.
git-svn-id: svn+ssh://marvin.3it.usherbrooke.ca/svn/introlab/johnny0/svn/trunk/ros-pkgs/irl_robots/jn0_description@3107 23a761d4-b60a-4777-9503-f06a07968eac

File: robots/jn0_standalone.urdf.xacro (robot description, xacro)
@@ -5,6 +5,4 @@
        xmlns:xacro="http://playerstage.sourceforge.net/gazebo/xmlschema/#interface"
        name="johnny_0" >
-    <!-- AZIMUT 3 files (includes common files found in irl_common_description) -->
-    <include filename="$(find az3_description)/robots/azimut_3.urdf.xacro" />
     <!-- Johnny-0 (the torso and arms) macro -->
     <include filename="$(find jn0_description)/robots/johnny_0.urdf.xacro" />

File: robots/johnny_0.urdf.xacro (robot description, xacro)
@@ -26,73 +26,98 @@
 		   {xxx}_msgs
 		 -->
-    <link name="base_link">
-        <inertial>
-            <mass value="10.000" />
-            <origin xyz="0 0 0" rpy="0 0 0" />
-            <inertia ixx="0.0001" ixy="0" ixz="0" iyy="0.000001" iyz="0" izz="0.0001" />
-        </inertial>
-        <visual>
-          <origin xyz="0 0 0" rpy="0 0 0" />
-          <geometry>
-            <box size="0.04 0.04 0.08" />
-          </geometry>
-          <material name="Red" />
-        </visual>
-        <collision>
-          <origin xyz="0 0 0" rpy="0 0 0" />
-        <geometry>
-          <box size="1.000 1.000 .001" />
-        </geometry>
-      </collision>
-    </link>
-	<property name="base_height"  value="0.25" />
-	<xacro:box_torso
-		name="torso"
-		parent="base_link"
-		xyz = "0 0 ${base_height}"
-		height       = "0.55"
-		stand_width  = "0.038"
-		chest_width  = "0.270"
-		chest_length = "0.21583"
-		chest_height = "0.37921"
-		/>
-	<xacro:irl_ptu
-		name="neck"
-		parent="torso_top_frame"
-		offset_x="0"
-		offset_y="0"
-		offset_z="0"
-    />
-	<xacro:jn0_head
-		name="head"
-		parent="neck_top_frame"
-		offset_x = "0"
-		offset_y = "0"
-		offset_z = "0.02"
-		/>
-	<xacro:arm
-		parent="torso_link"
-        side="R"
-        reflect="-1"
-		/>
-	<xacro:arm
-		parent="torso_link"
-        side="L"
-        reflect="1"
-		/>
-	<xacro:kinect_static
-		name="openni"
-		parent="head_link"
-		xyz="0.070 0 0.17" rpy="0 -0.051 0"
-		angle="0.0"
-		/>
-	<xacro:hokuyo_lx04_laser_v0
-		name="base_laser"
-		parent="base"
-		ros_topic="base_scan"
-		update_rate="20"
-		min_angle="-1.57"
-		max_angle="1.57" >
-		<origin xyz="0.1 0.0 ${base_height}" rpy="0 0 0" />
-	</xacro:hokuyo_lx04_laser_v0>
+    <xacro:macro name="johnny_0" params="base_height">
+        <link name="base_link">
+            <inertial>
+                <mass value="10.000" />
+                <origin xyz="0 0 0" rpy="0 0 0" />
+                <inertia ixx="0.0001" ixy="0" ixz="0" iyy="0.000001" iyz="0" izz="0.0001" />
+            </inertial>
+            <visual>
+              <origin xyz="0 0 0" rpy="0 0 0" />
+              <geometry>
+                <box size="0.04 0.04 0.08" />
+              </geometry>
+              <material name="Red" />
+            </visual>
+            <collision>
+              <origin xyz="0 0 0" rpy="0 0 0" />
+            <geometry>
+              <box size="1.000 1.000 .001" />
+            </geometry>
+          </collision>
+        </link>
+        <xacro:box_torso
+            name="torso"
+            parent="base_link"
+            xyz = "0 0 ${base_height}"
+            height       = "0.55"
+            stand_width  = "0.038"
+            chest_width  = "0.270"
+            chest_length = "0.21583"
+            chest_height = "0.37921"
+            />
+        <xacro:irl_ptu
+            name="neck"
+            parent="torso_top_frame"
+            offset_x="0"
+            offset_y="0"
+            offset_z="0"
+        />
+        <xacro:jn0_head
+            name="head"
+            parent="neck_top_frame"
+            offset_x = "0"
+            offset_y = "0"
+            offset_z = "0.02"
+            />
+        <joint name="imv_camera_fixed_joint" type="fixed">
+            <origin xyz="0.00 0.00 -0.02" rpy="0 0 0"/>
+            <parent link="torso_top_frame"/>
+            <child  link="imv_camera_link"/>
+        </joint>
+        <link name="imv_camera_link">
+            <inertial>
+                <mass value="0.1"/>
+                <origin xyz="0 0 0" rpy="0 0 0"/>
+                <inertia ixx="0.0001" ixy="0.0" iyy="0.0001" iyz="0.0" izz="0.0001"/>
+            </inertial>
+            <visual>
+                <origin xyz="0.0.0" rpy="0.0.0"/>
+                <geometry>
+                    <box size="0.04 0.04 0.04"/>
+                </geometry>
+            </visual>
+            <collision>
+                <origin xyz="0.0.0" rpy="0.0.0"/>
+                <geometry>
+                    <box size="0.04 0.04 0.04"/>
+                </geometry>
+            </collision>
+        </link>
+        <xacro:arm
+            parent="torso_link"
+            side="R"
+            reflect="-1"
+            />
+        <xacro:arm
+            parent="torso_link"
+            side="L"
+            reflect="1"
+            />
+        <xacro:kinect_static
+            name="openni"
+            parent="head_link"
+            xyz="0.070 0 0.17" rpy="0 -0.051 0"
+            angle="0.0"
+            />
+        <xacro:hokuyo_lx04_laser_v0
+            name="base_laser"
+            parent="base"
+            ros_topic="base_scan"
+            update_rate="20"
+            min_angle="-1.57"
+            max_angle="1.57" >
+            <origin xyz="0.1 0.0 ${base_height}" rpy="0 0 0" />
+        </xacro:hokuyo_lx04_laser_v0>
+    </xacro:macro>
 </robot>
