Commit message: change some urdf files to not link the robot with the floor and to initiate the robot above the floor (adding a base_foot_print link) + adding the default controller of pr2 for johnny_0
git-svn-id: svn+ssh://marvin.3it.usherbrooke.ca/svn/introlab/johnny0/svn/branches/M6/ros-pkgs/johnny_0_model/johnny_0_description@558 23a761d4-b60a-4777-9503-f06a07968eac

File: robots/johnny_0.urdf.xacro (robot description, xacro)
@@ -4,5 +4,5 @@
        xmlns:interface="http://playerstage.sourceforge.net/gazebo/xmlschema/#interface"
        xmlns:xacro="http://playerstage.sourceforge.net/gazebo/xmlschema/#interface"
-       name="brasADE" >
+       name="johnny_0" >
 	<!-- The following included files set up definitions of parts of the robot body -->
 	<include filename="$(find johnny_0_description)/urdf/common.xacro" />
@@ -27,5 +27,5 @@
        the origin block defines where the component is w.r.t its parent (in this case the parent
        is the world frame). For more, see http://www.ros.org/wiki/xacro -->
-	<xacro:base name="base" parent="world"/>
+	<xacro:base name="base" />
 	<xacro:wheel side="R" reflectSide="-1" face="B" reflectFace="-1" parent="base_link"/>
 	<xacro:wheel side="R" reflectSide="-1" face="F" reflectFace="1" parent="base_link"/>

File: urdf/base/base.urdf.xacro (robot description, xacro)
@@ -4,16 +4,18 @@
        xmlns:interface="http://playerstage.sourceforge.net/gazebo/xmlschema/#interface"
        xmlns:xacro="http://ros.org/wiki/xacro">
-	<xacro:macro name="base" params="name parent">
-		<joint name="${name}_fixed_joint" type="fixed">
+  <property name="base_collision_size_z" value="0.04" />
+	<xacro:macro name="base" params="name">
+		<!-- Suppression of the link between the world and the base -->
+		<!--joint name="${name}_fixed_joint" type="fixed">
 				<parent link="${parent}"/>
 				<child link="${name}_link"/>
 				<origin xyz="0 0 0.22" rpy="0 0 0" />
-		</joint>
+		</joint-->
 		<link name="${name}_link">
 		  <inertial>
-			<mass value="0.5" />
+			<mass value="50" />
 			<origin xyz="0 0 0" />
-			<inertia ixx="0" ixy="0" ixz="0"
-					 iyy="0" iyz="0" izz="0" />
+			<inertia ixx="3" ixy="0" ixz="0"
+					 iyy="3" iyz="0" izz="3" />
 		  </inertial>
 		  <visual name="${name}_visual">
@@ -24,10 +26,40 @@
 		  </visual>
 		  <collision name="${name}_collision">
-			<origin xyz="0 0 0" rpy="0 0 0" />
+			<origin xyz="0 0 0.01" rpy="0 0 0" />
 			<geometry name="${name}_collision_geom">
-				<box size="0.31322 0.30376 0.24729" />
+				<box size="0.30376 0.31322 0.2" />
 			</geometry>
 		  </collision>
 		</link>
+		<!-- base_footprint is a fictitious link(frame) that is on the ground right below base_link origin,
+			navigation stack dedpends on this frame -->
+		<link name="${name}_footprint">
+		  <inertial>
+			<mass value="1.0" />
+			<origin xyz="0 0 0" />
+			<inertia ixx="0.01" ixy="0.0" ixz="0.0"
+					iyy="0.01" iyz="0.0" izz="0.01" />
+		  </inertial>
+		  <visual>
+			<origin xyz="0 0 0" rpy="0 0 0" />
+			<geometry>
+			  <box size="0.01 0.01 0.01" />
+			</geometry>
+			<material name="Green" />
+		  </visual>
+		  <collision>
+			<!-- represent base collision with a simple rectangular model, positioned by base_size_z s.t. top
+				surface of the collision box matches the top surface of the PR2 base -->
+			<origin xyz="0 0 ${0.251+base_collision_size_z/2}" rpy="0 0 0" />
+			<geometry>
+			  <box size="0.001 0.001 0.001" />
+			</geometry>
+		  </collision>
+		</link>
+		<joint name="${name}_footprint_joint" type="fixed">
+		  <origin xyz="0 0 0.251" rpy="0 0 0" />
+		  <child link="${name}_link" />
+		  <parent link="${name}_footprint"/>
+		</joint>
 		<gazebo reference="${name}_link">
 			<material>Gazebo/Blue</material>

File: urdf/wheel/wheel.urdf.xacro (robot description, xacro)
@@ -83,8 +83,9 @@
 			</collision>
 		</link>
-		<joint name="wheel${side}${face}_wheel_fixed_joint" type="fixed">
+		<joint name="wheel${side}${face}_wheel_continuous_joint" type="continuous">
 			<parent link="wheel${side}${face}_ADE2_link"/>
 			<child link="wheel${side}${face}_wheel_link"/>
 			<origin xyz="0.07492 0 0" rpy="0 ${M_PI/2} 0" />
+			<axis xyz="0 0 1"/>
 		</joint>
 		<link name="wheel${side}${face}_wheel_link">

Commit message: Add the base laser to the johnny0 gazebo model, removes a logging message from az3_gazebo_ctrl.
git-svn-id: svn+ssh://marvin.3it.usherbrooke.ca/svn/introlab/johnny0/svn/branches/M6/ros-pkgs/johnny_0_model/johnny_0_description@611 23a761d4-b60a-4777-9503-f06a07968eac

File: robots/johnny_0.urdf.xacro (robot description, xacro)
@@ -8,4 +8,5 @@
 	<include filename="$(find johnny_0_description)/urdf/common.xacro" />
 	<!-- Description files -->
+	<include filename="$(find johnny_0_description)/urdf/sensors/hokuyo_lx04_laser.urdf.xacro" />
 	<include filename="$(find johnny_0_description)/urdf/base/base.urdf.xacro" />
 	<include filename="$(find johnny_0_description)/urdf/wheel/wheel.urdf.xacro" />

File: urdf/base/base.urdf.xacro (robot description, xacro)
@@ -4,7 +4,15 @@
        xmlns:interface="http://playerstage.sourceforge.net/gazebo/xmlschema/#interface"
        xmlns:xacro="http://ros.org/wiki/xacro">
-	<!-- Include files for extansions -->
+	<!-- Include files for extensions -->
 	<include filename="$(find johnny_0_description)/urdf/base/base.gazebo.xacro" />
 	<property name="base_collision_size_z" value="0.04" />
+	<!-- Warning: eye-balled values for the laser position. -->
+	<property name="base_laser_x" value="0.15" />
+	<property name="base_laser_y" value="0.0" />
+	<property name="base_laser_z" value="0.4" />
+	<property name="base_laser_size_x" value="0.06" />
+	<property name="base_laser_size_y" value="0.06" />
+	<property name="base_laser_size_z" value="0.03" />
+	<property name="base_laser_collision_offset_z" value="0.023" />
 	<xacro:macro name="base" params="name">
 		<!-- Suppression of the link between the world and the base -->
@@ -57,5 +65,5 @@
 		  <collision>
 			<!-- represent base collision with a simple rectangular model, positioned by base_size_z s.t. top
-				surface of the collision box matches the top surface of the PR2 base -->
+				surface of the collision box matches the top surface of the AZ3 base -->
 			<origin xyz="0 0 ${0.251+base_collision_size_z/2}" rpy="0 0 0" />
 			<geometry>
@@ -64,4 +72,11 @@
 		  </collision>
 		</link>
+		<!-- front laser -->
+		<xacro:hokuyo_lx04_laser_v0 name="${name}_laser" parent="${name}"
+			ros_topic="/sensors/base_scan" update_rate="20" min_angle="-2.2689"
+			max_angle="2.2689" >
+			<origin xyz="${base_laser_x} ${base_laser_y} ${base_laser_z}"
+			rpy="0 0 0" />
+		</xacro:hokuyo_lx04_laser_v0>
 		<!-- gazebo extensions -->
 		<xacro:johnny_0_base_gazebo name="${name}" />

Commit message: refs #155 adding the kinect in johnny_0 model, have to check if it is at the reight place
git-svn-id: svn+ssh://marvin.3it.usherbrooke.ca/svn/introlab/johnny0/svn/branches/M8/ros-pkgs/johnny_0_model/johnny_0_description@1049 23a761d4-b60a-4777-9503-f06a07968eac

File: robots/johnny_0.urdf.xacro (robot description, xacro)
@@ -43,3 +43,6 @@
 		<origin xyz="0.06 0 ${head_size_z/2 + bumblebee_size_z/2}" />
 	</xacro:bumblebee>
+	<xacro:bumblebee name="kinect_camera" parent="torso_link">
+		<origin xyz="0.17 0 ${torso_size_z/2 + bumblebee_size_z/2}" />
+	</xacro:bumblebee>
 </robot>

Commit message: refs #155 adding the kinect in the urdf model of johnny_0
git-svn-id: svn+ssh://marvin.3it.usherbrooke.ca/svn/introlab/johnny0/svn/branches/M8/ros-pkgs/johnny_0_model/johnny_0_description@1062 23a761d4-b60a-4777-9503-f06a07968eac

File: robots/johnny_0.urdf.xacro (robot description, xacro)
@@ -16,4 +16,5 @@
 	<include filename="$(find johnny_0_description)/urdf/head/head.urdf.xacro" />
 	<include filename="$(find johnny_0_description)/urdf/camera/bumblebee.urdf.xacro" />
+	<include filename="$(find johnny_0_description)/urdf/camera/kinect.urdf.xacro" />
 	<!-- generic simulator_gazebo plugins for starting mechanism control, ros time, ros battery -->
 	<include filename="$(find johnny_0_description)/gazebo/gazebo.urdf.xacro" />
@@ -43,6 +44,6 @@
 		<origin xyz="0.06 0 ${head_size_z/2 + bumblebee_size_z/2}" />
 	</xacro:bumblebee>
-	<xacro:bumblebee name="kinect_camera" parent="torso_link">
-		<origin xyz="0.17 0 ${torso_size_z/2 + bumblebee_size_z/2}" />
-	</xacro:bumblebee>
+	<xacro:kinect name="openni_camera" parent="torso_link">
+		<origin xyz="0.17 0 ${torso_size_z/2 + kinect_size_z/2}" rpy="0 -0.35 0"/>
+	</xacro:kinect>
 </robot>

Commit message: Refs #176. Using azimut 3 from irl_common_description
git-svn-id: svn+ssh://marvin.3it.usherbrooke.ca/svn/introlab/johnny0/svn/branches/M9/ros-pkgs/irl_robots/jn0_description@1273 23a761d4-b60a-4777-9503-f06a07968eac

File: robots/johnny_0.urdf.xacro (robot description, xacro)
@@ -6,19 +6,20 @@
        name="johnny_0" >
 	<!-- The following included files set up definitions of parts of the robot body -->
-	<include filename="$(find johnny_0_description)/urdf/common.xacro" />
+	<include filename="$(find jn0_description)/urdf/common.xacro" />
 	<!-- Description files -->
-	<include filename="$(find johnny_0_description)/urdf/sensors/hokuyo_lx04_laser.urdf.xacro" />
-	<include filename="$(find johnny_0_description)/urdf/base/base.urdf.xacro" />
-	<include filename="$(find johnny_0_description)/urdf/wheel/wheel.urdf.xacro" />
-	<include filename="$(find johnny_0_description)/urdf/baseTorsoLink/baseTorsoLink.urdf.xacro" />
-	<include filename="$(find johnny_0_description)/urdf/torso/torso.urdf.xacro" />
-	<include filename="$(find johnny_0_description)/urdf/arm/arm.urdf.xacro" />
-	<include filename="$(find johnny_0_description)/urdf/head/head.urdf.xacro" />
-	<include filename="$(find johnny_0_description)/urdf/camera/bumblebee.urdf.xacro" />
-	<include filename="$(find johnny_0_description)/urdf/camera/kinect.urdf.xacro" />
+	<include filename="$(find jn0_description)/urdf/sensors/hokuyo_lx04_laser.urdf.xacro" />
+	<!--include filename="$(find jn0_description)/urdf/base/base.urdf.xacro" /-->
+	<!--include filename="$(find jn0_description)/urdf/wheel/wheel.urdf.xacro" /-->
+	<include filename="$(find jn0_description)/urdf/baseTorsoLink/baseTorsoLink.urdf.xacro" />
+	<include filename="$(find jn0_description)/urdf/torso/torso.urdf.xacro" />
+	<include filename="$(find jn0_description)/urdf/arm/arm.urdf.xacro" />
+	<include filename="$(find jn0_description)/urdf/head/head.urdf.xacro" />
+	<include filename="$(find jn0_description)/urdf/camera/bumblebee.urdf.xacro" />
+	<include filename="$(find jn0_description)/urdf/camera/kinect.urdf.xacro" />
 	<!-- generic simulator_gazebo plugins for starting mechanism control, ros time, ros battery -->
-	<include filename="$(find johnny_0_description)/gazebo/gazebo.urdf.xacro" />
+	<include filename="$(find jn0_description)/gazebo/gazebo.urdf.xacro" />
 	<!-- materials for visualization -->
-	<include filename="$(find johnny_0_description)/urdf/materials.urdf.xacro" />
+	<!-- FIXME  Materials from azimut -->
+	<!--include filename="$(find jn0_description)/urdf/materials.urdf.xacro" /-->
 	<!-- Now we can start using the macros included above to define the actual PR2 -->
 	<!-- The first use of a macro.
@@ -37,9 +38,6 @@
 	<property name="base_laser_size_z" value="0.03" />
 	<property name="base_laser_collision_offset_z" value="0.023" />
-	<xacro:base name="base" />
-	<xacro:wheel side="R" reflectSide="-1" face="B" reflectFace="-1" parent="base_link"/>
-	<xacro:wheel side="R" reflectSide="-1" face="F" reflectFace="1" parent="base_link"/>
-	<xacro:wheel side="L" reflectSide="1" face="B" reflectFace="-1" parent="base_link"/>
-	<xacro:wheel side="L" reflectSide="1" face="F" reflectFace="1" parent="base_link"/>
+	<!--xacro:base name="base" /-->
+	<include filename="$(find az3_description)/robots/azimut_3.urdf.xacro" />
 	<xacro:baseTorsoLink name="baseTorsoLink" parent="base_link"/>
 	<xacro:torso name="torso" parent="baseTorsoLink_link"/>

File: urdf/arm/ADE_pitch_elbow/ADE_pitch_elbow.urdf.xacro (robot description, xacro)
@@ -4,5 +4,5 @@
        xmlns:interface="http://playerstage.sourceforge.net/gazebo/xmlschema/#interface"
        xmlns:xacro="http://ros.org/wiki/xacro">
-	<include filename="$(find johnny_0_description)/urdf/arm/arm.transmission.xacro" />
+	<include filename="$(find jn0_description)/urdf/arm/arm.transmission.xacro" />
 	<xacro:macro name="ADE_pitch_elbow" params="side reflect parent">
 		<link name="ADE_pitch_elbow${side}_box">
@@ -88,5 +88,5 @@
 		</joint>
 		<!-- extensions -->
-		<xacro:johnny_0_ADE_pitch_elbow_transmission side="${side}" />
+		<xacro:jn0_ADE_pitch_elbow_transmission side="${side}" />
 		<gazebo reference="ADE_pitch_elbow${side}_box">
 			<material>Gazebo/Green</material>

File: urdf/arm/ADE_pitch_shoulder/ADE_pitch_shoulder.urdf.xacro (robot description, xacro)
@@ -4,5 +4,5 @@
        xmlns:interface="http://playerstage.sourceforge.net/gazebo/xmlschema/#interface"
        xmlns:xacro="http://ros.org/wiki/xacro">
-	<include filename="$(find johnny_0_description)/urdf/arm/arm.transmission.xacro" />
+	<include filename="$(find jn0_description)/urdf/arm/arm.transmission.xacro" />
 	<xacro:macro name="ADE_pitch_shoulder" params="side reflect parent">
 		<joint name="ADE_pitch_shoulder${side}_fixed_1_joint" type="fixed">
@@ -88,5 +88,5 @@
 		</link>
 		<!-- extensions -->
-		<xacro:johnny_0_ADE_pitch_shoulder_transmission side="${side}" />
+		<xacro:jn0_ADE_pitch_shoulder_transmission side="${side}" />
 		<gazebo reference="ADE_pitch_shoulder${side}_link">
 			<material>Gazebo/Red</material>

File: urdf/arm/ADE_roll/ADE_roll.urdf.xacro (robot description, xacro)
@@ -4,5 +4,5 @@
        xmlns:interface="http://playerstage.sourceforge.net/gazebo/xmlschema/#interface"
        xmlns:xacro="http://ros.org/wiki/xacro">
-	<include filename="$(find johnny_0_description)/urdf/arm/arm.transmission.xacro" />
+	<include filename="$(find jn0_description)/urdf/arm/arm.transmission.xacro" />
 	<xacro:macro name="ADE_roll" params="side reflect parent">
 		<joint name="ADE_roll${side}_fixed_origine_joint" type="fixed">
@@ -89,5 +89,5 @@
 		</link>
 		<!-- extensions -->
-		<xacro:johnny_0_ADE_roll_shoulder_transmission side="${side}" />
+		<xacro:jn0_ADE_roll_shoulder_transmission side="${side}" />
 		<gazebo reference="ADE_roll${side}_box">
 			<material>Gazebo/Blue</material>

File: urdf/arm/arm.transmission.xacro (robot description, xacro)
@@ -6,5 +6,5 @@
   <!-- ============================   Arm   ============================ -->
   <!-- ADE roll shoulder -->
-  <xacro:macro name="johnny_0_ADE_roll_shoulder_transmission" params="side" >
+  <xacro:macro name="jn0_ADE_roll_shoulder_transmission" params="side" >
     <transmission type="pr2_mechanism_model/SimpleTransmission" name="${side}_ADE_roll_shoulder_trans">
       <actuator name="${side}_ADE_roll_shoulder_motor" />
@@ -14,5 +14,5 @@
   </xacro:macro>
   <!-- ADE pitch shoulder -->
-  <xacro:macro name="johnny_0_ADE_pitch_shoulder_transmission" params="side" >
+  <xacro:macro name="jn0_ADE_pitch_shoulder_transmission" params="side" >
     <transmission type="pr2_mechanism_model/SimpleTransmission" name="${side}_ADE_pitch_shoulder_trans">
       <actuator name="${side}_ADE_pitch_shoulder_motor" />
@@ -22,5 +22,5 @@
   </xacro:macro>
   <!--  ADE pitch elbow -->
-  <xacro:macro name="johnny_0_ADE_pitch_elbow_transmission" params="side" >
+  <xacro:macro name="jn0_ADE_pitch_elbow_transmission" params="side" >
     <transmission type="pr2_mechanism_model/SimpleTransmission" name="${side}_ADE_pitch_elbow_trans">
       <actuator name="${side}_ADE_pitch_elbow_motor" />

File: urdf/arm/arm.urdf.xacro (robot description, xacro)
@@ -5,9 +5,9 @@
        xmlns:xacro="http://playerstage.sourceforge.net/gazebo/xmlschema/#interface"
        name="arm">
-	<include filename="$(find johnny_0_description)/urdf/arm/ADE_roll/ADE_roll.urdf.xacro" />
-	<include filename="$(find johnny_0_description)/urdf/arm/ADE_pitch_shoulder/ADE_pitch_shoulder.urdf.xacro" />
-	<include filename="$(find johnny_0_description)/urdf/arm/ADE_pitch_elbow/ADE_pitch_elbow.urdf.xacro" />
-	<include filename="$(find johnny_0_description)/urdf/arm/forearm/forearm.urdf.xacro" />
-	<include filename="$(find johnny_0_description)/urdf/arm/hand/hand.urdf.xacro" />
+	<include filename="$(find jn0_description)/urdf/arm/ADE_roll/ADE_roll.urdf.xacro" />
+	<include filename="$(find jn0_description)/urdf/arm/ADE_pitch_shoulder/ADE_pitch_shoulder.urdf.xacro" />
+	<include filename="$(find jn0_description)/urdf/arm/ADE_pitch_elbow/ADE_pitch_elbow.urdf.xacro" />
+	<include filename="$(find jn0_description)/urdf/arm/forearm/forearm.urdf.xacro" />
+	<include filename="$(find jn0_description)/urdf/arm/hand/hand.urdf.xacro" />
 	<xacro:macro name="arm" params="side reflect parent">
 		<xacro:ADE_roll side="${side}" reflect="${reflect}" parent="${parent}"/>

File: urdf/head/head.transmission.xacro (robot description, xacro)
@@ -6,5 +6,5 @@
   <!-- ============================   Head   ============================ -->
   <!-- Head pan (or yaw) -->
-  <xacro:macro name="johnny_0_head_pan_transmission" >
+  <xacro:macro name="jn0_head_pan_transmission" >
     <transmission type="pr2_mechanism_model/SimpleTransmission" name="head_pan_trans">
       <actuator name="head_pan_motor" />
@@ -14,5 +14,5 @@
   </xacro:macro>
   <!-- Head tilt (or roll) -->
-  <xacro:macro name="johnny_0_head_tilt_transmission" >
+  <xacro:macro name="jn0_head_tilt_transmission" >
     <transmission type="pr2_mechanism_model/SimpleTransmission" name="head_tilt_trans">
       <actuator name="head_tilt_motor" />

File: urdf/head/head.urdf.xacro (robot description, xacro)
@@ -4,5 +4,5 @@
        xmlns:interface="http://playerstage.sourceforge.net/gazebo/xmlschema/#interface"
        xmlns:xacro="http://ros.org/wiki/xacro">
-	<include filename="$(find johnny_0_description)/urdf/head/head.transmission.xacro" />
+	<include filename="$(find jn0_description)/urdf/head/head.transmission.xacro" />
 	<property name="pan_size_z" value="0.05" />
 	<property name="head_size_z" value="0.17" />
@@ -119,6 +119,6 @@
 		</link>
 		<!-- extansions -->
-		<xacro:johnny_0_head_tilt_transmission />
-		<xacro:johnny_0_head_pan_transmission />
+		<xacro:jn0_head_tilt_transmission />
+		<xacro:jn0_head_pan_transmission />
 		<gazebo reference="${name}_link">
 			<material>Gazebo/Green</material>

File: urdf/sensors/hokuyo_lx04_laser.urdf.xacro (robot description, xacro)
@@ -4,5 +4,5 @@
        xmlns:interface="http://playerstage.sourceforge.net/gazebo/xmlschema/#interface"
        xmlns:xacro="http://ros.org/wiki/xacro">
-  <include filename="$(find johnny_0_description)/urdf/sensors/hokuyo_lx04_laser.gazebo.xacro" />
+  <include filename="$(find jn0_description)/urdf/sensors/hokuyo_lx04_laser.gazebo.xacro" />
   <xacro:macro name="hokuyo_lx04_laser_v0" params="name parent *origin ros_topic update_rate min_angle max_angle">
     <joint name="${name}_joint" type="fixed">

File: urdf/sensors/hokuyo_lx30_laser.urdf.xacro (robot description, xacro)
@@ -4,5 +4,5 @@
        xmlns:interface="http://playerstage.sourceforge.net/gazebo/xmlschema/#interface"
        xmlns:xacro="http://ros.org/wiki/xacro">
-  <include filename="$(find johnny_0_description)/urdf/sensors/hokuyo_lx30_laser.gazebo.xacro" />
+  <include filename="$(find jn0_description)/urdf/sensors/hokuyo_lx30_laser.gazebo.xacro" />
   <xacro:macro name="hokuyo_lx30_laser_v0" params="name parent *origin ros_topic update_rate min_angle max_angle">
     <joint name="${name}_joint" type="fixed">

Commit message: Refs #176. Moving sensors to irl_common_description. Merged kinect and kinect_camera models.
git-svn-id: svn+ssh://marvin.3it.usherbrooke.ca/svn/introlab/johnny0/svn/branches/M9/ros-pkgs/irl_robots/jn0_description@1275 23a761d4-b60a-4777-9503-f06a07968eac

File: robots/johnny_0.urdf.xacro (robot description, xacro)
@@ -8,13 +8,9 @@
 	<include filename="$(find jn0_description)/urdf/common.xacro" />
 	<!-- Description files -->
-	<include filename="$(find jn0_description)/urdf/sensors/hokuyo_lx04_laser.urdf.xacro" />
-	<!--include filename="$(find jn0_description)/urdf/base/base.urdf.xacro" /-->
-	<!--include filename="$(find jn0_description)/urdf/wheel/wheel.urdf.xacro" /-->
 	<include filename="$(find jn0_description)/urdf/baseTorsoLink/baseTorsoLink.urdf.xacro" />
 	<include filename="$(find jn0_description)/urdf/torso/torso.urdf.xacro" />
 	<include filename="$(find jn0_description)/urdf/arm/arm.urdf.xacro" />
 	<include filename="$(find jn0_description)/urdf/head/head.urdf.xacro" />
-	<include filename="$(find jn0_description)/urdf/camera/bumblebee.urdf.xacro" />
-	<include filename="$(find jn0_description)/urdf/camera/kinect.urdf.xacro" />
+	<include filename="$(find irl_common_description)/urdf/sensors/kinect.urdf.xacro" />
 	<!-- generic simulator_gazebo plugins for starting mechanism control, ros time, ros battery -->
 	<include filename="$(find jn0_description)/gazebo/gazebo.urdf.xacro" />
@@ -22,21 +18,5 @@
 	<!-- FIXME  Materials from azimut -->
 	<!--include filename="$(find jn0_description)/urdf/materials.urdf.xacro" /-->
-	<!-- Now we can start using the macros included above to define the actual PR2 -->
-	<!-- The first use of a macro.
-       A macro like this will expand to a set of link and joint definitions, and to additional
-       Gazebo-related extensions (sensor plugins, etc).  The macro takes an argument, name,
-       that equals "base", and uses it to generate names for its component links and joints
-       (e.g., base_link).  The included origin block is also an argument to the macro.  By convention,
-       the origin block defines where the component is w.r.t its parent (in this case the parent
-       is the world frame). For more, see http://www.ros.org/wiki/xacro -->
-	<!-- Warning: eye-balled values for the laser position. -->
-	<property name="base_laser_x" value="0.10" />
-	<property name="base_laser_y" value="-0.04" />
-	<property name="base_laser_z" value="0.200" />
-	<property name="base_laser_size_x" value="0.06" />
-	<property name="base_laser_size_y" value="0.06" />
-	<property name="base_laser_size_z" value="0.03" />
-	<property name="base_laser_collision_offset_z" value="0.023" />
-	<!--xacro:base name="base" /-->
+	<!-- Base Azimut 3 + Laser -->
 	<include filename="$(find az3_description)/robots/azimut_3.urdf.xacro" />
 	<xacro:baseTorsoLink name="baseTorsoLink" parent="base_link"/>
@@ -47,9 +27,9 @@
 		<origin xyz="0.04 0 ${torso_size_z/2}" />
 	</xacro:head>
-	<xacro:bumblebee name="head_camera" parent="head_head_link">
-		<origin xyz="0.06 0 ${head_size_z/2 + bumblebee_size_z/2}" />
-	</xacro:bumblebee>
-	<xacro:kinect name="openni_camera" parent="torso_link">
-		<origin xyz="0.17 0 ${torso_size_z/2 + kinect_size_z/2}" rpy="0 -0.35 0"/>
-	</xacro:kinect>
+	<xacro:kinect_static
+		name="openni"
+		parent="torso_link"
+		xyz="0.17 0 ${torso_size_z/2}" rpy="0 0 0"
+		angle="-0.35"
+		/>
 </robot>
