Commit message: Refs #176. Importing head and torso meshes/urdf from Arnaud
git-svn-id: svn+ssh://marvin.3it.usherbrooke.ca/svn/introlab/johnny0/svn/branches/M9/ros-pkgs/irl_robots/jn0_description@1282 23a761d4-b60a-4777-9503-f06a07968eac

File: robots/johnny_0.urdf.xacro (robot description, xacro)
@@ -8,5 +8,5 @@
 	<include filename="$(find irl_common_description)/urdf/common.xacro" />
 	<!-- Description files -->
-	<include filename="$(find irl_common_description)/urdf/jn0_torso/torso_box.urdf.xacro" />
+	<include filename="$(find irl_common_description)/urdf/jn0_torso/reddy_torso.urdf.xacro" />
 	<include filename="$(find irl_common_description)/urdf/reddy_arm/arm.urdf.xacro" />
 	<include filename="$(find irl_common_description)/urdf/jn0_head/head.urdf.xacro" />
@@ -18,26 +18,43 @@
 	<!--include filename="$(find jn0_description)/urdf/materials.urdf.xacro" /-->
 	<!-- TODO screenshots in irl_common_description ? -->
+	<!-- TODO ticket wg like robot package
+		 {xxx}_common
+		   {xxx}_description (urdf, robots, gazebo, meshes)
+		   {xxx}_machine
+		   {xxx}_msgs
+		 -->
 	<!-- Base Azimut 3 + Laser -->
 	<include filename="$(find az3_description)/robots/azimut_3.urdf.xacro" />
-	<property name="torso_size_z" value="0.37921" />
-	<xacro:jn0_torso_box
+	<property name="base_height"  value="0.17" />
+	<property name="torso_height" value="0.55" />
+	<!--xacro:box_torso
 		name="torso"
 		parent="base_link"
-		xyz = "0 0 0.3089"
+		xyz = "0 0 ${base_height}"
+		height       = "${torso_height}"
 		stand_width  = "0.038"
-		stand_height = "0.37038"
 		chest_width  = "0.270"
 		chest_length = "0.21583"
-		chest_height = "${torso_size_z}"
-		/>
-	<xacro:reddy_arm side="R" reflect="-1" parent="torso_link"/>
-	<xacro:reddy_arm side="L" reflect="1" parent="torso_link"/>
-	<xacro:head name="head" parent="torso_link">
-		<origin xyz="0.04 0 ${torso_size_z/2}" />
-	</xacro:head>
+		chest_height = "0.37921"
+		/-->
+	<xacro:reddy_torso name="torso" parent="base_link" />
+	<xacro:macro name="arm" params="side reflect">
+		<xacro:reddy_arm
+			name="${side}_arm"
+			reflect="${reflect}"
+			parent="torso_link"
+			offset_y="0.09"
+			offset_z="${torso_height}"
+			/>
+	</xacro:macro>
+	<xacro:arm side="r" reflect="-1"/>
+	<xacro:arm side="l" reflect="1"/>
+	<xacro:jn0_head name="head" parent="torso_link">
+		<origin xyz="0.04 0 ${torso_height}" />
+	</xacro:jn0_head>
 	<xacro:kinect_static
 		name="openni"
 		parent="torso_link"
-		xyz="0.17 0 ${torso_size_z/2}" rpy="0 0 0"
+		xyz="0.17 0 ${torso_height}" rpy="0 0 0"
 		angle="-0.35"
 		/>

Commit message: Refs #176. Splited head / pan tilt.
git-svn-id: svn+ssh://marvin.3it.usherbrooke.ca/svn/introlab/johnny0/svn/branches/M9/ros-pkgs/irl_robots/jn0_description@1284 23a761d4-b60a-4777-9503-f06a07968eac

File: robots/johnny_0.urdf.xacro (robot description, xacro)
@@ -10,4 +10,5 @@
 	<include filename="$(find irl_common_description)/urdf/jn0_torso/reddy_torso.urdf.xacro" />
 	<include filename="$(find irl_common_description)/urdf/reddy_arm/arm.urdf.xacro" />
+	<include filename="$(find irl_common_description)/urdf/actuators/pan_tilt_ptu46175.urdf.xacro" />
 	<include filename="$(find irl_common_description)/urdf/jn0_head/head.urdf.xacro" />
 	<include filename="$(find irl_common_description)/urdf/sensors/kinect.urdf.xacro" />
@@ -50,7 +51,18 @@
 	<xacro:arm side="r" reflect="-1"/>
 	<xacro:arm side="l" reflect="1"/>
-	<xacro:jn0_head name="head" parent="torso_link">
-		<origin xyz="0.04 0 ${torso_height}" />
-	</xacro:jn0_head>
+	<xacro:pan_tilt_ptu46175
+		name="neck"
+		parent="torso_link"
+		offset_x="0.03"
+		offset_y="0"
+		offset_z="${torso_height}"
+		/>
+	<xacro:jn0_head
+		name="head"
+		parent="neck_bracket_link"
+		offset_x = "0"
+		offset_y = "0"
+		offset_z = "0"
+		/>
 	<xacro:kinect_static
 		name="openni"

Commit message: Refs #111, #378. URDF fixes related to IMV camera as introduced in r3107
git-svn-id: svn+ssh://marvin.3it.usherbrooke.ca/svn/introlab/johnny0/svn/trunk/ros-pkgs/irl_robots/jn0_description@3108 23a761d4-b60a-4777-9503-f06a07968eac

File: robots/johnny_0.urdf.xacro (robot description, xacro)
@@ -80,8 +80,8 @@
                 <mass value="0.1"/>
                 <origin xyz="0 0 0" rpy="0 0 0"/>
-                <inertia ixx="0.0001" ixy="0.0" iyy="0.0001" iyz="0.0" izz="0.0001"/>
+                <inertia ixx="0.0001" ixy="0.0" ixz="0.0" iyy="0.0001" iyz="0.0" izz="0.0001"/>
             </inertial>
             <visual>
-                <origin xyz="0.0.0" rpy="0.0.0"/>
+                <origin xyz="0 0 0" rpy="0 0 0"/>
                 <geometry>
                     <box size="0.04 0.04 0.04"/>
@@ -89,5 +89,5 @@
             </visual>
             <collision>
-                <origin xyz="0.0.0" rpy="0.0.0"/>
+                <origin xyz="0 0 0" rpy="0 0 0"/>
                 <geometry>
                     <box size="0.04 0.04 0.04"/>

Commit message: Refs #111, #378. Geometry fixes in URDF, a few IMV face detection tests in standalone mode - pose transform errors remain.
git-svn-id: svn+ssh://marvin.3it.usherbrooke.ca/svn/introlab/johnny0/svn/trunk/ros-pkgs/irl_robots/jn0_description@3109 23a761d4-b60a-4777-9503-f06a07968eac

File: robots/johnny_0.urdf.xacro (robot description, xacro)
@@ -62,5 +62,5 @@
             offset_x="0"
             offset_y="0"
-            offset_z="0"
+            offset_z="0.045"
         />
         <xacro:jn0_head
@@ -72,5 +72,5 @@
             />
         <joint name="imv_camera_fixed_joint" type="fixed">
-            <origin xyz="0.00 0.00 -0.02" rpy="0 0 0"/>
+            <origin xyz="0.04 0.00 0.044" rpy="0 0 0"/>
             <parent link="torso_top_frame"/>
             <child  link="imv_camera_link"/>
