Commit message: Refs #89, #85. Working base controller for AZ3, fixed wheel positions and orientations to fit with the kinetics controller.
git-svn-id: svn+ssh://marvin.3it.usherbrooke.ca/svn/introlab/johnny0/svn/branches/M6/ros-pkgs/johnny_0_model/johnny_0_description@580 23a761d4-b60a-4777-9503-f06a07968eac

File: urdf/wheel/wheel.urdf.xacro (robot description, xacro)
@@ -11,5 +11,5 @@
 			<parent link="${parent}"/>
 			<child link="wheel${side}${face}_link"/>
-			<origin xyz="${reflectSide*0.17} ${reflectFace*0.17} -0.133645" rpy="0 0 ${reflectFace*(M_PI/4+(1-reflectSide)*M_PI/4)}" />
+			<origin xyz="${reflectFace*0.17} ${reflectSide*0.17} -0.133645" rpy="0 0 ${reflectSide*(M_PI/4+(1-reflectFace)*M_PI/4)}" />
 		</joint>
 		<link name="wheel${side}${face}_link">
@@ -89,5 +89,5 @@
 			<parent link="wheel${side}${face}_ADE2_link"/>
 			<child link="wheel${side}${face}_wheel_link"/>
-			<origin xyz="0.07492 0 0" rpy="0 ${M_PI/2} 0" />
+			<origin xyz="0.07492 0 0" rpy="0 ${-M_PI/2} 0" />
 			<axis xyz="0 0 1"/>
 		</joint>

Commit message: Refs #146. Fix the steering limits that prevented crab-mode and other ICRs.
git-svn-id: svn+ssh://marvin.3it.usherbrooke.ca/svn/introlab/johnny0/svn/branches/M8/ros-pkgs/johnny_0_model/johnny_0_description@939 23a761d4-b60a-4777-9503-f06a07968eac

File: urdf/wheel/wheel.urdf.xacro (robot description, xacro)
@@ -40,5 +40,5 @@
 		<link name="wheel${side}${face}_ADE_link">
 			<inertial>
-				<mass value="0.5" />
+				<mass value="5.0" />
 				<origin xyz="0 0 0" />
 				<inertia ixx="0" ixy="0" ixz="0"
@@ -63,5 +63,6 @@
 			<origin xyz="0 0 -0.12708" rpy="0 0 0" />
 			<axis xyz="0 0 1" rpy="0 0 0"/>
-			<limit effort="100" velocity="0.1" lower="-0.7854" upper="0.7854" />
+			<!-- See az3.cfg for max velocity value. -->
+			<limit effort="100" velocity="1.7442" lower="-1.5708" upper="1.5708" />
 			<!-- calibration reference_position="0.0"/ -->
 		</joint>
@@ -91,8 +92,10 @@
 			<origin xyz="0.07492 0 0" rpy="0 ${-M_PI/2} 0" />
 			<axis xyz="0 0 1"/>
+			<!-- See az3.cfg for max velocity value. -->
+			<limit effort="100" velocity="9.8837"/>
 		</joint>
 		<link name="wheel${side}${face}_wheel_link">
 			<inertial>
-				<mass value="0.5" />
+				<mass value="1.0" />
 				<origin xyz="0 0 0" />
 				<inertia ixx="0" ixy="0" ixz="0"
