Commit message: Refs #171. Moved base parameters out of az3_base URDF, configured in the robot URDF instead. Created a description for AZ2, measured dX1 on the actual robot. Missing wheel diameter parameter, but they're the same.
git-svn-id: svn+ssh://marvin.3it.usherbrooke.ca/svn/introlab/johnny0/svn/branches/AzMC/ros-pkgs/irl_robots/irl_common_description@1209 23a761d4-b60a-4777-9503-f06a07968eac

File: urdf/az3_base/base.urdf.xacro (robot description, xacro)
@@ -6,31 +6,5 @@
 	<!-- Include files for extensions -->
 	<include filename="$(find irl_common_description)/urdf/az3_base/base.gazebo.xacro" />
-	<property name="base_collision_size_z" value="0.04" />
-	<!-- Warning: eye-balled values for the laser position. -->
-	<property name="base_laser_x" value="0.15" />
-	<property name="base_laser_y" value="0.0" />
-	<property name="base_laser_z" value="0.4" />
-	<property name="base_laser_size_x" value="0.06" />
-	<property name="base_laser_size_y" value="0.06" />
-	<property name="base_laser_size_z" value="0.03" />
-	<property name="base_laser_collision_offset_z" value="0.023" />
-	<!-- Properties of the base -->
-	<property name="base_mass" value="26.576444" />
-	<property name="base_cg_x" value="0.001534" />
-	<property name="base_cg_y" value="0.000052" />
-	<property name="base_cg_z" value="0.029541" />
-	<property name="base_ixx" value="1" />
-	<property name="base_ixy" value="0" />
-	<property name="base_ixz" value="0" />
-	<property name="base_iyy" value="1" />
-	<property name="base_iyz" value="0" />
-	<property name="base_izz" value="1" />
 	<xacro:macro name="az3_base" params="name">
-		<!-- Suppression of the link between the world and the base -->
-		<!--joint name="${name}_fixed_joint" type="fixed">
-				<parent link="${parent}"/>
-				<child link="${name}_link"/>
-				<origin xyz="0 0 0.22" rpy="0 0 0" />
-		</joint-->
 		<link name="${name}_link">
 		  <inertial>

File: urdf/az3_wheel_group/wheel.urdf.xacro (robot description, xacro)
@@ -7,32 +7,4 @@
 	<include filename="$(find irl_common_description)/urdf/az3_wheel_group/wheel.gazebo.xacro" />
 	<include filename="$(find irl_common_description)/urdf/az3_wheel_group/wheel.transmission.xacro" />
-	<!-- Distance between base and linkWheel -->
-	<property name="dX0" value="0.18194605" />
-	<property name="dY0" value="0.18194605" />
-	<property name="dZ0" value="-0.06282066" />
-	<!-- Distance between linkWheel and prop wheel joint -->
-	<property name="dX1" value="0.08748000" />
-	<!-- Properties of the link between the base and the wheel -->
-	<property name="linkWheel_mass" value="0.935764" />
-	<property name="linkWheel_cg_x" value="0.048556" />
-	<property name="linkWheel_cg_y" value="0.000041" />
-	<property name="linkWheel_cg_z" value="0.014578" />
-	<property name="linkWheel_ixx" value="0.001359" />
-	<property name="linkWheel_ixy" value="0.000002" />
-	<property name="linkWheel_ixz" value="0.000154" />
-	<property name="linkWheel_iyy" value="0.004142" />
-	<property name="linkWheel_iyz" value="0.000001" />
-	<property name="linkWheel_izz" value="0.003414" />
-	<!-- Properties of the link between the wheel -->
-	<property name="wheel_mass" value="0.940025" />
-	<property name="wheel_cg_x" value="0.006637" />
-	<property name="wheel_cg_y" value="0.000000" />
-	<property name="wheel_cg_z" value="-0.000004" />
-	<property name="wheel_ixx" value="0.002007" />
-	<property name="wheel_ixy" value="0.000000" />
-	<property name="wheel_ixz" value="0.000000" />
-	<property name="wheel_iyy" value="0.001169" />
-	<property name="wheel_iyz" value="0.000000" />
-	<property name="wheel_izz" value="0.001169" />
 	<xacro:macro name="az3_wheel_group" params="side reflectSide face reflectFace parent">
 		<joint name="wheel${side}${face}_revolute_joint" type="revolute">

Commit message: Refs #171. A few fixes to the AZ2 and AZ3 description.
git-svn-id: svn+ssh://marvin.3it.usherbrooke.ca/svn/introlab/johnny0/svn/branches/AzMC/ros-pkgs/irl_robots/irl_common_description@1215 23a761d4-b60a-4777-9503-f06a07968eac

File: urdf/az3_base/base.urdf.xacro (robot description, xacro)
@@ -31,5 +31,5 @@
 		</link>
 		<joint name="${name}_footprint_joint" type="fixed">
-		  <origin xyz="0 0 0.251" rpy="0 0 0" />
+		  <origin xyz="0 0 ${base_footprint_height}" rpy="0 0 0" />
 		  <child link="${name}_link" />
 		  <parent link="${name}_footprint"/>
