Commit message: Refs #171. A few fixes to the AZ3 URDF: direction joint position and velocity limits.
git-svn-id: svn+ssh://marvin.3it.usherbrooke.ca/svn/introlab/johnny0/svn/branches/AzMC/ros-pkgs/irl_robots/irl_common_description@1202 23a761d4-b60a-4777-9503-f06a07968eac

File: urdf/az3_wheel_group/wheel.urdf.xacro (robot description, xacro)
@@ -11,5 +11,5 @@
 	<property name="dY0" value="0.18194605" />
 	<property name="dZ0" value="-0.06282066" />
-	<!-- Distance between base and linkWheel -->
+	<!-- Distance between linkWheel and prop wheel joint -->
 	<property name="dX1" value="0.08748000" />
 	<!-- Properties of the link between the base and the wheel -->
@@ -41,5 +41,5 @@
 			<origin xyz="${reflectFace*dX0} ${reflectSide*dY0} ${dZ0}" rpy="0 0 ${reflectSide*(M_PI/4+(1-reflectFace)*M_PI/4)}" />
 			<axis xyz="0 0 1" rpy="0 0 0"/>
-			<limit effort="100" velocity="0.1" lower="-0.7854" upper="0.7854" />
+			<limit effort="100" velocity="1.7442" lower="-1.5708" upper="1.5708" />
 		</joint>
 		<link name="wheel${side}${face}_linkWheel_link">

Commit message: Refs #171. Configurable wheel size for az3_wheel_group. The wheels do not have the exact same diameter, actually. The collision model will fit the actual wheel size, but the mesh might appear to be floating. We could also calculate the scaling factor of the mesh, but it might clash with the suspension link rendering.
git-svn-id: svn+ssh://marvin.3it.usherbrooke.ca/svn/introlab/johnny0/svn/branches/AzMC/ros-pkgs/irl_robots/irl_common_description@1210 23a761d4-b60a-4777-9503-f06a07968eac

File: urdf/az3_wheel_group/wheel.urdf.xacro (robot description, xacro)
@@ -55,7 +55,7 @@
 			</visual>
 			<collision name="wheel${side}${face}_wheel_collision">
-				<origin xyz="0 0 0" rpy="0 0 0" />
+				<origin xyz="0 0 0" rpy="0 ${M_PI/2} 0" />
 				<geometry name="wheel${side}${face}_wheel_collision_geom">
-					<mesh filename="package://irl_common_description/meshes/az3_wheel_group/wheel.stl"  />
+                    <cylinder radius="${wheel_diameter/2}" length="${wheel_width}"/>
 				</geometry>
 			</collision>

Commit message: Refs #169, #171. (ROS) Modified direction limits to avoid interference with MC constraints handling.
git-svn-id: svn+ssh://marvin.3it.usherbrooke.ca/svn/introlab/johnny0/svn/branches/AzMC/ros-pkgs/irl_robots/irl_common_description@1231 23a761d4-b60a-4777-9503-f06a07968eac

File: urdf/az3_wheel_group/wheel.urdf.xacro (robot description, xacro)
@@ -13,5 +13,5 @@
 			<origin xyz="${reflectFace*dX0} ${reflectSide*dY0} ${dZ0}" rpy="0 0 ${reflectSide*(M_PI/4+(1-reflectFace)*M_PI/4)}" />
 			<axis xyz="0 0 1" rpy="0 0 0"/>
-			<limit effort="100" velocity="1.7442" lower="-1.5708" upper="1.5708" />
+			<limit effort="100" velocity="1.8" lower="${-M_PI/2-0.1}" upper="${M_PI/2+0.1}" />
 		</joint>
 		<link name="wheel${side}${face}_linkWheel_link">
