Commit message: Refs #330. IMU message publication and URDF integration for IRL-1.
git-svn-id: svn+ssh://marvin.3it.usherbrooke.ca/svn/introlab/johnny0/svn/trunk/ros-pkgs/irl_robots/irl_common_description@2552 23a761d4-b60a-4777-9503-f06a07968eac

File: urdf/jn0_torso/box_torso.urdf.xacro (robot description, xacro)
@@ -61,4 +61,18 @@
             </collision>
         </link>
+        <!-- IMU attached to the frame -->
+        <joint name="${name}_imu_fixed" type="fixed">
+            <parent link="${name}_top_frame"/>
+            <child link="${name}_imu_link"/>
+            <origin xyz="0.065 0.0 -0.12" rpy="0 0 -${M_PI/2}"/>
+        </joint>
+        <link name="${name}_imu_link">
+            <visual>
+                <origin xyz="0 0 0" rpy="0 0 0"/>
+                <geometry>
+                    <box size="0.02 0.02 0.02"/>
+                </geometry>
+            </visual>
+        </link>
 	</xacro:macro>
 </robot>
