Commit message: Refs #176. Importing head and torso meshes/urdf from Arnaud
git-svn-id: svn+ssh://marvin.3it.usherbrooke.ca/svn/introlab/johnny0/svn/branches/M9/ros-pkgs/irl_robots/irl_common_description@1282 23a761d4-b60a-4777-9503-f06a07968eac

File: urdf/common_geometry.xacro (robot description, xacro)
@@ -13,5 +13,6 @@
 			<inertia
 				ixx="0.001" ixy="0.0" ixz="0.0"
-				iyy="0.001" iyz="0.0" izz="0.001" />
+				iyy="0.001" iyz="0.0"
+				izz="0.001" />
 			</inertial>
 	</xacro:macro>
@@ -28,10 +29,11 @@
 		</material>
 	</xacro:macro>
-	<xacro:macro name="simple_box" params="name lwh xyz rpy mass rviz_rgba material">
+	<!-- Generic shape -->
+	<xacro:macro name="simple_shape" params="name xyz rpy mass rviz_rgba material *shape">
 		<link name="${name}">
 			<visual>
 				<origin xyz="${xyz}" rpy="${rpy}" />
 				<geometry>
-					<box size="${lwh}" />
+					<xacro:insert_block name="shape" />
 				</geometry>
 				<material name="${name}_color">
@@ -42,5 +44,5 @@
 				<origin xyz="${xyz}" rpy="${rpy}" />
 				<geometry>
-					<box size="${lwh}" />
+					<xacro:insert_block name="shape" />
 				</geometry>
 			</collision>
@@ -49,3 +51,25 @@
 		<xacro:simple_gazebo name="${name}" material="${material}" />
 	</xacro:macro>
+	<!-- Shapes specializations -->
+	<xacro:macro name="simple_box" params="lwh name xyz rpy mass rviz_rgba material">
+		<xacro:simple_shape
+			name="${name}" xyz="${xyz}" rpy="${rpy}"
+			mass="${mass}" rviz_rgba="${rviz_rgba}" material="${material}">
+			<box size="${lwh}" />
+		</xacro:simple_shape>
+	</xacro:macro>
+	<xacro:macro name="simple_cylinder" params="radius length name xyz rpy mass rviz_rgba material">
+		<xacro:simple_shape
+			name="${name}" xyz="${xyz}" rpy="${rpy}"
+			mass="${mass}" rviz_rgba="${rviz_rgba}" material="${material}">
+			<cylinder radius="${radius}" length="${length}" />
+		</xacro:simple_shape>
+	</xacro:macro>
+	<xacro:macro name="simple_sphere" params="radius name xyz rpy mass rviz_rgba material">
+		<xacro:simple_shape
+			name="${name}" xyz="${xyz}" rpy="${rpy}"
+			mass="${mass}" rviz_rgba="${rviz_rgba}" material="${material}">
+			<sphere radius="${radius}" />
+		</xacro:simple_shape>
+	</xacro:macro>
 </robot>

File: urdf/jn0_head/head.transmission.xacro (robot description, xacro)
@@ -6,5 +6,5 @@
   <!-- ============================   Head   ============================ -->
   <!-- Head pan (or yaw) -->
-  <xacro:macro name="jn0_head_pan_transmission" >
+  <!--xacro:macro name="johnny_0_head_pan_transmission" >
     <transmission type="pr2_mechanism_model/SimpleTransmission" name="head_pan_trans">
       <actuator name="head_pan_motor" />
@@ -12,7 +12,7 @@
       <mechanicalReduction>6.0</mechanicalReduction>
     </transmission>
-  </xacro:macro>
+  </xacro:macro-->
   <!-- Head tilt (or roll) -->
-  <xacro:macro name="jn0_head_tilt_transmission" >
+  <!--xacro:macro name="johnny_0_head_tilt_transmission" >
     <transmission type="pr2_mechanism_model/SimpleTransmission" name="head_tilt_trans">
       <actuator name="head_tilt_motor" />
@@ -20,4 +20,4 @@
       <mechanicalReduction>6.0</mechanicalReduction>
     </transmission>
-  </xacro:macro>
+  </xacro:macro-->
 </robot>

File: urdf/jn0_head/head.urdf.xacro (robot description, xacro)
@@ -5,126 +5,308 @@
        xmlns:xacro="http://ros.org/wiki/xacro">
 	<include filename="$(find irl_common_description)/urdf/jn0_head/head.transmission.xacro" />
-	<property name="pan_size_z" value="0.05" />
-	<property name="head_size_z" value="0.17" />
-	<xacro:macro name="head" params="name parent *origin">
+	<xacro:macro name="jn0_head" params="name parent">
 		<joint name="${name}_fixed_joint" type="fixed">
 			<parent link="${parent}"/>
-			<child link="${name}_pan_link"/>
-			<insert_block name="origin" />
+			<child link="${name}_link"/>
 			<!--origin xyz="0.02 0 0.2228115" rpy="0 0 0" /-->
-		</joint>
-		<link name="${name}_pan_link">
+			<origin xyz="-0.02 0.03 0.545" rpy="0 0 0" />
+		</joint>
+		<link name="${name}_link">
+			<inertial>
+				<mass value="0.2" />
+				<origin xyz="0 0 0" />
+				<inertia ixx="0" ixy="0" ixz="0"
+						 iyy="0" iyz="0" izz="0" />
+			</inertial>
+			<visual name="${name}_visual">
+				<origin xyz="0 0 0" rpy="0 0 -${M_PI/2}" />
+				<!--origin xyz="0 0 0" rpy="0 0 0" /-->
+				<geometry name="${name}_visual_geom">
+					<!--box size="0.04 0.04 0.066413" /-->
+					<mesh filename="package://irl_common_description/meshes/jn0_head/neckTilt.dae"  />
+				</geometry>
+			</visual>
+			<collision name="${name}_collision">
+				<origin xyz="0 0 0" rpy="0 0 -${M_PI/2}" />
+				<geometry name="${name}_collision_geom">
+					<!--box size="0.04 0.04 0.066413" /-->
+					<mesh filename="package://irl_common_description/meshes/jn0_head/neckTilt.STL"  />
+				</geometry>
+			</collision>
+		</link>
+		<joint name="${name}_tilt_joint" type="revolute">
+			<parent link="${name}_link"/>
+			<child link="${name}_head_link_tmp"/>
+			<!--origin xyz="-0.02 0 0.0966715" rpy="0 0 0" /-->
+			<origin xyz="0 -0.014 0.045" rpy="0 0 -${M_PI/2}" />
+			<axis xyz="0 0 1" rpy="0 0 0"/>
+			<limit effort="100" velocity="0.1" lower="-0.7" upper="0.7" />
+		</joint>
+		<link name="${name}_head_link_tmp">
+			<inertial>
+				<mass value="0.001" />
+				<origin xyz="0 0 0" />
+				<inertia ixx="0" ixy="0" ixz="0"
+						 iyy="0" iyz="0" izz="0" />
+			</inertial>
+			<visual name="${name}_head_tmp_visual">
+				<origin xyz="0 0 0" rpy="0 0 0" />
+				<geometry name="${name}_head_tmp_visual_geom">
+					<mesh filename="package://irl_common_description/meshes/jn0_head/neckpan.dae"  />
+					<!--sphere radius="0.001" /-->
+				</geometry>
+			</visual>
+			<collision name="${name}_head_tmp_collision">
+				<origin xyz="0 0 0" rpy="0 0 0" />
+				<geometry name="${name}_head_tmp_collision_geom">
+					<mesh filename="package://irl_common_description/meshes/jn0_head/neckpan.STL"  />
+				</geometry>
+			</collision>
+		</link>
+		<!--joint name="${name}_pan_joint" type="revolute"-->
+		<joint name="${name}_pan_joint" type="fixed">
+			<parent link="${name}_head_link_tmp"/>
+			<child link="${name}_head_link_tmp2"/>
+			<origin xyz="-0.01 0.08 0.04" rpy="${M_PI/2} 0 0" />
+			<!--axis xyz="1 0 0" rpy="0 0 0"/-->
+			<!--limit effort="100" velocity="0.1" lower="-0.7854" upper="0.7854" /-->
+		</joint>
+		<link name="${name}_head_link_tmp2">
+			<inertial>
+				<mass value="0.001" />
+				<origin xyz="0 0 0" />
+				<inertia ixx="0" ixy="0" ixz="0"
+						 iyy="0" iyz="0" izz="0" />
+			</inertial>
+			<visual name="${name}_head_tmp2_visual">
+				<origin xyz="0 0 0" rpy="0 0 0" />
+				<geometry name="${name}_head_tmp2_visual_geom">
+					<mesh filename="package://irl_common_description/meshes/jn0_head/panBraket.dae"  />
+					<!--sphere radius="0.001" /-->
+				</geometry>
+			</visual>
+			<collision name="${name}_head_tmp2_collision">
+				<origin xyz="0 0 0" rpy="0 0 0" />
+				<geometry name="${name}_head_tmp2_collision_geom">
+					<mesh filename="package://irl_common_description/meshes/jn0_head/panBraket.STL"  />
+				</geometry>
+			</collision>
+		</link>
+		<joint name="${name}_fixed_joint_head" type="fixed">
+			<parent link="${name}_head_link_tmp2"/>
+			<child link="${name}_head_link"/>
+			<origin xyz="0.03 0.15 0" rpy="0 ${M_PI} 0" />
+		</joint>
+		<link name="${name}_head_link">
 			<inertial>
 				<mass value="0.5" />
-				<origin xyz="0 0 ${pan_size_z/2}" />
-				<inertia ixx="0" ixy="0" ixz="0"
-						 iyy="0" iyz="0" izz="0" />
-			</inertial>
-			<visual name="${name}_pan_visual">
-				<origin xyz="0 0 ${pan_size_z/2}" rpy="0 0 0" />
-				<geometry name="${name}_pan_visual_geom">
-					<box size="0.04 0.04 ${pan_size_z}" />
-				</geometry>
-			</visual>
-			<collision name="${name}_pan_collision">
-				<origin xyz="0 0 ${pan_size_z/2}" rpy="0 0 0" />
-				<geometry name="${name}_pan_collision_geom">
-					<box size="0.04 0.04 ${pan_size_z}" />
-				</geometry>
-			</collision>
-		</link>
-		<joint name="${name}_pan_joint" type="revolute">
-			<parent link="${name}_pan_link"/>
-			<child link="${name}_tilt_link"/>
-			<origin xyz="0 0 ${pan_size_z}" rpy="0 0 0" />
-			<axis xyz="0 0 1" rpy="0 0 0"/>
-			<limit effort="100" velocity="0.1" lower="-0.7854" upper="0.7854" />
-			<!-- calibration reference_position="0.0"/ -->
-		</joint>
-		<link name="${name}_tilt_link">
-			<inertial>
-				<mass value="0.001" />
-				<origin xyz="0 0 0.023" />
-				<inertia ixx="0" ixy="0" ixz="0"
-						 iyy="0" iyz="0" izz="0" />
-			</inertial>
-			<visual name="${name}_tilt_visual">
-				<origin xyz="0 0 0.023" rpy="0 0 0" />
-				<geometry name="${name}_tilt_visual_geom">
-					<box size="0.04 0.04 0.046" />
-				</geometry>
-			</visual>
-			<collision name="${name}_tilt_collision">
-				<origin xyz="0 0 0.023" rpy="0 0 0" />
-				<geometry name="${name}_tilt_collision_geom">
-					<box size="0.04 0.04 0.046" />
-				</geometry>
-			</collision>
-		</link>
-		<joint name="${name}_tilt_joint" type="revolute">
-			<parent link="${name}_tilt_link"/>
-			<child link="${name}_neck_link"/>
-			<!-- distance between tilt axis and beginning of the head plus the half of the head height-->
-			<origin xyz="0 0 0.046" rpy="0 0 0" />
-			<axis xyz="0 1 0" rpy="0 0 0"/>
-			<limit effort="100" velocity="0.1" lower="-0.7" upper="0.7" />
-			<!-- calibration reference_position="0.0"/ -->
-		</joint>
-		<link name="${name}_neck_link">
-			<inertial>
-				<mass value="0.001" />
-				<origin xyz="0 0 0.04" />
-				<inertia ixx="0" ixy="0" ixz="0"
-						 iyy="0" iyz="0" izz="0" />
-			</inertial>
-			<visual name="${name}_neck_visual">
-				<origin xyz="0 0 0.04" rpy="0 0 0" />
-				<geometry name="${name}_neck_visual_geom">
-					<box size="0.04 0.04 0.08" />
-				</geometry>
-			</visual>
-			<collision name="${name}_neck_collision">
-				<origin xyz="0 0 0.04" rpy="0 0 0" />
-				<geometry name="${name}_neck_collision_geom">
-					<box size="0.04 0.04 0.08" />
-				</geometry>
-			</collision>
-		</link>
-		<joint name="${name}_neck_joint" type="fixed">
-			<parent link="${name}_neck_link"/>
-			<child link="${name}_head_link"/>
-			<!-- distance between tilt axis and beginning of the head plus the half of the head height-->
-			<origin xyz="0 0 ${0.06 + head_size_z/2}" rpy="0 0 0" />
-			<!-- calibration reference_position="0.0"/ -->
-		</joint>
-		<link name="${name}_head_link">
-			<inertial>
-				<mass value="0.5" />
-				<origin xyz="0 0 0" />
+				<origin xyz="0 0 0" rpy="0 0 0" />
 				<inertia ixx="0" ixy="0" ixz="0"
 						 iyy="0" iyz="0" izz="0" />
 			</inertial>
 			<visual name="${name}_head_visual">
+				<!--origin xyz="0.03 0 0.03" rpy="${M_PI/2} 0 ${M_PI/2}" /-->
 				<origin xyz="0 0 0" rpy="0 0 0" />
 				<geometry name="${name}_head_visual_geom">
-					<box size="0.17 0.19 ${head_size_z}" />
+					<mesh filename="package://irl_common_description/meshes/jn0_head/head.dae"  />
+					<!--box size="0.16268 0.17418 0.12693" /-->
 				</geometry>
 			</visual>
 			<collision name="${name}_head_collision">
+				<!--origin xyz="0.03 0 0.03" rpy="${M_PI/2} 0 ${M_PI/2}" /-->
 				<origin xyz="0 0 0" rpy="0 0 0" />
 				<geometry name="${name}_head_collision_geom">
-					<box size="0.17 0.19 ${head_size_z}" />
+					<mesh filename="package://irl_common_description/meshes/jn0_head/head.STL"  />
+					<!--box size="0.16268 0.17418 0.12693" /-->
+				</geometry>
+			</collision>
+		</link>
+		<!--joint name="${name}_right_eye" type="revolute"-->
+		<joint name="${name}_right_eye" type="fixed">
+			<parent link="${name}_head_link"/>
+			<child link="${name}_right_eye_link"/>
+			<origin xyz="0.02 -0.01 0.02" rpy="0 0 0" />
+			<!--axis xyz="1 0 0" rpy="0 0 0"/-->
+			<!--limit effort="100" velocity="0.1" lower="-0.7854" upper="0.7854" /-->
+		</joint>
+		<link name="${name}_right_eye_link">
+			<inertial>
+				<mass value="0.001" />
+				<origin xyz="0 0 0" />
+				<inertia ixx="0" ixy="0" ixz="0"
+						 iyy="0" iyz="0" izz="0" />
+			</inertial>
+			<visual name="${name}_right_eye_visual">
+				<origin xyz="0 0 0" rpy="0 0 0" />
+				<geometry name="${name}_right_eye_visual_geom">
+					<mesh filename="package://irl_common_description/meshes/jn0_head/eye.dae"  />
+					<!--sphere radius="0.001" /-->
+				</geometry>
+			</visual>
+			<collision name="${name}_right_eye_collision">
+				<origin xyz="0 0 0" rpy="0 0 0" />
+				<geometry name="${name}_right_eye_collision_geom">
+					<mesh filename="package://irl_common_description/meshes/jn0_head/eye.STL"  />
+				</geometry>
+			</collision>
+		</link>
+		<joint name="${name}_right_black_eye" type="fixed">
+			<parent link="${name}_right_eye_link"/>
+			<child link="${name}_right_black_eye_link"/>
+			<origin xyz="0.02 0.02 0.02" rpy="0 0 0" />
+		</joint>
+		<link name="${name}_right_black_eye_link">
+			<inertial>
+				<mass value="0.001" />
+				<origin xyz="0 0 0" />
+				<inertia ixx="0" ixy="0" ixz="0"
+						 iyy="0" iyz="0" izz="0" />
+			</inertial>
+			<visual name="${name}_right_black_eye_visual">
+				<origin xyz="0 0 0" rpy="0 0 0" />
+				<geometry name="${name}_right_black_eye_visual_geom">
+					<cylinder radius="0.01" length="0.01"/>
+				</geometry>
+			</visual>
+			<collision name="${name}_right_black_eye_collision">
+				<origin xyz="0 0 0" rpy="0 0 0" />
+				<geometry name="${name}_right_black_eye_collision_geom">
+					<cylinder radius="0.05" length="0.05"/>
+				</geometry>
+			</collision>
+		</link>
+		<!--joint name="${name}_left_eye" type="revolute"-->
+		<joint name="${name}_left_eye" type="fixed">
+			<parent link="${name}_head_link"/>
+			<child link="${name}_left_eye_link"/>
+			<origin xyz="-0.06 -0.01 0.02" rpy="0 0 0" />
+			<!--axis xyz="1 0 0" rpy="0 0 0"/-->
+			<!--limit effort="100" velocity="0.1" lower="-0.7854" upper="0.7854" /-->
+		</joint>
+		<link name="${name}_left_eye_link">
+			<inertial>
+				<mass value="0.001" />
+				<origin xyz="0 0 0" />
+				<inertia ixx="0" ixy="0" ixz="0"
+						 iyy="0" iyz="0" izz="0" />
+			</inertial>
+			<visual name="${name}_left_eye_visual">
+				<origin xyz="0 0 0" rpy="0 0 0" />
+				<geometry name="${name}_right_eye_visual_geom">
+					<mesh filename="package://irl_common_description/meshes/jn0_head/eye.dae"  />
+					<!--sphere radius="0.001" /-->
+				</geometry>
+			</visual>
+			<collision name="${name}_left_eye_collision">
+				<origin xyz="0 0 0" rpy="0 0 0" />
+				<geometry name="${name}_right_eye_collision_geom">
+					<mesh filename="package://irl_common_description/meshes/jn0_head/eye.STL"  />
+				</geometry>
+			</collision>
+		</link>
+		<joint name="${name}_left_black_eye" type="fixed">
+			<parent link="${name}_left_eye_link"/>
+			<child link="${name}_left_black_eye_link"/>
+			<origin xyz="0.02 0.02 0.02" rpy="0 0 0" />
+		</joint>
+		<link name="${name}_left_black_eye_link">
+			<inertial>
+				<mass value="0.001" />
+				<origin xyz="0 0 0" />
+				<inertia ixx="0" ixy="0" ixz="0"
+						 iyy="0" iyz="0" izz="0" />
+			</inertial>
+			<visual name="${name}_left_black_eye_visual">
+				<origin xyz="0 0 0" rpy="0 0 0" />
+				<geometry name="${name}_left_black_eye_visual_geom">
+					<cylinder radius="0.01" length="0.01"/>
+				</geometry>
+			</visual>
+			<collision name="${name}_left_black_eye_collision">
+				<origin xyz="0 0 0" rpy="0 0 0" />
+				<geometry name="${name}_left_black_eye_collision_geom">
+					<cylinder radius="0.05" length="0.05"/>
+				</geometry>
+			</collision>
+		</link>
+		<!--joint name="${name}_left_eyebrow" type="revolute"-->
+		<joint name="${name}_left_eyebrow" type="fixed">
+			<parent link="${name}_head_link"/>
+			<child link="${name}_left_eyebrow_link"/>
+			<origin xyz="-0.07 0.035 0.045" rpy="0 0 0" />
+			<!--axis xyz="1 0 0" rpy="0 0 0"/-->
+			<!--limit effort="100" velocity="0.1" lower="-0.7854" upper="0.7854" /-->
+		</joint>
+		<link name="${name}_left_eyebrow_link">
+			<inertial>
+				<mass value="0.001" />
+				<origin xyz="0 0 0" />
+				<inertia ixx="0" ixy="0" ixz="0"
+						 iyy="0" iyz="0" izz="0" />
+			</inertial>
+			<visual name="${name}_left_eyebrow_visual">
+				<origin xyz="0 0 0" rpy="0 0 0" />
+				<geometry name="${name}_left_eyebrow_visual_geom">
+					<mesh filename="package://irl_common_description/meshes/jn0_head/eyebrow.dae"  />
+					<!--sphere radius="0.001" /-->
+				</geometry>
+			</visual>
+			<collision name="${name}_left_eyebrow_collision">
+				<origin xyz="0 0 0" rpy="0 0 0" />
+				<geometry name="${name}_left_eyebrow_collision_geom">
+					<mesh filename="package://irl_common_description/meshes/jn0_head/eyebrow.STL"  />
+				</geometry>
+			</collision>
+		</link>
+		<!--joint name="${name}_right_eyebrow" type="revolute"-->
+		<joint name="${name}_right_eyebrow" type="fixed">
+			<parent link="${name}_head_link"/>
+			<child link="${name}_right_eyebrow_link"/>
+			<origin xyz="0.07 0.035 0.045" rpy="0 0 0" />
+			<!--axis xyz="1 0 0" rpy="0 0 0"/-->
+			<!--limit effort="100" velocity="0.1" lower="-0.7854" upper="0.7854" /-->
+		</joint>
+		<link name="${name}_right_eyebrow_link">
+			<inertial>
+				<mass value="0.001" />
+				<origin xyz="0 0 0" />
+				<inertia ixx="0" ixy="0" ixz="0"
+						 iyy="0" iyz="0" izz="0" />
+			</inertial>
+			<visual name="${name}_right_eyebrow_visual">
+				<origin xyz="0 0 0" rpy="0 ${M_PI} 0" />
+				<geometry name="${name}_right_eyebrow_visual_geom">
+					<mesh filename="package://irl_common_description/meshes/jn0_head/eyebrow.dae"  />
+					<!--sphere radius="0.001" /-->
+				</geometry>
+			</visual>
+			<collision name="${name}_right_eyebrow_collision">
+				<origin xyz="0 0 0" rpy="0 ${M_PI} 0" />
+				<geometry name="${name}_right_eyebrow_collision_geom">
+					<mesh filename="package://irl_common_description/meshes/jn0_head/eyebrow.STL"  />
 				</geometry>
 			</collision>
 		</link>
 		<!-- extansions -->
-		<xacro:jn0_head_tilt_transmission />
-		<xacro:jn0_head_pan_transmission />
-		<gazebo reference="${name}_link">
+		<xacro:johnny_0_head_tilt_transmission />
+		<xacro:johnny_0_head_pan_transmission />
+		<gazebo reference="${name}_right_black_eye_link">
+			<material>Gazebo/Black</material>
+		</gazebo>
+		<gazebo reference="${name}_left_black_eye_link">
+			<material>Gazebo/Black</material>
+		</gazebo>
+		<gazebo reference="${name}_right_eyebrow_link">
+			<material>Gazebo/Black</material>
+		</gazebo>
+		<gazebo reference="${name}_left_eyebrow_link">
+			<material>Gazebo/Black</material>
+		</gazebo>
+		<!--gazebo reference="${name}_link">
 			<material>Gazebo/Green</material>
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
File: urdf/jn0_torso/box_torso.urdf.xacro (robot description, xacro)
@@ -5,5 +5,5 @@
        xmlns:xacro="http://ros.org/wiki/xacro">
 	<include filename="$(find irl_common_description)/urdf/common_geometry.xacro" />
-	<xacro:macro name="jn0_torso_box" params="name parent xyz stand_width stand_height chest_width chest_height chest_length">
+	<xacro:macro name="box_torso" params="name parent xyz height stand_width chest_width chest_height chest_length">
 		<!-- "Stand", the bar supporting the torso -->
 		<joint name="${name}_stand_fixed_joint" type="fixed">
@@ -14,6 +14,6 @@
 		<xacro:simple_box
 			name = "${name}_stand_link"
-			lwh  = "${stand_width} ${stand_width} ${stand_height}"
-			xyz  = "0 0 0"
+			lwh  = "${stand_width} ${stand_width} ${height - chest_height}"
+			xyz  = "0 0 ${(height - chest_height) / 2}"
 			rpy  = "0 0 0"
 			mass = "0.5"
@@ -22,7 +22,7 @@
 		/>
 		<joint name="${name}_fixed_joint" type="fixed">
-			<parent link="${name}_stand_link"/>
+			<parent link="${parent}"/>
 			<child link="${name}_link"/>
-			<origin xyz="0 0 ${stand_height}" rpy="0 0 0" />
+			<origin xyz="${xyz}" rpy="0 0 0" />
 		</joint>
 		<!-- Actual torso represented by a box -->
@@ -30,5 +30,5 @@
 			name = "${name}_link"
 			lwh  = "${chest_length} ${chest_width} ${chest_height}"
-			xyz  = "0 0 0"
+			xyz  = "0 0 ${height - chest_height/2}"
 			rpy  = "0 0 0"
 			mass = "0.5"

File: urdf/reddy_arm/arm.transmission.xacro (robot description, xacro)
@@ -4,26 +4,25 @@
        xmlns:interface="http://playerstage.sourceforge.net/gazebo/xmlschema/#interface"
        xmlns:xacro="http://ros.org/wiki/xacro">
-  <!-- ============================   Arm   ============================ -->
   <!-- ADE roll shoulder -->
-  <xacro:macro name="jn0_ADE_roll_shoulder_transmission" params="side" >
-    <transmission type="pr2_mechanism_model/SimpleTransmission" name="${side}_ADE_roll_shoulder_trans">
-      <actuator name="${side}_ADE_roll_shoulder_motor" />
-      <joint name="ADE_roll${side}_revolute_joint" />
+  <xacro:macro name="reddy_arm_shoulder_roll_transmission" params="name" >
+      <transmission type="pr2_mechanism_model/SimpleTransmission" name="${name}">
+      <actuator name="${name}_motor" />
+      <joint name="${name}_revolute_joint" />
       <mechanicalReduction>1.0</mechanicalReduction>
     </transmission>
   </xacro:macro>
   <!-- ADE pitch shoulder -->
-  <xacro:macro name="jn0_ADE_pitch_shoulder_transmission" params="side" >
-    <transmission type="pr2_mechanism_model/SimpleTransmission" name="${side}_ADE_pitch_shoulder_trans">
-      <actuator name="${side}_ADE_pitch_shoulder_motor" />
-      <joint name="ADE_pitch_shoulder${side}_revolute_joint" />
+  <xacro:macro name="reddy_arm_shoulder_pitch_transmission" params="name" >
+    <transmission type="pr2_mechanism_model/SimpleTransmission" name="${name}">
+      <actuator name="${name}_motor" />
+      <joint name="${name}_revolute_joint" />
       <mechanicalReduction>1.0</mechanicalReduction>
     </transmission>
   </xacro:macro>
   <!--  ADE pitch elbow -->
-  <xacro:macro name="jn0_ADE_pitch_elbow_transmission" params="side" >
-    <transmission type="pr2_mechanism_model/SimpleTransmission" name="${side}_ADE_pitch_elbow_trans">
-      <actuator name="${side}_ADE_pitch_elbow_motor" />
-      <joint name="ADE_pitch_elbow${side}_revolute_joint" />
+  <xacro:macro name="reddy_arm_elbow_pitch_transmission" params="name" >
+    <transmission type="pr2_mechanism_model/SimpleTransmission" name="${name}">
+      <actuator name="${name}_motor" />
+      <joint name="${name}_revolute_joint" />
       <mechanicalReduction>1.0</mechanicalReduction>
     </transmission>
