Commit message: Refs #176. Importing head and torso meshes/urdf from Arnaud
git-svn-id: svn+ssh://marvin.3it.usherbrooke.ca/svn/introlab/johnny0/svn/branches/M9/ros-pkgs/irl_robots/irl_common_description@1282 23a761d4-b60a-4777-9503-f06a07968eac

File: urdf/reddy_arm/arm.urdf.xacro (robot description, xacro)
@@ -5,15 +5,37 @@
        xmlns:xacro="http://playerstage.sourceforge.net/gazebo/xmlschema/#interface"
        name="arm">
-	<include filename="$(find irl_common_description)/urdf/reddy_arm/ADE_roll/ADE_roll.urdf.xacro" />
-	<include filename="$(find irl_common_description)/urdf/reddy_arm/ADE_pitch_shoulder/ADE_pitch_shoulder.urdf.xacro" />
-	<include filename="$(find irl_common_description)/urdf/reddy_arm/ADE_pitch_elbow/ADE_pitch_elbow.urdf.xacro" />
-	<include filename="$(find irl_common_description)/urdf/reddy_arm/forearm/forearm.urdf.xacro" />
-	<include filename="$(find irl_common_description)/urdf/reddy_arm/hand/hand.urdf.xacro" />
-	<xacro:macro name="reddy_arm" params="side reflect parent">
-		<xacro:ADE_roll side="${side}" reflect="${reflect}" parent="${parent}"/>
-		<xacro:ADE_pitch_shoulder side="${side}" reflect="${reflect}" parent="ADE_roll${side}_link"/>
-		<xacro:ADE_pitch_elbow side="${side}" reflect="${reflect}" parent="ADE_pitch_shoulder${side}_box"/>
-		<xacro:forearm side="${side}" reflect="${reflect}" parent="ADE_pitch_elbow${side}_link"/>
-		<xacro:hand side="${side}" reflect="${reflect}" parent="forearm${side}"/>
+	<include filename="$(find irl_common_description)/urdf/reddy_arm/shoulder_roll.urdf.xacro" />
+	<include filename="$(find irl_common_description)/urdf/reddy_arm/shoulder_pitch.urdf.xacro" />
+	<include filename="$(find irl_common_description)/urdf/reddy_arm/elbow_pitch.urdf.xacro" />
+	<include filename="$(find irl_common_description)/urdf/reddy_arm/forearm.urdf.xacro" />
+	<include filename="$(find irl_common_description)/urdf/reddy_arm/hand.urdf.xacro" />
+	<xacro:macro name="reddy_arm" params="name reflect parent offset_y offset_z">
+		<xacro:reddy_arm_shoulder_roll
+			name="${name}_shoulder_roll"
+			reflect="${reflect}"
+			parent="${parent}"
+			offset_y="${offset_y}"
+			offset_z="${offset_z - 0.09}"
+			/>
+		<xacro:reddy_arm_shoulder_pitch
+			name="${name}_shoulder_pitch"
+			reflect="${reflect}"
+			parent="${name}_shoulder_roll_link"
+			/>
+		<xacro:reddy_arm_elbow_pitch
+			name="${name}_elbow_pitch"
+			reflect="${reflect}"
+			parent="${name}_shoulder_pitch_box"
+			/>
+		<xacro:forearm
+			name="${name}_forearm"
+			reflect="${reflect}"
+			parent="${name}_elbow_pitch_link"
+			/>
+		<xacro:hand
+			name="${name}_hand"
+			reflect="${reflect}"
+			parent="${name}_forearm"
+			/>
 	</xacro:macro>
 </robot>

File: urdf/reddy_arm/elbow_pitch.urdf.xacro (robot description, xacro)
@@ -5,6 +5,6 @@
        xmlns:xacro="http://ros.org/wiki/xacro">
 	<include filename="$(find irl_common_description)/urdf/reddy_arm/arm.transmission.xacro" />
-	<xacro:macro name="ADE_pitch_elbow" params="side reflect parent">
-		<link name="ADE_pitch_elbow${side}_box">
+	<xacro:macro name="reddy_arm_elbow_pitch" params="name reflect parent">
+		<link name="${name}_box">
 			<inertial>
 				<mass value="1.105" />
@@ -16,16 +16,19 @@
 			<visual>
 				<origin xyz="0 0 0" rpy="0 0 0" />
-				<geometry name="ADE_pitch_elbow${side}_box_visual_geom">
+				<geometry name="${name}_box_visual_geom">
 					<box size="0.088678 0.084137 0.1524" />
 				</geometry>
+				<material name="${name}_color">
+					<color rgba="0 0 1 1"/>
+				</material>
 			</visual>
 			<collision>
 				<origin xyz="0 0 0" rpy="0 0 0 " />
-				<geometry name="ADE_pitch_elbow${side}_box_collision_geom">
+				<geometry name="${name}_box_collision_geom">
 					<box size="0.088678 0.084137 0.1524" />
 				</geometry>
 			</collision>
 		</link>
-		<link name="ADE_pitch_elbow${side}_fixation">
+		<link name="${name}_fixation">
 			<inertial>
 				<mass value="0.001" />
@@ -37,5 +40,5 @@
 			<visual>
 				<origin xyz="0 0 0" rpy="0 0 0" />
-				<geometry name="ADE_pitch_elbow${side}_fixation_visual_geom">
+				<geometry name="${name}_fixation_visual_geom">
 					<sphere radius="0.001" />
 				</geometry>
@@ -43,10 +46,10 @@
 			<collision>
 				<origin xyz="0 0 0" rpy="0 0 0 " />
-				<geometry name="ADE_pitch_elbow${side}_fixation_collision_geom">
+				<geometry name="${name}_fixation_collision_geom">
 					<sphere radius="0.001" />
 				</geometry>
 			</collision>
 		</link>
-		<link name="ADE_pitch_elbow${side}_link">
+		<link name="${name}_link">
 			<inertial>
 				<mass value="0.045" />
@@ -58,5 +61,5 @@
 			<visual>
 				<origin xyz="0 0 0" rpy="0 0 0" />
-				<geometry name="ADE_pitch_elbow${side}_link_visual_geom">
+				<geometry name="${name}_link_visual_geom">
 					<box size="0.047 0.01 0.01" />
 				</geometry>
@@ -64,17 +67,17 @@
 			<collision>
 				<origin xyz="0 0 0" rpy="0 0 0 " />
-				<geometry name="ADE_pitch_elbow${side}_link_collision_geom">
+				<geometry name="${name}_link_collision_geom">
 					<box size="0.047 0.01 0.01" />
 				</geometry>
 			</collision>
 		</link>
-		<joint name="ADE_pitch_elbow${side}_fixed_1_joint" type="fixed">
+		<joint name="${name}_fixed_1_joint" type="fixed">
 			<parent link="${parent}"/>
-			<child link="ADE_pitch_elbow${side}_box"/>
+			<child link="${name}_box"/>
 			<origin xyz="0 0 -0.1524" rpy="0 0 ${(reflect-1)*M_PI/2}" />
 		</joint>
-		<joint name="ADE_pitch_elbow${side}_revolute_joint" type="revolute">
-			<parent link="ADE_pitch_elbow${side}_box"/>
-			<child link="ADE_pitch_elbow${side}_fixation"/>
+		<joint name="${name}_revolute_joint" type="revolute">
+			<parent link="${name}_box"/>
+			<child link="${name}_fixation"/>
 			<origin xyz="0 -0.03 -0.05" rpy="0 0 -1.5708" />
 			<axis xyz="0 1 0" rpy="0 0 0"/>
@@ -82,15 +85,15 @@
 			<!-- calibration reference_position="0.0"/ -->
 		</joint>
-		<joint name="ADE_pitch_elbow${side}_fixed_2_joint" type="fixed">
-			<parent link="ADE_pitch_elbow${side}_fixation"/>
-			<child link="ADE_pitch_elbow${side}_link"/>
+		<joint name="${name}_fixed_2_joint" type="fixed">
+			<parent link="${name}_fixation"/>
+			<child link="${name}_link"/>
 			<origin xyz="0.0235 0 0" rpy="0 0 0" />
 		</joint>
 		<!-- extensions -->
-		<xacro:jn0_ADE_pitch_elbow_transmission side="${side}" />
-		<gazebo reference="ADE_pitch_elbow${side}_box">
+		<xacro:reddy_arm_elbow_pitch_transmission name="${name}_trans" />
+		<gazebo reference="${name}_box">
 			<material>Gazebo/Green</material>
 		</gazebo>
-		<gazebo reference="ADE_pitch_elbow${side}_link">
+		<gazebo reference="${name}_link">
 			<material>Gazebo/Red</material>
 		</gazebo>

File: urdf/reddy_arm/shoulder_pitch.urdf.xacro (robot description, xacro)
@@ -5,11 +5,11 @@
        xmlns:xacro="http://ros.org/wiki/xacro">
 	<include filename="$(find irl_common_description)/urdf/reddy_arm/arm.transmission.xacro" />
-	<xacro:macro name="ADE_pitch_shoulder" params="side reflect parent">
-		<joint name="ADE_pitch_shoulder${side}_fixed_1_joint" type="fixed">
+	<xacro:macro name="reddy_arm_shoulder_pitch" params="name reflect parent">
+		<joint name="${name}_fixed_1_joint" type="fixed">
 			<parent link="${parent}"/>
-			<child link="ADE_pitch_shoulder${side}_link"/>
+			<child link="${name}_link"/>
 			<origin xyz="0 0 0.03" rpy="0 -1.5708 0" />
 		</joint>
-		<link name="ADE_pitch_shoulder${side}_link">
+		<link name="${name}_link">
 			<inertial>
 				<mass value="0.045" />
@@ -21,5 +21,5 @@
 			<visual>
 				<origin xyz="0 0 0" rpy="0 0 0" />
-				<geometry name="ADE_pitch_shoulder${side}_link_visual_geom">
+				<geometry name="${name}_link_visual_geom">
 					<box size="0.047 0.01 0.01" />
 				</geometry>
@@ -27,12 +27,12 @@
 			<collision>
 				<origin xyz="0 0 0" rpy="0 0 0 " />
-				<geometry name="ADE_pitch_shoulder${side}_link_collision_geom">
+				<geometry name="${name}_link_collision_geom">
 					<box size="0.047 0.01 0.01" />
 				</geometry>
 			</collision>
 		</link>
-		<joint name="ADE_pitch_shoulder${side}_revolute_joint" type="revolute">
-			<parent link="ADE_pitch_shoulder${side}_link"/>
-			<child link="ADE_pitch_shoulder${side}_fixation"/>
+		<joint name="${name}_revolute_joint" type="revolute">
+			<parent link="${name}_link"/>
+			<child link="${name}_fixation"/>
 			<origin xyz="0.0235 0 0" rpy="0 0 0" />
 			<axis xyz="0 1 0" rpy="0 0 0"/>
@@ -40,5 +40,5 @@
 			<!-- calibration reference_position="0.0"/ -->
 		</joint>
-		<link name="ADE_pitch_shoulder${side}_fixation">
+		<link name="${name}_fixation">
 			<inertial>
 				<mass value="0.001" />
@@ -50,5 +50,5 @@
 			<visual>
 				<origin xyz="0 0 0" rpy="0 0 0" />
-				<geometry name="ADE_pitch_shoulder${side}_fixation_visual_geom">
+				<geometry name="${name}_fixation_visual_geom">
 					<sphere radius="0.001" />
 				</geometry>
@@ -56,15 +56,15 @@
 			<collision>
 				<origin xyz="0 0 0" rpy="0 0 0 " />
-				<geometry name="ADE_pitch_shoulder${side}_fixation_collision_geom">
+				<geometry name="${name}_fixation_collision_geom">
 					<sphere radius="0.001" />
 				</geometry>
 			</collision>
 		</link>
-		<joint name="ADE_pitch_shoulder${side}_fixed_2_joint" type="fixed">
-			<parent link="ADE_pitch_shoulder${side}_fixation"/>
-			<child link="ADE_pitch_shoulder${side}_box"/>
+		<joint name="${name}_fixed_2_joint" type="fixed">
+			<parent link="${name}_fixation"/>
+			<child link="${name}_box"/>
 			<origin xyz="0.05 0 -0.03" rpy="0 -0.7854 0" />
 		</joint>
-		<link name="ADE_pitch_shoulder${side}_box">
+		<link name="${name}_box">
 			<inertial>
 				<mass value="1.105" />
@@ -76,11 +76,14 @@
 			<visual>
 				<origin xyz="0 0 0" rpy="0 0 0" />
-				<geometry name="ADE_pitch_shoulder${side}_box_visual_geom">
+				<geometry name="${name}_box_visual_geom">
 					<box size="0.088678 0.084137 0.1524" />
 				</geometry>
+				<material name="${name}_color">
+					<color rgba="0 0 1 1"/>
+				</material>
 			</visual>
 			<collision>
 				<origin xyz="0 0 0" rpy="0 0 0 " />
-				<geometry name="ADE_pitch_shoulder${side}_box_collision_geom">
+				<geometry name="${name}_box_collision_geom">
 					<box size="0.088678 0.084137 0.1524" />
 				</geometry>
@@ -88,9 +91,9 @@
 		</link>
 		<!-- extensions -->
-		<xacro:jn0_ADE_pitch_shoulder_transmission side="${side}" />
-		<gazebo reference="ADE_pitch_shoulder${side}_link">
+		<xacro:reddy_arm_shoulder_pitch_transmission name="${name}_trans" />
+		<gazebo reference="${name}_link">
 			<material>Gazebo/Red</material>
 		</gazebo>
-		<gazebo reference="ADE_pitch_shoulder${side}_box">
+		<gazebo reference="${name}_box">
 			<material>Gazebo/Blue</material>
 		</gazebo>

File: urdf/reddy_arm/shoulder_roll.urdf.xacro (robot description, xacro)
@@ -5,11 +5,11 @@
        xmlns:xacro="http://ros.org/wiki/xacro">
 	<include filename="$(find irl_common_description)/urdf/reddy_arm/arm.transmission.xacro" />
-	<xacro:macro name="ADE_roll" params="side reflect parent">
-		<joint name="ADE_roll${side}_fixed_origine_joint" type="fixed">
+	<xacro:macro name="reddy_arm_shoulder_roll" params="name reflect parent offset_y offset_z">
+		<joint name="${name}_fixed_origine_joint" type="fixed">
 			<parent link="${parent}"/>
-			<child link="ADE_roll${side}_box"/>
-			<origin xyz="0 ${reflect*0.09} 0.1" rpy="0 0 ${(reflect-1)*M_PI/2+M_PI/2}" />
+			<child link="${name}_box"/>
+			<origin xyz="0 ${reflect*offset_y} ${offset_z}" rpy="0 0 ${(reflect-1)*M_PI/2+M_PI/2}" />
 		</joint>
-		<link name="ADE_roll${side}_box">
+		<link name="${name}_box">
 			<inertial>
 				<mass value="1.105" />
@@ -21,5 +21,5 @@
 			<visual>
 				<origin xyz="0 0 0" rpy="0 0 0" />
-				<geometry name="ADE_roll${side}_box_visual_geom">
+				<geometry name="${name}_box_visual_geom">
 					<box size="0.084137 0.088678 0.1524" />
 				</geometry>
@@ -27,15 +27,15 @@
 			<collision>
 				<origin xyz="0 0 0" rpy="0 0 0 " />
-				<geometry name="ADE_roll${side}_box_collision_geom">
+				<geometry name="${name}_box_collision_geom">
 					<box size="0.084137 0.088678 0.1524" />
 				</geometry>
 			</collision>
 		</link>
-		<joint name="ADE_roll${side}_fixed_joint" type="fixed">
-			<parent link="ADE_roll${side}_box"/>
-			<child link="ADE_roll${side}_cylinder"/>
+		<joint name="${name}_fixed_joint" type="fixed">
+			<parent link="${name}_box"/>
+			<child link="${name}_cylinder"/>
 			<origin xyz="0.0500285 0 0.0491765" rpy="0 1.5708 0" />
 		</joint>
-		<link name="ADE_roll${side}_cylinder">
+		<link name="${name}_cylinder">
 			<inertial>
 				<mass value="0.117" />
@@ -47,5 +47,5 @@
 			<visual>
 				<origin xyz="0 0 0" rpy="0 0 0" />
-				<geometry name="ADE_roll${side}_cylinder_visual_geom">
+				<geometry name="${name}_cylinder_visual_geom">
 					<cylinder radius="0.0270235" length="0.011379"/>
 				</geometry>
@@ -53,5 +53,5 @@
 			<collision>
 				<origin xyz="0 0 0" rpy="0 0 0 " />
-				<geometry name="ADE_roll${side}_cylinder_collision_geom">
+				<geometry name="${name}_cylinder_collision_geom">
 					<cylinder radius="0.0270235" length="0.011379"/>
 				</geometry>
@@ -59,7 +59,7 @@
 		</link>
 		<!-- On peut ajouter safety_controller -->
-		<joint name="ADE_roll${side}_revolute_joint" type="revolute">
-			<parent link="ADE_roll${side}_cylinder"/>
-			<child link="ADE_roll${side}_link"/>
+		<joint name="${name}_revolute_joint" type="revolute">
+			<parent link="${name}_cylinder"/>
+			<child link="${name}_link"/>
 			<origin xyz="0 0 0.013" rpy="0 0 0" />
 			<axis xyz="0 0 1" rpy="0 0 0"/>
@@ -67,5 +67,5 @@
 			<!-- calibration reference_position="0.0"/ -->
 		</joint>
-		<link name="ADE_roll${side}_link">
+		<link name="${name}_link">
 			<inertial>
 				<mass value="0.1" />
@@ -77,5 +77,5 @@
 			<visual>
 				<origin xyz="0 0 0" rpy="0 0 0" />
-				<geometry name="ADE_roll${side}_link_visual_geom">
+				<geometry name="${name}_link_visual_geom">
 					<cylinder radius="0.015" length="0.015847"/>
 				</geometry>
@@ -83,5 +83,5 @@
 			<collision>
 				<origin xyz="0 0 0" rpy="0 0 0 " />
-				<geometry name="ADE_roll${side}_link_collision_geom">
+				<geometry name="${name}_link_collision_geom">
 					<cylinder radius="0.015" length="0.015847"/>
 				</geometry>
@@ -89,12 +89,12 @@
 		</link>
 		<!-- extensions -->
-		<xacro:jn0_ADE_roll_shoulder_transmission side="${side}" />
-		<gazebo reference="ADE_roll${side}_box">
+		<xacro:reddy_arm_shoulder_roll_transmission name="${name}_shoulder_trans" />
+		<gazebo reference="${name}_box">
 			<material>Gazebo/Blue</material>
 		</gazebo>
-		<gazebo reference="ADE_roll${side}_cylinder">
+		<gazebo reference="${name}_cylinder">
 			<material>Gazebo/Blue</material>
 		</gazebo>
-		<gazebo reference="ADE_roll${side}_link">
+		<gazebo reference="${name}_link">
 			<material>Gazebo/Red</material>
 		</gazebo>
