Commit message: Refs #176. Renaming parts
git-svn-id: svn+ssh://marvin.3it.usherbrooke.ca/svn/introlab/johnny0/svn/branches/M9/ros-pkgs/irl_robots/irl_common_description@1279 23a761d4-b60a-4777-9503-f06a07968eac

File: urdf/jn0_head/head.urdf.xacro (robot description, xacro)
@@ -4,5 +4,5 @@
        xmlns:interface="http://playerstage.sourceforge.net/gazebo/xmlschema/#interface"
        xmlns:xacro="http://ros.org/wiki/xacro">
-	<include filename="$(find jn0_description)/urdf/head/head.transmission.xacro" />
+	<include filename="$(find irl_common_description)/urdf/jn0_head/head.transmission.xacro" />
 	<property name="pan_size_z" value="0.05" />
 	<property name="head_size_z" value="0.17" />

File: urdf/jn0_torso/torso_box.urdf.xacro (robot description, xacro)
@@ -5,10 +5,44 @@
        xmlns:xacro="http://ros.org/wiki/xacro">
 	<property name="torso_size_z" value="0.37921" />
-	<xacro:macro name="torso" params="name parent">
+	<xacro:macro name="jn0_torso_box" params="name parent">
+		<!--
+			"Stand", the bar supporting the torso
+		-->
+		<joint name="${name}_stand_fixed_joint" type="fixed">
+			<parent link="${parent}"/>
+			<child link="${name}_stand_link"/>
+			<origin xyz="0 0 0.3089" rpy="0 0 0" />
+		</joint>
+		<link name="${name}_stand_link">
+			<inertial>
+				<mass value="0.5" />
+				<origin xyz="0 0 0" />
+				<inertia ixx="0" ixy="0" ixz="0"
+						 iyy="0" iyz="0" izz="0" />
+			</inertial>
+			<visual name="${name}_stand_visual">
+				<origin xyz="0 0 0" rpy="0 0 0" />
+				<geometry name="${name}_stand_visual_geom">
+					<box size="0.038 0.038 0.37038" />
+				</geometry>
+			</visual>
+			<collision name="${name}_stand_collision">
+				<origin xyz="0 0 0" rpy="0 0 0" />
+				<geometry name="${name}_stand_collision_geom">
+					<box size="0.038 0.038 0.37038" />
+				</geometry>
+			</collision>
+		</link>
+		<gazebo reference="${name}_stand_link">
+			<material>Gazebo/Grey</material>
+		</gazebo>
 		<joint name="${name}_fixed_joint" type="fixed">
-			<parent link="${parent}"/>
+			<parent link="${name}_stand_link"/>
 			<child link="${name}_link"/>
 			<origin xyz="0 0 0.374795" rpy="0 0 0" />
 		</joint>
+		<!--
+			Actual torso represented by a box
+		-->
 		<link name="${name}_link">
 			<inertial>

File: urdf/reddy_arm/ADE_pitch_elbow/ADE_pitch_elbow.urdf.xacro (robot description, xacro)
@@ -4,5 +4,5 @@
        xmlns:interface="http://playerstage.sourceforge.net/gazebo/xmlschema/#interface"
        xmlns:xacro="http://ros.org/wiki/xacro">
-	<include filename="$(find jn0_description)/urdf/arm/arm.transmission.xacro" />
+	<include filename="$(find irl_common_description)/urdf/reddy_arm/arm.transmission.xacro" />
 	<xacro:macro name="ADE_pitch_elbow" params="side reflect parent">
 		<link name="ADE_pitch_elbow${side}_box">

File: urdf/reddy_arm/ADE_pitch_shoulder/ADE_pitch_shoulder.urdf.xacro (robot description, xacro)
@@ -4,5 +4,5 @@
        xmlns:interface="http://playerstage.sourceforge.net/gazebo/xmlschema/#interface"
        xmlns:xacro="http://ros.org/wiki/xacro">
-	<include filename="$(find jn0_description)/urdf/arm/arm.transmission.xacro" />
+	<include filename="$(find irl_common_description)/urdf/reddy_arm/arm.transmission.xacro" />
 	<xacro:macro name="ADE_pitch_shoulder" params="side reflect parent">
 		<joint name="ADE_pitch_shoulder${side}_fixed_1_joint" type="fixed">

File: urdf/reddy_arm/ADE_roll/ADE_roll.urdf.xacro (robot description, xacro)
@@ -4,5 +4,5 @@
        xmlns:interface="http://playerstage.sourceforge.net/gazebo/xmlschema/#interface"
        xmlns:xacro="http://ros.org/wiki/xacro">
-	<include filename="$(find jn0_description)/urdf/arm/arm.transmission.xacro" />
+	<include filename="$(find irl_common_description)/urdf/reddy_arm/arm.transmission.xacro" />
 	<xacro:macro name="ADE_roll" params="side reflect parent">
 		<joint name="ADE_roll${side}_fixed_origine_joint" type="fixed">

File: urdf/reddy_arm/arm.urdf.xacro (robot description, xacro)
@@ -5,10 +5,10 @@
        xmlns:xacro="http://playerstage.sourceforge.net/gazebo/xmlschema/#interface"
        name="arm">
-	<include filename="$(find jn0_description)/urdf/arm/ADE_roll/ADE_roll.urdf.xacro" />
-	<include filename="$(find jn0_description)/urdf/arm/ADE_pitch_shoulder/ADE_pitch_shoulder.urdf.xacro" />
-	<include filename="$(find jn0_description)/urdf/arm/ADE_pitch_elbow/ADE_pitch_elbow.urdf.xacro" />
-	<include filename="$(find jn0_description)/urdf/arm/forearm/forearm.urdf.xacro" />
-	<include filename="$(find jn0_description)/urdf/arm/hand/hand.urdf.xacro" />
-	<xacro:macro name="arm" params="side reflect parent">
+	<include filename="$(find irl_common_description)/urdf/reddy_arm/ADE_roll/ADE_roll.urdf.xacro" />
+	<include filename="$(find irl_common_description)/urdf/reddy_arm/ADE_pitch_shoulder/ADE_pitch_shoulder.urdf.xacro" />
+	<include filename="$(find irl_common_description)/urdf/reddy_arm/ADE_pitch_elbow/ADE_pitch_elbow.urdf.xacro" />
+	<include filename="$(find irl_common_description)/urdf/reddy_arm/forearm/forearm.urdf.xacro" />
+	<include filename="$(find irl_common_description)/urdf/reddy_arm/hand/hand.urdf.xacro" />
+	<xacro:macro name="reddy_arm" params="side reflect parent">
 		<xacro:ADE_roll side="${side}" reflect="${reflect}" parent="${parent}"/>
 		<xacro:ADE_pitch_shoulder side="${side}" reflect="${reflect}" parent="ADE_roll${side}_link"/>

Commit message: Refs #176. Splited head / pan tilt.
git-svn-id: svn+ssh://marvin.3it.usherbrooke.ca/svn/introlab/johnny0/svn/branches/M9/ros-pkgs/irl_robots/irl_common_description@1284 23a761d4-b60a-4777-9503-f06a07968eac

File: urdf/jn0_head/head.urdf.xacro (robot description, xacro)
@@ -4,147 +4,65 @@
        xmlns:interface="http://playerstage.sourceforge.net/gazebo/xmlschema/#interface"
        xmlns:xacro="http://ros.org/wiki/xacro">
-	<include filename="$(find irl_common_description)/urdf/jn0_head/head.transmission.xacro" />
-	<xacro:macro name="jn0_head" params="name parent">
+	<include filename="$(find irl_common_description)/urdf/common_geometry.xacro" />
+	<!-- TODO Parametrize right/left eyes -->
+	<xacro:macro name="jn0_head" params="name parent offset_x offset_y offset_z">
 		<joint name="${name}_fixed_joint" type="fixed">
 			<parent link="${parent}"/>
 			<child link="${name}_link"/>
-			<!--origin xyz="0.02 0 0.2228115" rpy="0 0 0" /-->
-			<origin xyz="-0.02 0.03 0.545" rpy="0 0 0" />
+			<!--origin xyz="0.03 0.15 0" rpy="0 ${M_PI} 0" /-->
+			<origin xyz="${offset_x} ${offset_y} ${offset_z}" rpy="0 ${M_PI} 0" />
 		</joint>
 		<link name="${name}_link">
-			<inertial>
-				<mass value="0.2" />
-				<origin xyz="0 0 0" />
-				<inertia ixx="0" ixy="0" ixz="0"
-						 iyy="0" iyz="0" izz="0" />
-			</inertial>
-			<visual name="${name}_visual">
-				<origin xyz="0 0 0" rpy="0 0 -${M_PI/2}" />
-				<!--origin xyz="0 0 0" rpy="0 0 0" /-->
-				<geometry name="${name}_visual_geom">
-					<!--box size="0.04 0.04 0.066413" /-->
-					<mesh filename="package://irl_common_description/meshes/jn0_head/neckTilt.dae"  />
+			<xacro:simple_inertial mass="0.5"/>
+			<visual name="${name}_head_visual">
+				<origin xyz="0 0 0" rpy="0 0 0" />
+				<geometry>
+					<mesh filename="package://irl_common_description/meshes/jn0_head/head.dae"  />
 				</geometry>
 			</visual>
-			<collision name="${name}_collision">
-				<origin xyz="0 0 0" rpy="0 0 -${M_PI/2}" />
-				<geometry name="${name}_collision_geom">
-					<!--box size="0.04 0.04 0.066413" /-->
-					<mesh filename="package://irl_common_description/meshes/jn0_head/neckTilt.STL"  />
+			<collision>
+				<origin xyz="0 0 0" rpy="0 0 0" />
+				<geometry>
+					<mesh filename="package://irl_common_description/meshes/jn0_head/head.STL"  />
 				</geometry>
 			</collision>
 		</link>
-		<joint name="${name}_tilt_joint" type="revolute">
+		<joint name="${name}_right_eye" type="fixed">
 			<parent link="${name}_link"/>
-			<child link="${name}_head_link_tmp"/>
-			<!--origin xyz="-0.02 0 0.0966715" rpy="0 0 0" /-->
-			<origin xyz="0 -0.014 0.045" rpy="0 0 -${M_PI/2}" />
-			<axis xyz="0 0 1" rpy="0 0 0"/>
-			<limit effort="100" velocity="0.1" lower="-0.7" upper="0.7" />
+			<child link="${name}_right_eye_link"/>
+			<origin xyz="0.02 -0.01 0.02" rpy="0 0 0" />
 		</joint>
-		<link name="${name}_head_link_tmp">
-			<inertial>
-				<mass value="0.001" />
-				<origin xyz="0 0 0" />
-				<inertia ixx="0" ixy="0" ixz="0"
-						 iyy="0" iyz="0" izz="0" />
-			</inertial>
-			<visual name="${name}_head_tmp_visual">
+		<joint name="${name}_left_eye" type="fixed">
+			<parent link="${name}_link"/>
+			<child link="${name}_left_eye_link"/>
+			<origin xyz="-0.06 -0.01 0.02" rpy="0 0 0" />
+		</joint>
+		<link name="${name}_right_eye_link">
+			<xacro:simple_inertial mass="0.001"/>
+			<visual>
 				<origin xyz="0 0 0" rpy="0 0 0" />
-				<geometry name="${name}_head_tmp_visual_geom">
-					<mesh filename="package://irl_common_description/meshes/jn0_head/neckpan.dae"  />
-					<!--sphere radius="0.001" /-->
+				<geometry>
+					<mesh filename="package://irl_common_description/meshes/jn0_head/eye.dae"  />
 				</geometry>
 			</visual>
-			<collision name="${name}_head_tmp_collision">
+			<collision name="${name}_right_eye_collision">
 				<origin xyz="0 0 0" rpy="0 0 0" />
-				<geometry name="${name}_head_tmp_collision_geom">
-					<mesh filename="package://irl_common_description/meshes/jn0_head/neckpan.STL"  />
+				<geometry>
+					<mesh filename="package://irl_common_description/meshes/jn0_head/eye.STL"  />
 				</geometry>
 			</collision>
 		</link>
-		<!--joint name="${name}_pan_joint" type="revolute"-->
-		<joint name="${name}_pan_joint" type="fixed">
-			<parent link="${name}_head_link_tmp"/>
-			<child link="${name}_head_link_tmp2"/>
-			<origin xyz="-0.01 0.08 0.04" rpy="${M_PI/2} 0 0" />
-			<!--axis xyz="1 0 0" rpy="0 0 0"/-->
-			<!--limit effort="100" velocity="0.1" lower="-0.7854" upper="0.7854" /-->
-		</joint>
-		<link name="${name}_head_link_tmp2">
-			<inertial>
-				<mass value="0.001" />
-				<origin xyz="0 0 0" />
-				<inertia ixx="0" ixy="0" ixz="0"
-						 iyy="0" iyz="0" izz="0" />
-			</inertial>
-			<visual name="${name}_head_tmp2_visual">
+		<link name="${name}_left_eye_link">
+			<xacro:simple_inertial mass="0.001"/>
+			<visual>
 				<origin xyz="0 0 0" rpy="0 0 0" />
-				<geometry name="${name}_head_tmp2_visual_geom">
-					<mesh filename="package://irl_common_description/meshes/jn0_head/panBraket.dae"  />
-					<!--sphere radius="0.001" /-->
-				</geometry>
-			</visual>
-			<collision name="${name}_head_tmp2_collision">
-				<origin xyz="0 0 0" rpy="0 0 0" />
-				<geometry name="${name}_head_tmp2_collision_geom">
-					<mesh filename="package://irl_common_description/meshes/jn0_head/panBraket.STL"  />
-				</geometry>
-			</collision>
-		</link>
-		<joint name="${name}_fixed_joint_head" type="fixed">
-			<parent link="${name}_head_link_tmp2"/>
-			<child link="${name}_head_link"/>
-			<origin xyz="0.03 0.15 0" rpy="0 ${M_PI} 0" />
-		</joint>
-		<link name="${name}_head_link">
-			<inertial>
-				<mass value="0.5" />
-				<origin xyz="0 0 0" rpy="0 0 0" />
-				<inertia ixx="0" ixy="0" ixz="0"
-						 iyy="0" iyz="0" izz="0" />
-			</inertial>
-			<visual name="${name}_head_visual">
-				<!--origin xyz="0.03 0 0.03" rpy="${M_PI/2} 0 ${M_PI/2}" /-->
-				<origin xyz="0 0 0" rpy="0 0 0" />
-				<geometry name="${name}_head_visual_geom">
-					<mesh filename="package://irl_common_description/meshes/jn0_head/head.dae"  />
-					<!--box size="0.16268 0.17418 0.12693" /-->
-				</geometry>
-			</visual>
-			<collision name="${name}_head_collision">
-				<!--origin xyz="0.03 0 0.03" rpy="${M_PI/2} 0 ${M_PI/2}" /-->
-				<origin xyz="0 0 0" rpy="0 0 0" />
-				<geometry name="${name}_head_collision_geom">
-					<mesh filename="package://irl_common_description/meshes/jn0_head/head.STL"  />
-					<!--box size="0.16268 0.17418 0.12693" /-->
-				</geometry>
-			</collision>
-		</link>
-		<!--joint name="${name}_right_eye" type="revolute"-->
-		<joint name="${name}_right_eye" type="fixed">
-			<parent link="${name}_head_link"/>
-			<child link="${name}_right_eye_link"/>
-			<origin xyz="0.02 -0.01 0.02" rpy="0 0 0" />
-			<!--axis xyz="1 0 0" rpy="0 0 0"/-->
-			<!--limit effort="100" velocity="0.1" lower="-0.7854" upper="0.7854" /-->
-		</joint>
-		<link name="${name}_right_eye_link">
-			<inertial>
-				<mass value="0.001" />
-				<origin xyz="0 0 0" />
-				<inertia ixx="0" ixy="0" ixz="0"
-						 iyy="0" iyz="0" izz="0" />
-			</inertial>
-			<visual name="${name}_right_eye_visual">
-				<origin xyz="0 0 0" rpy="0 0 0" />
-				<geometry name="${name}_right_eye_visual_geom">
+				<geometry>
 					<mesh filename="package://irl_common_description/meshes/jn0_head/eye.dae"  />
 					<!--sphere radius="0.001" /-->
 				</geometry>
 			</visual>
-			<collision name="${name}_right_eye_collision">
+			<collision name="${name}_left_eye_collision">
 				<origin xyz="0 0 0" rpy="0 0 0" />
-				<geometry name="${name}_right_eye_collision_geom">
+				<geometry>
 					<mesh filename="package://irl_common_description/meshes/jn0_head/eye.STL"  />
 				</geometry>
@@ -156,14 +74,14 @@
 			<origin xyz="0.02 0.02 0.02" rpy="0 0 0" />
 		</joint>
+		<joint name="${name}_left_black_eye" type="fixed">
+			<parent link="${name}_left_eye_link"/>
+			<child link="${name}_left_black_eye_link"/>
+			<origin xyz="0.02 0.02 0.02" rpy="0 0 0" />
+		</joint>
 		<link name="${name}_right_black_eye_link">
-			<inertial>
-				<mass value="0.001" />
-				<origin xyz="0 0 0" />
-				<inertia ixx="0" ixy="0" ixz="0"
-						 iyy="0" iyz="0" izz="0" />
-			</inertial>
-			<visual name="${name}_right_black_eye_visual">
+			<xacro:simple_inertial mass="0.001"/>
+			<visual>
 				<origin xyz="0 0 0" rpy="0 0 0" />
-				<geometry name="${name}_right_black_eye_visual_geom">
+				<geometry>
 					<cylinder radius="0.01" length="0.01"/>
 				</geometry>
@@ -171,53 +89,14 @@
 			<collision name="${name}_right_black_eye_collision">
 				<origin xyz="0 0 0" rpy="0 0 0" />
-				<geometry name="${name}_right_black_eye_collision_geom">
+				<geometry>
 					<cylinder radius="0.05" length="0.05"/>
 				</geometry>
 			</collision>
 		</link>
-		<!--joint name="${name}_left_eye" type="revolute"-->
-		<joint name="${name}_left_eye" type="fixed">
-			<parent link="${name}_head_link"/>
-			<child link="${name}_left_eye_link"/>
-			<origin xyz="-0.06 -0.01 0.02" rpy="0 0 0" />
-			<!--axis xyz="1 0 0" rpy="0 0 0"/-->
-			<!--limit effort="100" velocity="0.1" lower="-0.7854" upper="0.7854" /-->
-		</joint>
-		<link name="${name}_left_eye_link">
-			<inertial>
-				<mass value="0.001" />
-				<origin xyz="0 0 0" />
-				<inertia ixx="0" ixy="0" ixz="0"
-						 iyy="0" iyz="0" izz="0" />
-			</inertial>
-			<visual name="${name}_left_eye_visual">
+		<link name="${name}_left_black_eye_link">
+			<xacro:simple_inertial mass="0.001"/>
+			<visual>
 				<origin xyz="0 0 0" rpy="0 0 0" />
-				<geometry name="${name}_right_eye_visual_geom">
-					<mesh filename="package://irl_common_description/meshes/jn0_head/eye.dae"  />
-					<!--sphere radius="0.001" /-->
-				</geometry>
-			</visual>
-			<collision name="${name}_left_eye_collision">
-				<origin xyz="0 0 0" rpy="0 0 0" />
-				<geometry name="${name}_right_eye_collision_geom">
-					<mesh filename="package://irl_common_description/meshes/jn0_head/eye.STL"  />
-				</geometry>
-			</collision>
-		</link>
-		<joint name="${name}_left_black_eye" type="fixed">
-			<parent link="${name}_left_eye_link"/>
-			<child link="${name}_left_black_eye_link"/>
-			<origin xyz="0.02 0.02 0.02" rpy="0 0 0" />
-		</joint>
-		<link name="${name}_left_black_eye_link">
-			<inertial>
-				<mass value="0.001" />
-				<origin xyz="0 0 0" />
-				<inertia ixx="0" ixy="0" ixz="0"
-						 iyy="0" iyz="0" izz="0" />
-			</inertial>
-			<visual name="${name}_left_black_eye_visual">
-				<origin xyz="0 0 0" rpy="0 0 0" />
-				<geometry name="${name}_left_black_eye_visual_geom">
+				<geometry>
 					<cylinder radius="0.01" length="0.01"/>
 				</geometry>
@@ -225,27 +104,24 @@
 			<collision name="${name}_left_black_eye_collision">
 				<origin xyz="0 0 0" rpy="0 0 0" />
-				<geometry name="${name}_left_black_eye_collision_geom">
+				<geometry>
 					<cylinder radius="0.05" length="0.05"/>
 				</geometry>
 			</collision>
 		</link>
-		<!--joint name="${name}_left_eyebrow" type="revolute"-->
 		<joint name="${name}_left_eyebrow" type="fixed">
-			<parent link="${name}_head_link"/>
+			<parent link="${name}_link"/>
 			<child link="${name}_left_eyebrow_link"/>
 			<origin xyz="-0.07 0.035 0.045" rpy="0 0 0" />
-			<!--axis xyz="1 0 0" rpy="0 0 0"/-->
-			<!--limit effort="100" velocity="0.1" lower="-0.7854" upper="0.7854" /-->
+		</joint>
+		<joint name="${name}_right_eyebrow" type="fixed">
+			<parent link="${name}_link"/>
+			<child link="${name}_right_eyebrow_link"/>
+			<origin xyz="0.07 0.035 0.045" rpy="0 0 0" />
 		</joint>
 		<link name="${name}_left_eyebrow_link">
-			<inertial>
-				<mass value="0.001" />
-				<origin xyz="0 0 0" />
-				<inertia ixx="0" ixy="0" ixz="0"
-						 iyy="0" iyz="0" izz="0" />
-			</inertial>
-			<visual name="${name}_left_eyebrow_visual">
+			<xacro:simple_inertial mass="0.001"/>
+			<visual>
 				<origin xyz="0 0 0" rpy="0 0 0" />
-				<geometry name="${name}_left_eyebrow_visual_geom">
+				<geometry>
 					<mesh filename="package://irl_common_description/meshes/jn0_head/eyebrow.dae"  />
 					<!--sphere radius="0.001" /-->
@@ -254,27 +130,14 @@
 			<collision name="${name}_left_eyebrow_collision">
 				<origin xyz="0 0 0" rpy="0 0 0" />
-				<geometry name="${name}_left_eyebrow_collision_geom">
+				<geometry>
 					<mesh filename="package://irl_common_description/meshes/jn0_head/eyebrow.STL"  />
 				</geometry>
 			</collision>
 		</link>
-		<!--joint name="${name}_right_eyebrow" type="revolute"-->
-		<joint name="${name}_right_eyebrow" type="fixed">
-			<parent link="${name}_head_link"/>
-			<child link="${name}_right_eyebrow_link"/>
-			<origin xyz="0.07 0.035 0.045" rpy="0 0 0" />
-			<!--axis xyz="1 0 0" rpy="0 0 0"/-->
-			<!--limit effort="100" velocity="0.1" lower="-0.7854" upper="0.7854" /-->
-		</joint>
 		<link name="${name}_right_eyebrow_link">
-			<inertial>
-				<mass value="0.001" />
-				<origin xyz="0 0 0" />
-				<inertia ixx="0" ixy="0" ixz="0"
-						 iyy="0" iyz="0" izz="0" />
-			</inertial>
-			<visual name="${name}_right_eyebrow_visual">
+			<xacro:simple_inertial mass="0.001"/>
+			<visual>
 				<origin xyz="0 0 0" rpy="0 ${M_PI} 0" />
-				<geometry name="${name}_right_eyebrow_visual_geom">
+				<geometry>
 					<mesh filename="package://irl_common_description/meshes/jn0_head/eyebrow.dae"  />
 					<!--sphere radius="0.001" /-->
@@ -283,12 +146,9 @@
 			<collision name="${name}_right_eyebrow_collision">
 				<origin xyz="0 0 0" rpy="0 ${M_PI} 0" />
-				<geometry name="${name}_right_eyebrow_collision_geom">
+				<geometry>
 					<mesh filename="package://irl_common_description/meshes/jn0_head/eyebrow.STL"  />
 				</geometry>
 			</collision>
 		</link>
-		<!-- extansions -->
-		<xacro:johnny_0_head_tilt_transmission />
-		<xacro:johnny_0_head_pan_transmission />
 		<gazebo reference="${name}_right_black_eye_link">
 			<material>Gazebo/Black</material>
@@ -306,5 +166,5 @@
 			<material>Gazebo/Green</material>
 		</gazebo-->
-		<!--gazebo reference="${name}_head_link">
+		<!--gazebo reference="${name}_link">
 			<material>Gazebo/Red</material>
 		</gazebo-->
