Commit message: Refs #175. Some work done for the UniDrive and interactive arm configuration. Possible timing problem with the driver: can't reliably get a full state or conversion ratios.
git-svn-id: svn+ssh://marvin.3it.usherbrooke.ca/svn/introlab/johnny0/svn/branches/M9/ros-pkgs/irl_robots/irl_common_description@1324 23a761d4-b60a-4777-9503-f06a07968eac

File: urdf/actuators/DEA.urdf.xacro (robot description, xacro)
@@ -6,5 +6,5 @@
 	<include filename="$(find irl_common_description)/urdf/common_geometry.xacro" />
 	<!--
-		Differential Elestic Actuator
+		Differential Elastic Actuator
 		    origin v
 		___________
@@ -56,4 +56,11 @@
 		</joint>
 		<link name="${name}_end_frame" />
+		<!-- Transmission for the actuator -->
+		<transmission type="pr2_mechanism_model/SimpleTransmission"
+			name="$name}_transmission">
+			<actuator name="${name}_motor"/>
+			<joint name="${name}_rotor_joint"/>
+			<mechanicalReduction>1.0</mechanicalReduction>
+		</transmission>
 	</xacro:macro>
 </robot>
