Commit message: Refs #176. Fixed pan tilt joints and materials
git-svn-id: svn+ssh://marvin.3it.usherbrooke.ca/svn/introlab/johnny0/svn/branches/M9/ros-pkgs/irl_robots/irl_common_description@1287 23a761d4-b60a-4777-9503-f06a07968eac

File: urdf/actuators/pan_tilt_ptu46175.urdf.xacro (robot description, xacro)
@@ -6,69 +6,69 @@
 	<include filename="$(find irl_common_description)/urdf/common_geometry.xacro" />
 	<include filename="$(find irl_common_description)/urdf/actuators/pan_tilt_ptu46175.transmission.xacro" />
+	<!-- (private) Generic pan tilt link -->
+	<xacro:macro name="_pan_tilt_ptu46175_link" params="name xyz rpy mesh mass">
+		<link name="${name}">
+			<xacro:simple_inertial mass="${mass}" />
+			<visual>
+				<origin xyz="${xyz}" rpy="${rpy}" />
+				<geometry>
+					<mesh filename="package://irl_common_description/meshes/actuators/pan_tilt_ptu46175/${mesh}.dae"  />
+				</geometry>
+			</visual>
+			<collision>
+				<origin xyz="${xyz}" rpy="${rpy}" />
+				<geometry>
+					<mesh filename="package://irl_common_description/meshes/actuators/pan_tilt_ptu46175/${mesh}.stl"  />
+				</geometry>
+			</collision>
+		</link>
+	</xacro:macro>
 	<xacro:macro name="pan_tilt_ptu46175" params="name parent offset_x offset_y offset_z">
 		<joint name="${name}_fixed_joint" type="fixed">
 			<parent link="${parent}"/>
 			<child link="${name}_tilt_link"/>
-			<origin xyz="${offset_x-0.03} ${offset_y+0.03} ${offset_z}" rpy="0 0 0" />
+			<origin xyz="${offset_x} ${offset_y} ${offset_z}" rpy="0 0 0" />
 		</joint>
-		<link name="${name}_tilt_link">
-			<xacro:simple_inertial mass="0.2" />
-			<visual>
-				<origin xyz="0 0 0" rpy="0 0 -${M_PI/2}" />
-				<geometry>
-					<mesh filename="package://irl_common_description/meshes/actuators/pan_tilt_ptu46175/tilt.dae"  />
-				</geometry>
-			</visual>
-			<collision name="${name}_collision">
-				<origin xyz="0 0 0" rpy="0 0 -${M_PI/2}" />
-				<geometry>
-					<mesh filename="package://irl_common_description/meshes/actuators/pan_tilt_ptu46175/tilt.stl"  />
-				</geometry>
-			</collision>
-		</link>
+		<xacro:_pan_tilt_ptu46175_link
+			name="${name}_tilt_link"
+			xyz="-0.07 0.045 0"
+			rpy="0 0 -${M_PI/2}"
+			mass="0.2"
+			mesh="tilt"
+			/>
 		<joint name="${name}_tilt_joint" type="revolute">
 			<parent link="${name}_tilt_link"/>
 			<child link="${name}_pan_link"/>
-			<origin xyz="0 -0.014 0.045" rpy="0 0 -${M_PI/2}" />
+			<origin xyz="0 0 0.045" rpy="0 0 0" />
 			<axis xyz="0 0 1" rpy="0 0 0"/>
 			<limit effort="100" velocity="0.1" lower="-0.7" upper="0.7" />
 		</joint>
-		<link name="${name}_pan_link">
-			<xacro:simple_inertial mass="0.001" />
-			<visual>
-				<origin xyz="0 0 0" rpy="0 0 0" />
-				<geometry>
-					<mesh filename="package://irl_common_description/meshes/actuators/pan_tilt_ptu46175/pan.dae"  />
-				</geometry>
-			</visual>
-			<collision name="${name}_head_tmp_collision">
-				<origin xyz="0 0 0" rpy="0 0 0" />
-				<geometry>
-					<mesh filename="package://irl_common_description/meshes/actuators/pan_tilt_ptu46175/pan.stl"  />
-				</geometry>
-			</collision>
-		</link>
+		<xacro:_pan_tilt_ptu46175_link
+			name="${name}_pan_link"
+			xyz="-0.07 0.02 0"
+			rpy="0 0 -${M_PI/2}"
+			mass="0.001"
+			mesh="pan"
+			/>
 		<joint name="${name}_pan_joint" type="revolute">
 			<parent link="${name}_pan_link"/>
 			<child link="${name}_bracket_link"/>
-			<origin xyz="-0.01 0.08 0.04" rpy="${M_PI/2} 0 0" />
+			<origin xyz="${0.025/2} ${0.065/2} 0.04" rpy="${M_PI/2} 0 ${-M_PI/2}" />
 			<axis xyz="1 0 0" rpy="0 0 0"/>
 			<limit effort="100" velocity="0.1" lower="-0.7854" upper="0.7854" />
 		</joint>
-		<link name="${name}_bracket_link">
-			<xacro:simple_inertial mass="0.001" />
-			<visual>
-				<origin xyz="0 0 0" rpy="0 0 0" />
-				<geometry>
-					<mesh filename="package://irl_common_description/meshes/actuators/pan_tilt_ptu46175/bracket.dae"  />
-				</geometry>
-			</visual>
-			<collision>
-				<origin xyz="0 0 0" rpy="0 0 0" />
-				<geometry>
-					<mesh filename="package://irl_common_description/meshes/actuators/pan_tilt_ptu46175/bracket.stl"  />
-				</geometry>
-			</collision>
-		</link>
+		<xacro:_pan_tilt_ptu46175_link
+			name="${name}_bracket_link"
+			xyz="0 0 0"
+			rpy="0 0 0"
+			mass="0.001"
+			mesh="bracket"
+			/>
+		<joint name="${name}_top_fixed_joint" type="fixed">
+			<parent link="${name}_bracket_link"/>
+			<child link="${name}_top"/>
+			<origin xyz="0 0 0.05" rpy="0 0 0" />
+		</joint>
+		<link name="${name}_top" />
 		<xacro:pan_tilt_ptu46175_tilt_transmission name="${name}_tilt_trans"/>
 		<xacro:pan_tilt_ptu46175_pan_transmission name="${name}_pan_trans"/>

Commit message: Fixed dimensions to fit all together, splited johnny-0 in reddy and junior
git-svn-id: svn+ssh://marvin.3it.usherbrooke.ca/svn/introlab/johnny0/svn/branches/M9/ros-pkgs/irl_robots/irl_common_description@1296 23a761d4-b60a-4777-9503-f06a07968eac

File: urdf/actuators/pan_tilt_ptu46175.urdf.xacro (robot description, xacro)
@@ -6,22 +6,9 @@
 	<include filename="$(find irl_common_description)/urdf/common_geometry.xacro" />
 	<include filename="$(find irl_common_description)/urdf/actuators/pan_tilt_ptu46175.transmission.xacro" />
-	<!-- (private) Generic pan tilt link -->
-	<xacro:macro name="_pan_tilt_ptu46175_link" params="name xyz rpy mesh mass">
-		<link name="${name}">
-			<xacro:simple_inertial mass="${mass}" />
-			<visual>
-				<origin xyz="${xyz}" rpy="${rpy}" />
-				<geometry>
-					<mesh filename="package://irl_common_description/meshes/actuators/pan_tilt_ptu46175/${mesh}.dae"  />
-				</geometry>
-			</visual>
-			<collision>
-				<origin xyz="${xyz}" rpy="${rpy}" />
-				<geometry>
-					<mesh filename="package://irl_common_description/meshes/actuators/pan_tilt_ptu46175/${mesh}.stl"  />
-				</geometry>
-			</collision>
-		</link>
-	</xacro:macro>
+	<!--
+		Directed Perception pan tilt PTU 46-17-5
+		origin : intersection between the bottom place and the tilt axis
+		${name}_top_frame parallel to origin when all angle are 0
+	-->
 	<xacro:macro name="pan_tilt_ptu46175" params="name parent offset_x offset_y offset_z">
 		<joint name="${name}_fixed_joint" type="fixed">
@@ -54,23 +41,41 @@
 			<parent link="${name}_pan_link"/>
 			<child link="${name}_bracket_link"/>
-			<origin xyz="${0.025/2} ${0.065/2} 0.04" rpy="${M_PI/2} 0 ${-M_PI/2}" />
-			<axis xyz="1 0 0" rpy="0 0 0"/>
+			<origin xyz="0 0 0.04" rpy="0 0 0" />
+			<axis xyz="0 1 0" rpy="0 0 0"/>
 			<limit effort="100" velocity="0.1" lower="-0.7854" upper="0.7854" />
 		</joint>
 		<xacro:_pan_tilt_ptu46175_link
 			name="${name}_bracket_link"
-			xyz="0 0 0"
-			rpy="0 0 0"
+			xyz="${0.025/2} ${0.065/2} -0.01"
+			rpy="${M_PI/2} 0 ${-M_PI/2}"
 			mass="0.001"
 			mesh="bracket"
 			/>
-		<joint name="${name}_top_fixed_joint" type="fixed">
+		<joint name="${name}_top_frame_fixed" type="fixed">
 			<parent link="${name}_bracket_link"/>
-			<child link="${name}_top"/>
+			<child link="${name}_top_frame"/>
 			<origin xyz="0 0 0.05" rpy="0 0 0" />
 		</joint>
-		<link name="${name}_top" />
+		<link name="${name}_top_frame" />
 		<xacro:pan_tilt_ptu46175_tilt_transmission name="${name}_tilt_trans"/>
 		<xacro:pan_tilt_ptu46175_pan_transmission name="${name}_pan_trans"/>
 	</xacro:macro>
+	<!-- (private) Generic pan tilt link -->
+	<xacro:macro name="_pan_tilt_ptu46175_link" params="name xyz rpy mesh mass">
+		<link name="${name}">
+			<xacro:simple_inertial mass="${mass}" />
+			<visual>
+				<origin xyz="${xyz}" rpy="${rpy}" />
+				<geometry>
+					<mesh filename="package://irl_common_description/meshes/actuators/pan_tilt_ptu46175/${mesh}.dae"  />
+				</geometry>
+			</visual>
+			<collision>
+				<origin xyz="${xyz}" rpy="${rpy}" />
+				<geometry>
+					<mesh filename="package://irl_common_description/meshes/actuators/pan_tilt_ptu46175/${mesh}.stl"  />
+				</geometry>
+			</collision>
+		</link>
+	</xacro:macro>
 </robot>

File: urdf/jn0_head/head.urdf.xacro (robot description, xacro)
@@ -5,168 +5,78 @@
        xmlns:xacro="http://ros.org/wiki/xacro">
 	<include filename="$(find irl_common_description)/urdf/common_geometry.xacro" />
-	<!-- TODO Parametrize right/left eyes -->
 	<xacro:macro name="jn0_head" params="name parent offset_x offset_y offset_z">
 		<joint name="${name}_fixed_joint" type="fixed">
 			<parent link="${parent}"/>
 			<child link="${name}_link"/>
-			<!--origin xyz="0.03 0.15 0" rpy="0 ${M_PI} 0" /-->
-			<origin xyz="${offset_x} ${offset_y} ${offset_z}" rpy="0 ${M_PI} 0" />
+			<origin xyz="${offset_x} ${offset_y} ${offset_z}" rpy="0 0 0" />
 		</joint>
-		<link name="${name}_link">
-			<xacro:simple_inertial mass="0.5"/>
-			<visual name="${name}_head_visual">
-				<origin xyz="0 0 0" rpy="0 0 0" />
+		<xacro:_jn0_head_link
+			name="${name}_link"
+			xyz="0.04 0 0.08"
+			rpy="${M_PI/2} 0 ${M_PI/2}"
+			mass="0.5"
+			mesh="head"
+			/>
+		<xacro:_jn0_head_eye name="${name}_l_eye" parent="${name}_link" reflect="1" />
+		<xacro:_jn0_head_eye name="${name}_r_eye" parent="${name}_link" reflect="-1"/>
+	</xacro:macro>
+	<xacro:macro name="_jn0_head_eye" params="name parent reflect">
+		<joint name="${name}" type="fixed">
+			<parent link="${parent}"/>
+			<child link="${name}_link"/>
+			<origin xyz="0.06 ${reflect*0.04} 0.09" rpy="0 0 0" />
+		</joint>
+		<xacro:_jn0_head_link
+			name="${name}_link"
+			xyz="0 -0.02 0.02"
+			rpy="0 ${M_PI/2} 0"
+			mass="0.001"
+			mesh="eye"
+			/>
+		<joint name="${name}_pupil" type="fixed">
+			<parent link="${name}_link"/>
+			<child link="${name}_pupil_link"/>
+			<origin xyz="0 0 0" rpy="0 0 0" />
+		</joint>
+		<xacro:simple_cylinder
+			name="${name}_pupil_link"
+			mass="0.001"
+			xyz="0.02 0 0"
+			rpy="0 ${M_PI/2} 0"
+			radius="0.01"
+			length="0.005"
+			rviz_rgba="0 0 0 1"
+			material="Gazebo/Black"
+			/>
+		<joint name="${name}_eyebrow" type="fixed">
+			<parent link="${name}_link"/>
+			<child link="${name}_eyebrow_link"/>
+			<!-- yaw = 0 when reflect = 1, M_PI when reflect = -1 !  -->
+			<origin xyz="0.028 0 0.035" rpy="0 0 ${M_PI*(reflect-1)/2}" />
+		</joint>
+		<xacro:_jn0_head_link
+			name="${name}_eyebrow_link"
+			xyz="0.0015 0.03 -0.015"
+			rpy="${M_PI/2} 0 ${-M_PI/2}"
+			mass="0.001"
+			mesh="eyebrow"
+			/>
+	</xacro:macro>
+	<xacro:macro name="_jn0_head_link" params="name mass xyz rpy mesh">
+		<link name="${name}">
+			<xacro:simple_inertial mass="${mass}"/>
+			<visual>
+				<origin xyz="${xyz}" rpy="${rpy}" />
 				<geometry>
-					<mesh filename="package://irl_common_description/meshes/jn0_head/head.dae"  />
+					<mesh filename="package://irl_common_description/meshes/jn0_head/${mesh}.dae" />
 				</geometry>
 			</visual>
 			<collision>
-				<origin xyz="0 0 0" rpy="0 0 0" />
+				<origin xyz="${xyz}" rpy="${rpy}" />
 				<geometry>
-					<mesh filename="package://irl_common_description/meshes/jn0_head/head.STL"  />
+					<mesh filename="package://irl_common_description/meshes/jn0_head/${mesh}.STL" />
 				</geometry>
 			</collision>
 		</link>
-		<joint name="${name}_right_eye" type="fixed">
-			<parent link="${name}_link"/>
-			<child link="${name}_right_eye_link"/>
-			<origin xyz="0.02 -0.01 0.02" rpy="0 0 0" />
-		</joint>
-		<joint name="${name}_left_eye" type="fixed">
-			<parent link="${name}_link"/>
-			<child link="${name}_left_eye_link"/>
-			<origin xyz="-0.06 -0.01 0.02" rpy="0 0 0" />
-		</joint>
-		<link name="${name}_right_eye_link">
-			<xacro:simple_inertial mass="0.001"/>
-			<visual>
-				<origin xyz="0 0 0" rpy="0 0 0" />
-				<geometry>
-					<mesh filename="package://irl_common_description/meshes/jn0_head/eye.dae"  />
-				</geometry>
-			</visual>
-			<collision name="${name}_right_eye_collision">
-				<origin xyz="0 0 0" rpy="0 0 0" />
-				<geometry>
-					<mesh filename="package://irl_common_description/meshes/jn0_head/eye.STL"  />
-				</geometry>
-			</collision>
-		</link>
-		<link name="${name}_left_eye_link">
-			<xacro:simple_inertial mass="0.001"/>
-			<visual>
-				<origin xyz="0 0 0" rpy="0 0 0" />
-				<geometry>
-					<mesh filename="package://irl_common_description/meshes/jn0_head/eye.dae"  />
-					<!--sphere radius="0.001" /-->
-				</geometry>
-			</visual>
-			<collision name="${name}_left_eye_collision">
-				<origin xyz="0 0 0" rpy="0 0 0" />
-				<geometry>
-					<mesh filename="package://irl_common_description/meshes/jn0_head/eye.STL"  />
-				</geometry>
-			</collision>
-		</link>
-		<joint name="${name}_right_black_eye" type="fixed">
-			<parent link="${name}_right_eye_link"/>
-			<child link="${name}_right_black_eye_link"/>
-			<origin xyz="0.02 0.02 0.02" rpy="0 0 0" />
-		</joint>
-		<joint name="${name}_left_black_eye" type="fixed">
-			<parent link="${name}_left_eye_link"/>
-			<child link="${name}_left_black_eye_link"/>
-			<origin xyz="0.02 0.02 0.02" rpy="0 0 0" />
-		</joint>
-		<link name="${name}_right_black_eye_link">
-			<xacro:simple_inertial mass="0.001"/>
-			<visual>
-				<origin xyz="0 0 0" rpy="0 0 0" />
-				<geometry>
-					<cylinder radius="0.01" length="0.01"/>
-				</geometry>
-			</visual>
-			<collision name="${name}_right_black_eye_collision">
-				<origin xyz="0 0 0" rpy="0 0 0" />
-				<geometry>
-					<cylinder radius="0.05" length="0.05"/>
-				</geometry>
-			</collision>
-		</link>
-		<link name="${name}_left_black_eye_link">
-			<xacro:simple_inertial mass="0.001"/>
-			<visual>
-				<origin xyz="0 0 0" rpy="0 0 0" />
-				<geometry>
-					<cylinder radius="0.01" length="0.01"/>
-				</geometry>
-			</visual>
-			<collision name="${name}_left_black_eye_collision">
-				<origin xyz="0 0 0" rpy="0 0 0" />
-				<geometry>
-					<cylinder radius="0.05" length="0.05"/>
-				</geometry>
-			</collision>
-		</link>
-		<joint name="${name}_left_eyebrow" type="fixed">
-			<parent link="${name}_link"/>
-			<child link="${name}_left_eyebrow_link"/>
-			<origin xyz="-0.07 0.035 0.045" rpy="0 0 0" />
-		</joint>
-		<joint name="${name}_right_eyebrow" type="fixed">
-			<parent link="${name}_link"/>
-			<child link="${name}_right_eyebrow_link"/>
-			<origin xyz="0.07 0.035 0.045" rpy="0 0 0" />
-		</joint>
-		<link name="${name}_left_eyebrow_link">
-			<xacro:simple_inertial mass="0.001"/>
-			<visual>
-				<origin xyz="0 0 0" rpy="0 0 0" />
-				<geometry>
-					<mesh filename="package://irl_common_description/meshes/jn0_head/eyebrow.dae"  />
-					<!--sphere radius="0.001" /-->
-				</geometry>
-			</visual>
-			<collision name="${name}_left_eyebrow_collision">
-				<origin xyz="0 0 0" rpy="0 0 0" />
-				<geometry>
-					<mesh filename="package://irl_common_description/meshes/jn0_head/eyebrow.STL"  />
-				</geometry>
-			</collision>
-		</link>
-		<link name="${name}_right_eyebrow_link">
-			<xacro:simple_inertial mass="0.001"/>
-			<visual>
-				<origin xyz="0 0 0" rpy="0 ${M_PI} 0" />
-				<geometry>
-					<mesh filename="package://irl_common_description/meshes/jn0_head/eyebrow.dae"  />
-					<!--sphere radius="0.001" /-->
-				</geometry>
-			</visual>
-			<collision name="${name}_right_eyebrow_collision">
-				<origin xyz="0 0 0" rpy="0 ${M_PI} 0" />
-				<geometry>
-					<mesh filename="package://irl_common_description/meshes/jn0_head/eyebrow.STL"  />
-				</geometry>
-			</collision>
-		</link>
-		<gazebo reference="${name}_right_black_eye_link">
-			<material>Gazebo/Black</material>
-		</gazebo>
-		<gazebo reference="${name}_left_black_eye_link">
-			<material>Gazebo/Black</material>
-		</gazebo>
-		<gazebo reference="${name}_right_eyebrow_link">
-			<material>Gazebo/Black</material>
-		</gazebo>
-		<gazebo reference="${name}_left_eyebrow_link">
-			<material>Gazebo/Black</material>
-		</gazebo>
-		<!--gazebo reference="${name}_link">
-			<material>Gazebo/Green</material>
-		</gazebo-->
-		<!--gazebo reference="${name}_link">
-			<material>Gazebo/Red</material>
-		</gazebo-->
 	</xacro:macro>
 </robot>

File: urdf/jn0_torso/box_torso.urdf.xacro (robot description, xacro)
@@ -26,5 +26,5 @@
 			<origin xyz="${xyz}" rpy="0 0 0" />
 		</joint>
-		<!-- Actual torso represented by a box -->
+		<!-- Chest represented by a box -->
 		<xacro:simple_box
 			name = "${name}_link"
@@ -35,5 +35,11 @@
 			rviz_rgba = "1 0 0 1"
 			material  = "Gazebo/Red"
-		/>
+			/>
+		<joint name="${name}_top_frame_fixed" type="fixed">
+			<parent link="${name}_link"/>
+			<child link="${name}_top_frame"/>
+			<origin xyz="0 0 ${height}" rpy="0 0 0" />
+		</joint>
+		<link name="${name}_top_frame" />
 	</xacro:macro>
 </robot>

File: urdf/jn0_torso/reddy_torso.urdf.xacro (robot description, xacro)
@@ -4,30 +4,22 @@
        xmlns:interface="http://playerstage.sourceforge.net/gazebo/xmlschema/#interface"
        xmlns:xacro="http://ros.org/wiki/xacro">
-	<xacro:macro name="reddy_torso" params="name parent">
+	<include filename="$(find irl_common_description)/urdf/common_geometry.xacro" />
+	<xacro:macro name="reddy_torso" params="name parent offset_x offset_y offset_z">
 		<joint name="${name}_fixed_joint" type="fixed">
 			<parent link="${parent}"/>
 			<child link="${name}_link"/>
-			<origin xyz="0 0 0.374795" rpy="0 0 0" />
+			<origin xyz="${offset_x} ${offset_y} ${offset_z}" rpy="0 0 0" />
 		</joint>
 		<link name="${name}_link">
-			<inertial>
-				<mass value="0.5" />
-				<origin xyz="0 0 0" />
-				<inertia ixx="0" ixy="0" ixz="0"
-						 iyy="0" iyz="0" izz="0" />
-			</inertial>
-			<visual name="${name}_visual">
-				<origin xyz="0.055 0 0.545" rpy="${M_PI/2} 0 -${M_PI/2}" />
-				<geometry name="${name}_visual_geom">
-					<!--box size="0.21583 0.270 0.37921" /-->
+			<xacro:simple_inertial mass="0.5" />
+			<visual>
+				<origin xyz="0.0575 0 0.75" rpy="${M_PI/2} 0 -${M_PI/2}" />
+				<geometry>
 					<mesh filename="package://irl_common_description/meshes/jn0_torso/reddy_torso.dae"  />
 				</geometry>
-				<material name="${name}_color">
-					<color rgba="1 0 0 1"/>
-				</material>
 			</visual>
-			<collision name="${name}_collision">
+			<collision>
 				<origin xyz="0 0 0" rpy="0 0 0" />
-				<geometry name="${name}_collision_geom">
+				<geometry>
 					<box size="0.21583 0.270 0.37921" />
 				</geometry>
@@ -37,4 +29,10 @@
 			<material>Gazebo/Red</material>
 		</gazebo>
+		<joint name="${name}_top_frame_fixed" type="fixed">
+			<parent link="${name}_link"/>
+			<child link="${name}_top_frame"/>
+			<origin xyz="0.0575 0 0.75" rpy="0 0 0" />
+		</joint>
+		<link name="${name}_top_frame" />
 	</xacro:macro>
 </robot>

File: urdf/reddy_arm/arm.urdf.xacro (robot description, xacro)
@@ -10,11 +10,12 @@
 	<include filename="$(find irl_common_description)/urdf/reddy_arm/forearm.urdf.xacro" />
 	<include filename="$(find irl_common_description)/urdf/reddy_arm/hand.urdf.xacro" />
-	<xacro:macro name="reddy_arm" params="name reflect parent offset_y offset_z">
+	<xacro:macro name="reddy_arm" params="name reflect parent offset_x offset_y offset_z">
 		<xacro:reddy_arm_shoulder_roll
 			name="${name}_shoulder_roll"
 			reflect="${reflect}"
 			parent="${parent}"
+			offset_x="${offset_x}"
 			offset_y="${offset_y}"
-			offset_z="${offset_z - 0.09}"
+			offset_z="${offset_z}"
 			/>
 		<xacro:reddy_arm_shoulder_pitch

File: urdf/reddy_arm/shoulder_roll.urdf.xacro (robot description, xacro)
@@ -5,9 +5,9 @@
        xmlns:xacro="http://ros.org/wiki/xacro">
 	<include filename="$(find irl_common_description)/urdf/reddy_arm/arm.transmission.xacro" />
-	<xacro:macro name="reddy_arm_shoulder_roll" params="name reflect parent offset_y offset_z">
+	<xacro:macro name="reddy_arm_shoulder_roll" params="name reflect parent offset_x offset_y offset_z">
 		<joint name="${name}_fixed_origine_joint" type="fixed">
 			<parent link="${parent}"/>
 			<child link="${name}_box"/>
-			<origin xyz="0 ${reflect*offset_y} ${offset_z}" rpy="0 0 ${(reflect-1)*M_PI/2+M_PI/2}" />
+			<origin xyz="${offset_x} ${reflect*offset_y} ${offset_z}" rpy="0 0 ${(reflect-1)*M_PI/2+M_PI/2}" />
 		</joint>
 		<link name="${name}_box">

Commit message: Refs #170, #175, #189. Upped the default period between CAN sent messages, added a timeout on the wait period between full states on the UniDriveV2 driver. Also includes a few URDF fixes and launch configuration for the full robot.
git-svn-id: svn+ssh://marvin.3it.usherbrooke.ca/svn/introlab/johnny0/svn/branches/M9/ros-pkgs/irl_robots/irl_common_description@1455 23a761d4-b60a-4777-9503-f06a07968eac

File: urdf/actuators/pan_tilt_ptu46175.urdf.xacro (robot description, xacro)
@@ -58,6 +58,8 @@
 		</joint>
 		<link name="${name}_top_frame" />
+        <!-- Managed by something else
 		<xacro:pan_tilt_ptu46175_tilt_transmission name="${name}_tilt_trans"/>
 		<xacro:pan_tilt_ptu46175_pan_transmission name="${name}_pan_trans"/>
+        -->
 	</xacro:macro>
 	<!-- (private) Generic pan tilt link -->

File: urdf/interactive_arm/arm.urdf.xacro (robot description, xacro)
@@ -86,6 +86,6 @@
 			/>
 		<!-- Forearm -->
-		<joint name="${name}_elbow_joint" type="revolute">
-			<parent link="${name}_shoulder_pitch_dea_end_frame"/>
+		<joint name="${name}_elbow_joint" type="fixed">
+			<parent link="${name}_elbow_dea_end_frame"/>
 			<child link="${name}_forearm_link"/>
 			<origin xyz="${_interactive_arm_elbow_offset} 0 0" rpy="0 0 0" />

Commit message: Refs #176. Reverse pan-tilt descriptions in URDF for ptu.
git-svn-id: svn+ssh://marvin.3it.usherbrooke.ca/svn/introlab/johnny0/svn/branches/M9/ros-pkgs/irl_robots/irl_common_description@1563 23a761d4-b60a-4777-9503-f06a07968eac

File: urdf/actuators/pan_tilt_ptu46175.urdf.xacro (robot description, xacro)
@@ -14,33 +14,33 @@
 		<joint name="${name}_fixed_joint" type="fixed">
 			<parent link="${parent}"/>
-			<child link="${name}_tilt_link"/>
+			<child link="${name}_pan_link"/>
 			<origin xyz="${offset_x} ${offset_y} ${offset_z}" rpy="0 0 0" />
 		</joint>
 		<xacro:_pan_tilt_ptu46175_link
-			name="${name}_tilt_link"
+			name="${name}_pan_link"
 			xyz="-0.07 0.045 0"
 			rpy="0 0 -${M_PI/2}"
 			mass="0.2"
+			mesh="pan"
+			/>
+		<joint name="${name}_pan_joint" type="revolute">
+			<parent link="${name}_pan_link"/>
+			<child link="${name}_tilt_link"/>
+			<origin xyz="0 0 0.045" rpy="0 0 0" />
+			<axis xyz="0 1 0" rpy="0 0 0"/>
+			<limit effort="100" velocity="0.1" lower="-0.7" upper="0.7" />
+		</joint>
+		<xacro:_pan_tilt_ptu46175_link
+			name="${name}_tilt_link"
+			xyz="-0.07 0.02 0"
+			rpy="0 0 -${M_PI/2}"
+			mass="0.001"
 			mesh="tilt"
 			/>
 		<joint name="${name}_tilt_joint" type="revolute">
 			<parent link="${name}_tilt_link"/>
-			<child link="${name}_pan_link"/>
-			<origin xyz="0 0 0.045" rpy="0 0 0" />
-			<axis xyz="0 0 1" rpy="0 0 0"/>
-			<limit effort="100" velocity="0.1" lower="-0.7" upper="0.7" />
-		</joint>
-		<xacro:_pan_tilt_ptu46175_link
-			name="${name}_pan_link"
-			xyz="-0.07 0.02 0"
-			rpy="0 0 -${M_PI/2}"
-			mass="0.001"
-			mesh="pan"
-			/>
-		<joint name="${name}_pan_joint" type="revolute">
-			<parent link="${name}_pan_link"/>
 			<child link="${name}_bracket_link"/>
 			<origin xyz="0 0 0.04" rpy="0 0 0" />
-			<axis xyz="0 1 0" rpy="0 0 0"/>
+			<axis xyz="0 0 1" rpy="0 0 0"/>
 			<limit effort="100" velocity="0.1" lower="-0.7854" upper="0.7854" />
 		</joint>
