Commit message: Refs #176. Corrected rotation axes for PTU.
git-svn-id: svn+ssh://marvin.3it.usherbrooke.ca/svn/introlab/johnny0/svn/branches/M9/ros-pkgs/irl_robots/irl_common_description@1564 23a761d4-b60a-4777-9503-f06a07968eac

File: urdf/actuators/pan_tilt_ptu46175.urdf.xacro (robot description, xacro)
@@ -28,5 +28,5 @@
 			<child link="${name}_tilt_link"/>
 			<origin xyz="0 0 0.045" rpy="0 0 0" />
-			<axis xyz="0 1 0" rpy="0 0 0"/>
+			<axis xyz="0 0 1" rpy="0 0 0"/>
 			<limit effort="100" velocity="0.1" lower="-0.7" upper="0.7" />
 		</joint>
@@ -42,5 +42,5 @@
 			<child link="${name}_bracket_link"/>
 			<origin xyz="0 0 0.04" rpy="0 0 0" />
-			<axis xyz="0 0 1" rpy="0 0 0"/>
+			<axis xyz="0 1 0" rpy="0 0 0"/>
 			<limit effort="100" velocity="0.1" lower="-0.7854" upper="0.7854" />
 		</joint>

Commit message: Closes #202, #203, #204, #211, #214, #218, #220, #221, #224. Merging M10 back to the trunk.
git-svn-id: svn+ssh://marvin.3it.usherbrooke.ca/svn/introlab/johnny0/svn/trunk/ros-pkgs/irl_robots/irl_common_description@1940 23a761d4-b60a-4777-9503-f06a07968eac

File: urdf/actuators/pan_tilt_ptu46175.urdf.xacro (robot description, xacro)
@@ -57,5 +57,24 @@
 			<origin xyz="0 0 0.05" rpy="0 0 0" />
 		</joint>
-		<link name="${name}_top_frame" />
+		<link name="${name}_top_frame">
+            <inertial>
+                <mass value="0.001" />
+                <origin xyz="0 0 0" rpy="0 0 0" />
+                <inertia ixx="0.0001" ixy="0" ixz="0" iyy="0.000001" iyz="0" izz="0.0001" />
+            </inertial>
+            <visual>
+              <origin xyz="0 0 0" rpy="0 0 0" />
+              <geometry>
+                <box size="0.04 0.04 0.08" />
+              </geometry>
+              <material name="Red" />
+            </visual>
+            <collision>
+              <origin xyz="0 0 0" rpy="0 0 0" />
+              <geometry>
+                <box size=".001 .001 .001" />
+              </geometry>
+            </collision>
+        </link>
         <!-- Managed by something else
 		<xacro:pan_tilt_ptu46175_tilt_transmission name="${name}_tilt_trans"/>

File: urdf/az3_base/base.urdf.xacro (robot description, xacro)
@@ -60,11 +60,4 @@
 		  </collision>
 		</link>
-		<!-- front laser -->
-		<xacro:hokuyo_lx04_laser_v0 name="${name}_laser" parent="${name}"
-			ros_topic="/sensors/base_scan" update_rate="20" min_angle="-2.2689"
-			max_angle="2.2689" >
-			<origin xyz="${base_laser_x} ${base_laser_y} ${base_laser_z}"
-			rpy="0 0 0" />
-		</xacro:hokuyo_lx04_laser_v0>
 		<!-- gazebo extensions -->
 		<xacro:az3_base_gazebo name="${name}" />

File: urdf/jn0_torso/box_torso.urdf.xacro (robot description, xacro)
@@ -41,5 +41,24 @@
 			<origin xyz="0 0 ${height}" rpy="0 0 0" />
 		</joint>
-		<link name="${name}_top_frame" />
+		<link name="${name}_top_frame">
+            <inertial>
+                <mass value="0.001" />
+                <origin xyz="0 0 0" rpy="0 0 0" />
+                <inertia ixx="0.0001" ixy="0" ixz="0" iyy="0.000001" iyz="0" izz="0.0001" />
+            </inertial>
+            <visual>
+              <origin xyz="0 0 0" rpy="0 0 0" />
+              <geometry>
+                <box size="0.04 0.04 0.08" />
+              </geometry>
+              <material name="Red" />
+            </visual>
+            <collision>
+              <origin xyz="0 0 0" rpy="0 0 0" />
+              <geometry>
+                <box size=".001 .001 .001" />
+              </geometry>
+            </collision>
+        </link>
 	</xacro:macro>
 </robot>

File: urdf/sensors/hokuyo_lx04_laser.urdf.xacro (robot description, xacro)
@@ -10,7 +10,7 @@
       <insert_block name="origin" />
       <parent link="${parent}_link"/>
-      <child link="${name}_frame"/>
+      <child link="${name}_link"/>
     </joint>
-    <link name="${name}_frame" type="laser">
+    <link name="${name}_link" type="laser">
       <inertial>
         <mass value="0.001" />
@@ -21,5 +21,5 @@
         <origin xyz="0 0 0" rpy="0 0 0" />
         <geometry>
-          <box size="0.001 0.001 0.001" />
+          <box size="0.04 0.04 0.08" />
         </geometry>
         <material name="Red" />

File: urdf/sensors/hokuyo_lx30_laser.urdf.xacro (robot description, xacro)
@@ -10,5 +10,5 @@
       <insert_block name="origin" />
       <parent link="${parent}_link"/>
-      <child link="${name}_frame"/>
+      <child link="${name}_link"/>
     </joint>
     <link name="${name}_frame" type="laser">

File: urdf/sensors/kinect.urdf.xacro (robot description, xacro)
@@ -48,4 +48,9 @@
 	<xacro:macro name="kinect_optical_frame" params="name">
 		<link name="${name}">
+			<inertial>
+				<mass value="0.001" />
+				<origin xyz="0 0 0" rpy="0 0 0" />
+				<inertia ixx="0.0001" ixy="0" ixz="0" iyy="0.000001" iyz="0" izz="0.0001" />
+			</inertial>
 			<visual>
 				<origin xyz="0 0 0.001" rpy="0 0 0" />
@@ -57,4 +62,10 @@
 				</material>
 			</visual>
+			<collision>
+				<origin xyz="0 0 0" rpy="0 0 0" />
+				<geometry>
+					<cylinder length="0.06" radius="0.01" />
+				</geometry>
+			</collision>
 		</link>
 	</xacro:macro>
@@ -67,4 +78,9 @@
 		</joint>
 		<link name="${name}_base_link">
+			<inertial>
+				<mass value="0.001" />
+				<origin xyz="0 0 0" rpy="0 0 0" />
+				<inertia ixx="0.0001" ixy="0" ixz="0" iyy="0.000001" iyz="0" izz="0.0001" />
+			</inertial>
 			<visual>
 				<geometry>
@@ -75,7 +91,18 @@
 				</material>
 			</visual>
+			<collision>
+				<origin xyz="0 0 0" rpy="0 0 0" />
+				<geometry>
+					<box size="0.06 0.08 0.02" />
+				</geometry>
+			</collision>
 		</link>
 		<!-- Missing joint here, defined in kinect.urdf.xacro -->
 		<link name="${name}_camera_link">
+			<inertial>
+				<mass value="0.001" />
+				<origin xyz="0 0 0" rpy="0 0 0" />
+				<inertia ixx="0.0001" ixy="0" ixz="0" iyy="0.000001" iyz="0" izz="0.0001" />
+			</inertial>
 			<visual>
 				<origin xyz="0 0 0.02" rpy="0 0 0" />
@@ -87,4 +114,10 @@
 				</material>
 			</visual>
+			<collision>
+				<origin xyz="0 0 0" rpy="0 0 0" />
+				<geometry>
+					<box size="0.06 0.26 0.035" />
+				</geometry>
+			</collision>
 		</link>
 		<xacro:kinect_optical_frame name="${name}_depth_optical_frame"/>
