Commit message: Refs #307. Geometry fixes for the new PTU controller, there might be a tilt angle sign issue in look_at.
git-svn-id: svn+ssh://marvin.3it.usherbrooke.ca/svn/introlab/johnny0/svn/trunk/ros-pkgs/irl_robots/irl_common_description@2685 23a761d4-b60a-4777-9503-f06a07968eac

File: urdf/actuators/irl_ptu.transmission.xacro (robot description, xacro)
@@ -4,6 +4,5 @@
 	xmlns:interface="http://playerstage.sourceforge.net/gazebo/xmlschema/#interface"
 	xmlns:xacro="http://ros.org/wiki/xacro">
-	<!-- Same transmission for both joints -->
-	<xacro:macro name="irl_ptu_transmission" params="name" >
+	<xacro:macro name="irl_ptu_pan_transmission" params="name" >
 		<transmission type="pr2_mechanism_model/SimpleTransmission" name="${name}_trans">
 			<actuator name="${name}_motor" />
@@ -12,3 +11,10 @@
 		</transmission>
 	</xacro:macro>
+	<xacro:macro name="irl_ptu_tilt_transmission" params="name" >
+		<transmission type="pr2_mechanism_model/SimpleTransmission" name="${name}_trans">
+			<actuator name="${name}_motor" />
+			<joint name="${name}_joint" />
+			<mechanicalReduction>-1.0</mechanicalReduction>
+		</transmission>
+	</xacro:macro>
 </robot>

File: urdf/actuators/irl_ptu.urdf.xacro (robot description, xacro)
@@ -56,6 +56,6 @@
         />
         <!-- Ignored by CAN manager, used in Gazebo -->
-		<xacro:irl_ptu_transmission name="${name}_pan"/>
-		<xacro:irl_ptu_transmission name="${name}_tilt"/>
+		<xacro:irl_ptu_pan_transmission name="${name}_pan"/>
+		<xacro:irl_ptu_tilt_transmission name="${name}_tilt"/>
     </xacro:macro>
 </robot>
