Commit message: Refs #307. Working integration of the new PTU into Johnny-0's launch configuration. Missing: some URDF work to match the actual geometry, slowing down the drives.
git-svn-id: svn+ssh://marvin.3it.usherbrooke.ca/svn/introlab/johnny0/svn/trunk/ros-pkgs/irl_robots/irl_common_description@2771 23a761d4-b60a-4777-9503-f06a07968eac

File: urdf/actuators/irl_ptu.urdf.xacro (robot description, xacro)
@@ -55,4 +55,29 @@
             material="black"
         />
+		<joint name="${name}_top_frame_fixed" type="fixed">
+			<parent link="${name}_bracket_link"/>
+			<child link="${name}_top_frame"/>
+			<origin xyz="0 0 0.016" rpy="0 0 0" />
+		</joint>
+		<link name="${name}_top_frame">
+            <inertial>
+                <mass value="0.001" />
+                <origin xyz="0 0 0" rpy="0 0 0" />
+                <inertia ixx="0.0001" ixy="0" ixz="0" iyy="0.000001" iyz="0" izz="0.0001" />
+            </inertial>
+            <visual>
+              <origin xyz="0 0 0" rpy="0 0 0" />
+              <geometry>
+                <box size="0.04 0.04 0.08" />
+              </geometry>
+              <material name="Red" />
+            </visual>
+            <collision>
+              <origin xyz="0 0 0" rpy="0 0 0" />
+              <geometry>
+                <box size=".001 .001 .001" />
+              </geometry>
+            </collision>
+        </link>
         <!-- Ignored by CAN manager, used in Gazebo -->
 		<xacro:irl_ptu_pan_transmission name="${name}_pan"/>
