Commit message: Refs #176. Added laser to junior
git-svn-id: svn+ssh://marvin.3it.usherbrooke.ca/svn/introlab/johnny0/svn/branches/M9/ros-pkgs/irl_robots/irl_common_description@1424 23a761d4-b60a-4777-9503-f06a07968eac

File: urdf/sensors/hokuyo_lx04_laser.urdf.xacro (robot description, xacro)
@@ -10,7 +10,7 @@
       <insert_block name="origin" />
       <parent link="${parent}_link"/>
-      <child link="${name}_link"/>
+      <child link="${name}_frame"/>
     </joint>
-    <link name="${name}_link" type="laser">
+    <link name="${name}_frame" type="laser">
       <inertial>
         <mass value="0.001" />

File: urdf/sensors/hokuyo_lx30_laser.urdf.xacro (robot description, xacro)
@@ -10,7 +10,7 @@
       <insert_block name="origin" />
       <parent link="${parent}_link"/>
-      <child link="${name}_link"/>
+      <child link="${name}_frame"/>
     </joint>
-    <link name="${name}_link" type="laser">
+    <link name="${name}_frame" type="laser">
       <inertial>
         <mass value="0.001" />
