Commit message: Refs #111. Adding missing frames in Kinect URDF.
git-svn-id: svn+ssh://marvin.3it.usherbrooke.ca/svn/introlab/johnny0/svn/trunk/ros-pkgs/irl_robots/irl_common_description@2572 23a761d4-b60a-4777-9503-f06a07968eac

File: urdf/sensors/kinect.urdf.xacro (robot description, xacro)
@@ -123,13 +123,25 @@
 		<xacro:kinect_optical_frame name="${name}_depth_optical_frame"/>
 		<xacro:kinect_optical_frame name="${name}_rgb_optical_frame"/>
+		<joint name="${name}_depth_joint" type="fixed">
+			<origin xyz="0 0.012 0.02" rpy="0 0 0" />
+			<parent link="${name}_camera_link" />
+			<child link="${name}_depth_frame" />
+		</joint>
+        <link name="${name}_depth_frame"/>
 		<joint name="${name}_depth_optical_joint" type="fixed">
-			<origin xyz="0 0.012 0.02" rpy="${-M_PI/2} 0 ${-M_PI/2}" />
-			<parent link="${name}_camera_link" />
+			<origin xyz="0 0 0" rpy="${-M_PI/2} 0 ${-M_PI/2}" />
+			<parent link="${name}_depth_frame" />
 			<child link="${name}_depth_optical_frame" />
 		</joint>
+		<joint name="${name}_rgb_joint" type="fixed">
+			<origin xyz="0 -0.025 0" rpy="0 0 0" />
+			<parent link="${name}_depth_frame" />
+			<child link="${name}_rgb_frame" />
+		</joint>
+        <link name="${name}_rgb_frame"/>
 		<joint name="${name}_rgb_optical_joint" type="fixed">
-			<origin xyz="0.025 0 0" rpy="0 0 0" />
-			<parent link="${name}_depth_optical_frame" />
-			<child link="${name}_rgb_optical_frame" />
+            <origin xyz="0 0 0" rpy="${-M_PI/2} 0 ${-M_PI/2}"/>
+			<parent link="${name}_rgb_frame"/>
+			<child link="${name}_rgb_optical_frame"/>
 		</joint>
 	</xacro:macro>

Commit message: Refs #342, #111. URDF fixes for the new Kinect configuration, small tweaks to Engage configuration in irl1_demo.
git-svn-id: svn+ssh://marvin.3it.usherbrooke.ca/svn/introlab/johnny0/svn/trunk/ros-pkgs/irl_robots/irl_common_description@3038 23a761d4-b60a-4777-9503-f06a07968eac

File: urdf/sensors/kinect.urdf.xacro (robot description, xacro)
@@ -13,5 +13,5 @@
 			/>
 		<joint name="${name}_camera_joint" type="fixed">
-			<origin xyz="0 0 0.02" rpy="0 ${angle} 0" />
+			<origin xyz="0 0 -0.01" rpy="0 ${angle} 0" />
 			<parent link="${name}_base_link"/>
 			<child link="${name}_camera_link"/>
