Commit message: Refs #171, #175, #189. Full interactive arm controller, removes the SetPoint debug message and adjusts the forearm angle in the URDF.
git-svn-id: svn+ssh://marvin.3it.usherbrooke.ca/svn/introlab/johnny0/svn/branches/M9/ros-pkgs/irl_robots/irl_common_description@1462 23a761d4-b60a-4777-9503-f06a07968eac

File: urdf/interactive_arm/arm.urdf.xacro (robot description, xacro)
@@ -107,5 +107,5 @@
 			<parent link="${name}_forearm_link"/>
 			<child link="${name}_hand_link"/>
-			<origin xyz="${_interactive_arm_forearm_length} 0 0" rpy="0 0 ${-35*M_PI/180}" />
+			<origin xyz="${_interactive_arm_forearm_length} 0 0" rpy="0 0 ${-M_PI/3}" />
 		</joint>
 		<xacro:simple_cylinder
