Commit message: Updating xacro macros.

File: robot_models/jn0_description/robots/jn0_full.urdf.xacro (robot description, xacro)
@@ -6,8 +6,8 @@
        name="johnny_0" >
     <!-- AZIMUT 3 files (includes common files found in irl_common_description) -->
-    <include filename="$(find az3_description)/robots/azimut_3.urdf.xacro" />
+    <xacro:include filename="$(find az3_description)/robots/azimut_3.urdf.xacro" />
     <!-- Johnny-0 (the torso and arms) macro -->
-    <include filename="$(find jn0_description)/robots/johnny_0.urdf.xacro" />
-    <property name="base_height"  value="0.25" />
+    <xacro:include filename="$(find jn0_description)/robots/johnny_0.urdf.xacro" />
+    <xacro:property name="base_height"  value="0.25" />
     <!-- Defines everything from base_link and up. -->
     <xacro:johnny_0 base_height="${base_height}" />

File: robot_models/jn0_description/robots/jn0_standalone.urdf.xacro (robot description, xacro)
@@ -6,6 +6,6 @@
        name="johnny_0" >
     <!-- Johnny-0 (the torso and arms) macro -->
-    <include filename="$(find jn0_description)/robots/johnny_0.urdf.xacro" />
-    <property name="base_height"  value="0.25" />
+    <xacro:include filename="$(find jn0_description)/robots/johnny_0.urdf.xacro" />
+    <xacro:property name="base_height"  value="0.25" />
     <!-- Defines everything from base_link and up. -->
     <xacro:johnny_0 base_height="${base_height}" />

File: robot_models/jn0_description/robots/johnny_0.urdf.xacro (robot description, xacro)
@@ -6,17 +6,17 @@
        name="johnny_0" >
 	<!-- The following included files set up definitions of parts of the robot body -->
-	<include filename="$(find irl_common_description)/urdf/common.xacro" />
+	<xacro:include filename="$(find irl_common_description)/urdf/common.xacro" />
 	<!-- Description files -->
-	<include filename="$(find irl_common_description)/urdf/jn0_torso/box_torso.urdf.xacro" />
-	<include filename="$(find irl_common_description)/urdf/jn0_arm/arm.urdf.xacro" />
-	<include filename="$(find irl_common_description)/urdf/actuators/irl_ptu.urdf.xacro" />
-	<include filename="$(find irl_common_description)/urdf/jn0_head/head.urdf.xacro" />
-	<include filename="$(find irl_common_description)/urdf/sensors/kinect.urdf.xacro" />
-	<include filename="$(find irl_common_description)/urdf/sensors/hokuyo_lx04_laser.urdf.xacro" />
+	<xacro:include filename="$(find irl_common_description)/urdf/jn0_torso/box_torso.urdf.xacro" />
+	<xacro:include filename="$(find irl_common_description)/urdf/jn0_arm/arm.urdf.xacro" />
+	<xacro:include filename="$(find irl_common_description)/urdf/actuators/irl_ptu.urdf.xacro" />
+	<xacro:include filename="$(find irl_common_description)/urdf/jn0_head/head.urdf.xacro" />
+	<xacro:include filename="$(find irl_common_description)/urdf/sensors/kinect.urdf.xacro" />
+	<xacro:include filename="$(find irl_common_description)/urdf/sensors/hokuyo_lx04_laser.urdf.xacro" />
 	<!-- generic simulator_gazebo plugins for starting mechanism control, ros time, ros battery -->
-	<include filename="$(find jn0_description)/gazebo/gazebo.urdf.xacro" />
+	<xacro:include filename="$(find jn0_description)/gazebo/gazebo.urdf.xacro" />
 	<!-- materials for visualization -->
 	<!-- FIXME  Materials from azimut -->
-	<include filename="$(find irl_common_description)/urdf/materials.urdf.xacro" />
+	<xacro:include filename="$(find irl_common_description)/urdf/materials.urdf.xacro" />
 	<!-- TODO screenshots in irl_common_description ? -->
 	<!-- TODO ticket wg like robot package

File: robot_models/jn0_description/robots/junior.urdf.xacro (robot description, xacro)
@@ -6,17 +6,17 @@
        name="johnny_0" >
 	<!-- The following included files set up definitions of parts of the robot body -->
-	<include filename="$(find irl_common_description)/urdf/common.xacro" />
+	<xacro:include filename="$(find irl_common_description)/urdf/common.xacro" />
 	<!-- Description files -->
-	<include filename="$(find irl_common_description)/urdf/jn0_torso/box_torso.urdf.xacro" />
-	<include filename="$(find irl_common_description)/urdf/interactive_arm/arm.urdf.xacro" />
-	<include filename="$(find irl_common_description)/urdf/actuators/pan_tilt_ptu46175.urdf.xacro" />
-	<include filename="$(find irl_common_description)/urdf/jn0_head/head.urdf.xacro" />
-	<include filename="$(find irl_common_description)/urdf/sensors/kinect.urdf.xacro" />
-	<include filename="$(find irl_common_description)/urdf/sensors/hokuyo_lx04_laser.urdf.xacro" />
+	<xacro:include filename="$(find irl_common_description)/urdf/jn0_torso/box_torso.urdf.xacro" />
+	<xacro:include filename="$(find irl_common_description)/urdf/interactive_arm/arm.urdf.xacro" />
+	<xacro:include filename="$(find irl_common_description)/urdf/actuators/pan_tilt_ptu46175.urdf.xacro" />
+	<xacro:include filename="$(find irl_common_description)/urdf/jn0_head/head.urdf.xacro" />
+	<xacro:include filename="$(find irl_common_description)/urdf/sensors/kinect.urdf.xacro" />
+	<xacro:include filename="$(find irl_common_description)/urdf/sensors/hokuyo_lx04_laser.urdf.xacro" />
 	<!-- generic simulator_gazebo plugins for starting mechanism control, ros time, ros battery -->
-	<include filename="$(find jn0_description)/gazebo/gazebo.urdf.xacro" />
+	<xacro:include filename="$(find jn0_description)/gazebo/gazebo.urdf.xacro" />
 	<!-- materials for visualization -->
 	<!-- FIXME  Materials from azimut -->
-	<include filename="$(find irl_common_description)/urdf/materials.urdf.xacro" />
+	<xacro:include filename="$(find irl_common_description)/urdf/materials.urdf.xacro" />
 	<!-- TODO screenshots in irl_common_description ? -->
 	<!-- TODO ticket wg like robot package
@@ -28,5 +28,5 @@
 	<!-- Junior torso with U2S base and separate laser -->
     <link name="base_link"/>
-	<property name="base_height"  value="0.45" />
+	<xacro:property name="base_height"  value="0.45" />
 	<xacro:box_torso
 		name="torso"

File: robot_models/jn0_description/robots/reddy.urdf.xacro (robot description, xacro)
@@ -6,15 +6,15 @@
        name="johnny_0" >
 	<!-- The following included files set up definitions of parts of the robot body -->
-	<include filename="$(find irl_common_description)/urdf/common.xacro" />
+	<xacro:include filename="$(find irl_common_description)/urdf/common.xacro" />
 	<!-- Description files -->
-	<include filename="$(find irl_common_description)/urdf/jn0_torso/reddy_torso.urdf.xacro" />
-	<include filename="$(find irl_common_description)/urdf/reddy_arm/arm.urdf.xacro" />
-	<include filename="$(find irl_common_description)/urdf/actuators/pan_tilt_ptu46175.urdf.xacro" />
-	<include filename="$(find irl_common_description)/urdf/jn0_head/head.urdf.xacro" />
-	<include filename="$(find irl_common_description)/urdf/sensors/kinect.urdf.xacro" />
+	<xacro:include filename="$(find irl_common_description)/urdf/jn0_torso/reddy_torso.urdf.xacro" />
+	<xacro:include filename="$(find irl_common_description)/urdf/reddy_arm/arm.urdf.xacro" />
+	<xacro:include filename="$(find irl_common_description)/urdf/actuators/pan_tilt_ptu46175.urdf.xacro" />
+	<xacro:include filename="$(find irl_common_description)/urdf/jn0_head/head.urdf.xacro" />
+	<xacro:include filename="$(find irl_common_description)/urdf/sensors/kinect.urdf.xacro" />
 	<!-- generic simulator_gazebo plugins for starting mechanism control, ros time, ros battery -->
-	<include filename="$(find jn0_description)/gazebo/gazebo.urdf.xacro" />
+	<xacro:include filename="$(find jn0_description)/gazebo/gazebo.urdf.xacro" />
 	<!-- materials for visualization -->
-	<include filename="$(find irl_common_description)/urdf/materials.urdf.xacro" />
+	<xacro:include filename="$(find irl_common_description)/urdf/materials.urdf.xacro" />
 	<link name="base_link" />
 	<xacro:reddy_torso
