Commit message: Renaming johnny_0 to jn0 to better fit the rest of the system, plus cleanup.

File: robot_models/jn0_description/robots/jn0.urdf.xacro (robot description, xacro)
@@ -1,5 +1,5 @@
 <?xml version="1.0"?>
 <robot xmlns:xacro="http://www.ros.org/wiki/xacro"
-       name="johnny_0" >
+       name="jn0" >
 	<!-- The following included files set up definitions of parts of the robot body -->
 	<xacro:include filename="$(find irl_common_description)/urdf/common.xacro" />
@@ -23,5 +23,5 @@
 		   {xxx}_msgs
 		 -->
-    <xacro:macro name="johnny_0" params="base_height">
+    <xacro:macro name="jn0" params="base_height">
         <link name="base_link">
             <!--
@@ -119,4 +119,9 @@
             <origin xyz="0.1 0.0 ${base_height}" rpy="0 0 0" />
         </xacro:hokuyo_lx04_laser_v0>
+        <!-- For ros_control in Gazebo, disregard otherwise -->
+        <gazebo>
+              <plugin name="gazebo_ros_control" filename="libgazebo_ros_control.so">
+              </plugin>
+        </gazebo>
     </xacro:macro>
 </robot>

File: robot_models/jn0_description/robots/jn0_standalone.urdf.xacro (robot description, xacro)
@@ -1,9 +1,9 @@
 <?xml version="1.0"?>
 <robot xmlns:xacro="http://www.ros.org/wiki/xacro"
-       name="johnny_0" >
+       name="jn0" >
     <!-- Johnny-0 (the torso and arms) macro -->
-    <xacro:include filename="$(find jn0_description)/robots/johnny_0.urdf.xacro" />
+    <xacro:include filename="$(find jn0_description)/robots/jn0_0.urdf.xacro" />
     <xacro:property name="base_height"  value="0.25" />
     <!-- Defines everything from base_link and up. -->
-    <xacro:johnny_0 base_height="${base_height}" />
+    <xacro:jn0 base_height="${base_height}" />
 </robot>
