Commit message: Adding missing fixed joint between world and base_link in the standalone JN0 gazebo config.

File: robot_models/jn0_description/robots/jn0_standalone.urdf.xacro (robot description, xacro)
@@ -7,3 +7,9 @@
     <!-- Defines everything from base_link and up. -->
     <xacro:jn0 base_height="${base_height}" />
+    <!-- Fixes the base_link to the world -->
+    <link name="world" />
+    <joint name="fixed" type="fixed">
+      <parent link="world"/>
+      <child link="base_link"/>
+    </joint>
 </robot>
