Commit message: Fixing laser definitions.

File: robot_models/irl_common_description/urdf/sensors/hokuyo_lx04_laser.gazebo.xacro (robot description, xacro)
@@ -4,19 +4,27 @@
     <gazebo reference="${name}_link">
       <sensor type="ray" name="${name}">
-        <rayCount>640</rayCount>
-        <rangeCount>640</rangeCount>
-        <laserCount>1</laserCount>
-        <origin>0.0 0.0 0.0</origin>
-        <displayRays>false</displayRays>
-        <minAngle>${min_angle*180.0/M_PI}</minAngle>
-        <maxAngle>${max_angle*180.0/M_PI}</maxAngle>
-        <minRange>0.05</minRange>
-        <maxRange>4.0</maxRange>
-        <resRange>0.01</resRange>
-        <updateRate>${update_rate}</updateRate>
+        <update_rate>${update_rate}</update_rate>
+        <visualize>false</visualize>
+        <ray>
+          <scan>
+            <horizontal>
+              <samples>640</samples>
+              <resolution>1</resolution>
+              <min_angle>${min_angle*180.0/M_PI}</min_angle>
+              <max_angle>${max_angle*180.0/M_PI}</max_angle>
+            </horizontal>
+          </scan>
+          <range>
+            <min>0.05</min>
+            <max>4.00</max>
+            <resolution>0.01</resolution>
+          </range>
+          <noise>
+            <type>gaussian</type>
+            <mean>0.00</mean>
+            <stddev>0.01</stddev>
+          </noise>
+        </ray>
         <plugin name="gazebo_ros_${name}_controller" filename="libgazebo_ros_laser.so">
-          <gaussianNoise>0.005</gaussianNoise>
-          <alwaysOn>true</alwaysOn>
-          <updateRate>${update_rate}</updateRate>
           <topicName>${ros_topic}</topicName>
           <frameName>${name}_link</frameName>

File: robot_models/irl_common_description/urdf/sensors/hokuyo_lx30_laser.gazebo.xacro (robot description, xacro)
@@ -3,25 +3,32 @@
   <xacro:macro name="hokuyo_lx30_laser_gazebo_v0" params="name ros_topic update_rate min_angle max_angle">
     <gazebo reference="${name}_link">
-      <sensor:ray name="${name}">
-        <rayCount>640</rayCount>
-        <rangeCount>640</rangeCount>
-        <laserCount>1</laserCount>
-        <origin>0.0 0.0 0.0</origin>
-        <displayRays>false</displayRays>
-        <minAngle>${min_angle*180.0/M_PI}</minAngle>
-        <maxAngle>${max_angle*180.0/M_PI}</maxAngle>
-        <minRange>0.05</minRange>
-        <maxRange>10.0</maxRange>
-        <resRange>0.01</resRange>
-        <updateRate>${update_rate}</updateRate>
-        <controller:gazebo_ros_laser name="gazebo_ros_${name}_controller" plugin="libgazebo_ros_laser.so">
-          <gaussianNoise>0.005</gaussianNoise>
-          <alwaysOn>true</alwaysOn>
-          <updateRate>${update_rate}</updateRate>
+      <sensor type="ray" name="${name}">
+        <update_rate>${update_rate}</update_rate>
+        <visualize>false</visualize>
+        <ray>
+          <scan>
+            <horizontal>
+              <samples>640</samples>
+              <resolution>1</resolution>
+              <min_angle>${min_angle*180.0/M_PI}</min_angle>
+              <max_angle>${max_angle*180.0/M_PI}</max_angle>
+            </horizontal>
+          </scan>
+          <range>
+            <min>0.05</min>
+            <max>30.0</max>
+            <resolution>0.01</resolution>
+          </range>
+          <noise>
+            <type>gaussian</type>
+            <mean>0.00</mean>
+            <stddev>0.01</stddev>
+          </noise>
+        </ray>
+        <plugin name="gazebo_ros_${name}_controller" filename="libgazebo_ros_laser.so">
           <topicName>${ros_topic}</topicName>
           <frameName>${name}_link</frameName>
-          <interface:laser name="gazebo_ros_${name}_iface" />
-        </controller:gazebo_ros_laser>
-      </sensor:ray>
+        </plugin>
+      </sensor>
     </gazebo>
   </xacro:macro>
