Commit message: Work on gazebo_ros_control integration, partial.

File: robot_models/irl_common_description/urdf/actuators/irl_ptu.transmission.xacro (robot description, xacro)
@@ -1,7 +1,4 @@
 <?xml version="1.0"?>
-<robot xmlns:sensor="http://playerstage.sourceforge.net/gazebo/xmlschema/#sensor"
-	xmlns:controller="http://playerstage.sourceforge.net/gazebo/xmlschema/#controller"
-	xmlns:interface="http://playerstage.sourceforge.net/gazebo/xmlschema/#interface"
-	xmlns:xacro="http://www.ros.org/wiki/xacro">
+<robot xmlns:xacro="http://www.ros.org/wiki/xacro">
 	<xacro:macro name="irl_ptu_pan_transmission" params="name" >
 		<transmission type="pr2_mechanism_model/SimpleTransmission" name="${name}_trans">
@@ -12,8 +9,13 @@
 	</xacro:macro>
 	<xacro:macro name="irl_ptu_tilt_transmission" params="name" >
-		<transmission type="pr2_mechanism_model/SimpleTransmission" name="${name}_trans">
-			<actuator name="${name}_motor" />
-			<joint name="${name}_joint" />
-			<mechanicalReduction>-1.0</mechanicalReduction>
+        <transmission type="transmission_interface/SimpleTransmission"
+                      name="${name}_trans">
+			<actuator name="${name}_motor">
+              <hardwareInterface>EffortJointInterface</hardwareInterface>
+			  <mechanicalReduction>-1.0</mechanicalReduction>
+            </actuator>
+			<joint name="${name}_joint">
+              <hardwareInterface>EffortJointInterface</hardwareInterface>
+            </joint>
 		</transmission>
 	</xacro:macro>

File: robot_models/irl_common_description/urdf/actuators/irl_ptu.urdf.xacro (robot description, xacro)
@@ -1,7 +1,4 @@
 <?xml version="1.0"?>
-<robot xmlns:sensor="http://playerstage.sourceforge.net/gazebo/xmlschema/#sensor"
-       xmlns:controller="http://playerstage.sourceforge.net/gazebo/xmlschema/#controller"
-       xmlns:interface="http://playerstage.sourceforge.net/gazebo/xmlschema/#interface"
-       xmlns:xacro="http://www.ros.org/wiki/xacro">
+<robot xmlns:xacro="http://www.ros.org/wiki/xacro">
 	<xacro:include filename="$(find irl_common_description)/urdf/common_geometry.xacro" />
 	<xacro:include filename="$(find irl_common_description)/urdf/actuators/irl_ptu.transmission.xacro" />

File: robot_models/irl_common_description/urdf/actuators/pan_tilt_ptu46175.transmission.xacro (robot description, xacro)
@@ -1,7 +1,4 @@
 <?xml version="1.0"?>
-<robot xmlns:sensor="http://playerstage.sourceforge.net/gazebo/xmlschema/#sensor"
-	xmlns:controller="http://playerstage.sourceforge.net/gazebo/xmlschema/#controller"
-	xmlns:interface="http://playerstage.sourceforge.net/gazebo/xmlschema/#interface"
-	xmlns:xacro="http://www.ros.org/wiki/xacro">
+<robot xmlns:xacro="http://www.ros.org/wiki/xacro">
 	<!-- Pan / Yaw -->
 	<xacro:macro name="pan_tilt_ptu46175_pan_transmission" params="name" >

Commit message: Fixing transmission syntax for PTU and namespaces for controllers/spawner.

File: robot_models/irl_common_description/urdf/actuators/irl_ptu.transmission.xacro (robot description, xacro)
@@ -2,20 +2,25 @@
 <robot xmlns:xacro="http://www.ros.org/wiki/xacro">
 	<xacro:macro name="irl_ptu_pan_transmission" params="name" >
-		<transmission type="pr2_mechanism_model/SimpleTransmission" name="${name}_trans">
-			<actuator name="${name}_motor" />
-			<joint name="${name}_joint" />
-			<mechanicalReduction>1.0</mechanicalReduction>
+        <transmission name="${name}_trans">
+            <type>transmission_interface/SimpleTransmission</type>
+			<joint name="${name}_joint">
+              <hardwareInterface>hardware_interface/EffortJointInterface</hardwareInterface>
+            </joint>
+			<actuator name="${name}_motor">
+              <hardwareInterface>hardware_interface/EffortJointInterface</hardwareInterface>
+			  <mechanicalReduction>-1.0</mechanicalReduction>
+            </actuator>
 		</transmission>
 	</xacro:macro>
 	<xacro:macro name="irl_ptu_tilt_transmission" params="name" >
-        <transmission type="transmission_interface/SimpleTransmission"
-                      name="${name}_trans">
+        <transmission name="${name}_trans">
+            <type>transmission_interface/SimpleTransmission</type>
+			<joint name="${name}_joint">
+              <hardwareInterface>hardware_interface/EffortJointInterface</hardwareInterface>
+            </joint>
 			<actuator name="${name}_motor">
-              <hardwareInterface>EffortJointInterface</hardwareInterface>
+              <hardwareInterface>hardware_interface/EffortJointInterface</hardwareInterface>
 			  <mechanicalReduction>-1.0</mechanicalReduction>
             </actuator>
-			<joint name="${name}_joint">
-              <hardwareInterface>EffortJointInterface</hardwareInterface>
-            </joint>
 		</transmission>
 	</xacro:macro>
