Commit message: Updating xacro macros.

File: robot_models/irl_common_description/urdf/actuators/DEA.urdf.xacro (robot description, xacro)
@@ -4,5 +4,5 @@
        xmlns:interface="http://playerstage.sourceforge.net/gazebo/xmlschema/#interface"
        xmlns:xacro="http://ros.org/wiki/xacro">
-	<include filename="$(find irl_common_description)/urdf/common_geometry.xacro" />
+	<xacro:include filename="$(find irl_common_description)/urdf/common_geometry.xacro" />
 	<!--
 		Differential Elastic Actuator
@@ -15,5 +15,5 @@
 		FIXME Masses, dimensions, limits etc. are very approximative
 	-->
-	<property name="_DEA_stator_length"  value="0.09" />
+	<xacro:property name="_DEA_stator_length"  value="0.09" />
 	<xacro:macro name="DEA" params="name parent xyz rpy shaft_length">
 		<joint name="${name}_stator_joint" type="fixed">

File: robot_models/irl_common_description/urdf/actuators/irl_ptu.urdf.xacro (robot description, xacro)
@@ -4,6 +4,6 @@
        xmlns:interface="http://playerstage.sourceforge.net/gazebo/xmlschema/#interface"
        xmlns:xacro="http://ros.org/wiki/xacro">
-	<include filename="$(find irl_common_description)/urdf/common_geometry.xacro" />
-	<include filename="$(find irl_common_description)/urdf/actuators/irl_ptu.transmission.xacro" />
+	<xacro:include filename="$(find irl_common_description)/urdf/common_geometry.xacro" />
+	<xacro:include filename="$(find irl_common_description)/urdf/actuators/irl_ptu.transmission.xacro" />
     <!-- Similar to the Directed Perception definition, but with Dynamixel
          actuators. -->

File: robot_models/irl_common_description/urdf/actuators/pan_tilt_ptu46175.urdf.xacro (robot description, xacro)
@@ -4,6 +4,6 @@
        xmlns:interface="http://playerstage.sourceforge.net/gazebo/xmlschema/#interface"
        xmlns:xacro="http://ros.org/wiki/xacro">
-	<include filename="$(find irl_common_description)/urdf/common_geometry.xacro" />
-	<include filename="$(find irl_common_description)/urdf/actuators/pan_tilt_ptu46175.transmission.xacro" />
+	<xacro:include filename="$(find irl_common_description)/urdf/common_geometry.xacro" />
+	<xacro:include filename="$(find irl_common_description)/urdf/actuators/pan_tilt_ptu46175.transmission.xacro" />
 	<!--
 		Directed Perception pan tilt PTU 46-17-5

File: robot_models/irl_common_description/urdf/az3_base/base.urdf.xacro (robot description, xacro)
@@ -5,5 +5,5 @@
        xmlns:xacro="http://ros.org/wiki/xacro">
 	<!-- Include files for extensions -->
-	<include filename="$(find irl_common_description)/urdf/az3_base/base.gazebo.xacro" />
+	<xacro:include filename="$(find irl_common_description)/urdf/az3_base/base.gazebo.xacro" />
 	<xacro:macro name="az3_base" params="name">
 		<link name="${name}_link">

File: robot_models/irl_common_description/urdf/az3_wheel_group/wheel.urdf.xacro (robot description, xacro)
@@ -5,6 +5,6 @@
        xmlns:xacro="http://ros.org/wiki/xacro">
 	<!-- Include files for extensions -->
-	<include filename="$(find irl_common_description)/urdf/az3_wheel_group/wheel.gazebo.xacro" />
-	<include filename="$(find irl_common_description)/urdf/az3_wheel_group/wheel.transmission.xacro" />
+	<xacro:include filename="$(find irl_common_description)/urdf/az3_wheel_group/wheel.gazebo.xacro" />
+	<xacro:include filename="$(find irl_common_description)/urdf/az3_wheel_group/wheel.transmission.xacro" />
 	<xacro:macro name="az3_wheel_group" params="side reflectSide face reflectFace parent">
 		<joint name="wheel${side}${face}_revolute_joint" type="revolute">

File: robot_models/irl_common_description/urdf/common.xacro (robot description, xacro)
@@ -1,5 +1,7 @@
 <?xml version="1.0"?>
-<robot>
-  <property name="M_PI" value="3.1415926535897931" />
-  <property name="VELOCITY_LIMIT_SCALE" value="0.6" />
+<robot
+  xmlns:xacro="http://www.ros.org/wiki/xacro"
+>
+  <xacro:property name="M_PI" value="3.1415926535897931" />
+  <xacro:property name="VELOCITY_LIMIT_SCALE" value="0.6" />
 </robot>

File: robot_models/irl_common_description/urdf/interactive_arm/arm.urdf.xacro (robot description, xacro)
@@ -12,11 +12,11 @@
 		FIXME Masses, dimensions, limits etc. are very approximative
 	-->
-	<include filename="$(find irl_common_description)/urdf/common_geometry.xacro" />
-	<include filename="$(find irl_common_description)/urdf/actuators/DEA.urdf.xacro" />
-	<property name="_interactive_arm_shoulder_yaw_offset"  value="0.1" />
-	<property name="_interactive_arm_shoulder_pitch_offset"  value="0.055" />
-	<property name="_interactive_arm_elbow_offset"  value="0.198" />
-	<property name="_interactive_arm_forearm_length"  value="0.145" />
-	<property name="_interactive_arm_hand_length"  value="0.2" />
+	<xacro:include filename="$(find irl_common_description)/urdf/common_geometry.xacro" />
+	<xacro:include filename="$(find irl_common_description)/urdf/actuators/DEA.urdf.xacro" />
+	<xacro:property name="_interactive_arm_shoulder_yaw_offset"  value="0.1" />
+	<xacro:property name="_interactive_arm_shoulder_pitch_offset"  value="0.055" />
+	<xacro:property name="_interactive_arm_elbow_offset"  value="0.198" />
+	<xacro:property name="_interactive_arm_forearm_length"  value="0.145" />
+	<xacro:property name="_interactive_arm_hand_length"  value="0.2" />
 	<xacro:macro name="interactive_arm" params="name parent offset_x offset_y offset_z">
 		<joint name="${name}_side_offset_fixed" type="fixed">

File: robot_models/irl_common_description/urdf/jn0_arm/arm.urdf.xacro (robot description, xacro)
@@ -5,8 +5,8 @@
 	   xmlns:xacro="http://playerstage.sourceforge.net/gazebo/xmlschema/#interface"
 	   name="arm" >
-	<include filename="$(find irl_common_description)/urdf/jn0_arm/shoulder/shoulder.urdf.xacro" />
-	<include filename="$(find irl_common_description)/urdf/jn0_arm/upper_arm/upper_arm.urdf.xacro" />
-	<include filename="$(find irl_common_description)/urdf/jn0_arm/forearm/forearm.urdf.xacro" />
-	<include filename="$(find irl_common_description)/urdf/jn0_arm/gripper/gripper.urdf.xacro" />
+	<xacro:include filename="$(find irl_common_description)/urdf/jn0_arm/shoulder/shoulder.urdf.xacro" />
+	<xacro:include filename="$(find irl_common_description)/urdf/jn0_arm/upper_arm/upper_arm.urdf.xacro" />
+	<xacro:include filename="$(find irl_common_description)/urdf/jn0_arm/forearm/forearm.urdf.xacro" />
+	<xacro:include filename="$(find irl_common_description)/urdf/jn0_arm/gripper/gripper.urdf.xacro" />
 	<xacro:macro name="arm" params="side reflect parent">
 		<xacro:johnny_0_shoulder side="${side}" reflect="${reflect}" parent="${parent}">

File: robot_models/irl_common_description/urdf/jn0_arm/forearm/forearm.urdf.xacro (robot description, xacro)
@@ -7,7 +7,7 @@
 	<!-- Things that are needed only for Gazebo (not the physical robot).  These include
 	sensor and controller plugin specifications -->
-	<include filename="$(find irl_common_description)/urdf/jn0_arm/forearm/forearm.gazebo.xacro" />
-	<include filename="$(find irl_common_description)/urdf/jn0_arm/forearm/forearm.transmission.xacro" />
-	<include filename="$(find irl_common_description)/urdf/common.xacro" />
+	<xacro:include filename="$(find irl_common_description)/urdf/jn0_arm/forearm/forearm.gazebo.xacro" />
+	<xacro:include filename="$(find irl_common_description)/urdf/jn0_arm/forearm/forearm.transmission.xacro" />
+	<xacro:include filename="$(find irl_common_description)/urdf/common.xacro" />
 	<!-- ============================   forearm   ============================ -->
 	<xacro:macro name="johnny_0_forearm" params="side parent reflect *origin">
@@ -17,5 +17,5 @@
 		<!--joint name="${side}_elbow_tilt_joint" type="continuous"-->
 			<axis xyz="0 0 1"/>
-			<insert_block name="origin" />
+			<xacro:insert_block name="origin" />
 			<parent link="${parent}"/>
 			<child link="${side}_forearm_link"/>

File: robot_models/irl_common_description/urdf/jn0_arm/gripper/gripper.urdf.xacro (robot description, xacro)
@@ -7,7 +7,7 @@
 	<!-- Things that are needed only for Gazebo (not the physical robot).  These include
 	sensor and controller plugin specifications -->
-	<include filename="$(find irl_common_description)/urdf/jn0_arm/gripper/gripper.gazebo.xacro" />
-	<include filename="$(find irl_common_description)/urdf/jn0_arm/gripper/gripper.transmission.xacro" />
-	<include filename="$(find irl_common_description)/urdf/common.xacro" />
+	<xacro:include filename="$(find irl_common_description)/urdf/jn0_arm/gripper/gripper.gazebo.xacro" />
+	<xacro:include filename="$(find irl_common_description)/urdf/jn0_arm/gripper/gripper.transmission.xacro" />
+	<xacro:include filename="$(find irl_common_description)/urdf/common.xacro" />
 	<!-- ============================   gripper   ============================ -->
 	<xacro:macro name="johnny_0_gripper" params="side parent reflect">

File: robot_models/irl_common_description/urdf/jn0_arm/shoulder/shoulder.urdf.xacro (robot description, xacro)
@@ -7,12 +7,12 @@
 	<!-- Things that are needed only for Gazebo (not the physical robot).  These include
 	sensor and controller plugin specifications -->
-	<include filename="$(find irl_common_description)/urdf/jn0_arm/shoulder/shoulder.gazebo.xacro" />
-	<include filename="$(find irl_common_description)/urdf/jn0_arm/shoulder/shoulder.transmission.xacro" />
-	<include filename="$(find irl_common_description)/urdf/common.xacro" />
+	<xacro:include filename="$(find irl_common_description)/urdf/jn0_arm/shoulder/shoulder.gazebo.xacro" />
+	<xacro:include filename="$(find irl_common_description)/urdf/jn0_arm/shoulder/shoulder.transmission.xacro" />
+	<xacro:include filename="$(find irl_common_description)/urdf/common.xacro" />
 	<!-- ============================   Shoulder   ============================ -->
 	<xacro:macro name="johnny_0_shoulder" params="side parent reflect *origin">
 		<!-- Shoulder fixed joint -->
 		<joint name="${side}_shoulder_fixed_joint" type="fixed">
-			<insert_block name="origin" />
+			<xacro:insert_block name="origin" />
 			<parent link="${parent}"/>
 			<child link="${side}_shoulder_fixed_link"/>

File: robot_models/irl_common_description/urdf/jn0_arm/upper_arm/upper_arm.urdf.xacro (robot description, xacro)
@@ -7,7 +7,7 @@
 	<!-- Things that are needed only for Gazebo (not the physical robot).  These include
 	sensor and controller plugin specifications -->
-	<include filename="$(find irl_common_description)/urdf/jn0_arm/upper_arm/upper_arm.gazebo.xacro" />
-	<include filename="$(find irl_common_description)/urdf/jn0_arm/upper_arm/upper_arm.transmission.xacro" />
-	<include filename="$(find irl_common_description)/urdf/common.xacro" />
+	<xacro:include filename="$(find irl_common_description)/urdf/jn0_arm/upper_arm/upper_arm.gazebo.xacro" />
+	<xacro:include filename="$(find irl_common_description)/urdf/jn0_arm/upper_arm/upper_arm.transmission.xacro" />
+	<xacro:include filename="$(find irl_common_description)/urdf/common.xacro" />
 	<!-- ============================   Upper arm   ============================ -->
 	<xacro:macro name="johnny_0_upper_arm" params="side parent reflect *origin">
@@ -17,5 +17,5 @@
 		<!--joint name="${side}_shoulder_roll_joint" type="fixed"-->
 			<axis xyz="0 0 1"/>
-			<insert_block name="origin" />
+			<xacro:insert_block name="origin" />
 			<parent link="${parent}"/>
 			<child link="${side}_upper_arm_link"/>

File: robot_models/irl_common_description/urdf/jn0_head/head.urdf.xacro (robot description, xacro)
@@ -4,5 +4,5 @@
        xmlns:interface="http://playerstage.sourceforge.net/gazebo/xmlschema/#interface"
        xmlns:xacro="http://ros.org/wiki/xacro">
-	<include filename="$(find irl_common_description)/urdf/common_geometry.xacro" />
+	<xacro:include filename="$(find irl_common_description)/urdf/common_geometry.xacro" />
 	<xacro:macro name="jn0_head" params="name parent offset_x offset_y offset_z">
 		<joint name="${name}_fixed_joint" type="fixed">

File: robot_models/irl_common_description/urdf/jn0_torso/box_torso.urdf.xacro (robot description, xacro)
@@ -4,5 +4,5 @@
        xmlns:interface="http://playerstage.sourceforge.net/gazebo/xmlschema/#interface"
        xmlns:xacro="http://ros.org/wiki/xacro">
-	<include filename="$(find irl_common_description)/urdf/common_geometry.xacro" />
+	<xacro:include filename="$(find irl_common_description)/urdf/common_geometry.xacro" />
 	<xacro:macro name="box_torso" params="name parent xyz height stand_width chest_width chest_height chest_length">
 		<!-- "Stand", the bar supporting the torso -->

File: robot_models/irl_common_description/urdf/jn0_torso/reddy_torso.urdf.xacro (robot description, xacro)
@@ -4,5 +4,5 @@
        xmlns:interface="http://playerstage.sourceforge.net/gazebo/xmlschema/#interface"
        xmlns:xacro="http://ros.org/wiki/xacro">
-	<include filename="$(find irl_common_description)/urdf/common_geometry.xacro" />
+	<xacro:include filename="$(find irl_common_description)/urdf/common_geometry.xacro" />
 	<xacro:macro name="reddy_torso" params="name parent offset_x offset_y offset_z">
 		<joint name="${name}_fixed_joint" type="fixed">

File: robot_models/irl_common_description/urdf/reddy_arm/arm.urdf.xacro (robot description, xacro)
@@ -5,9 +5,9 @@
        xmlns:xacro="http://playerstage.sourceforge.net/gazebo/xmlschema/#interface"
        name="arm">
-	<include filename="$(find irl_common_description)/urdf/reddy_arm/shoulder_roll.urdf.xacro" />
-	<include filename="$(find irl_common_description)/urdf/reddy_arm/shoulder_pitch.urdf.xacro" />
-	<include filename="$(find irl_common_description)/urdf/reddy_arm/elbow_pitch.urdf.xacro" />
-	<include filename="$(find irl_common_description)/urdf/reddy_arm/forearm.urdf.xacro" />
-	<include filename="$(find irl_common_description)/urdf/reddy_arm/hand.urdf.xacro" />
+	<xacro:include filename="$(find irl_common_description)/urdf/reddy_arm/shoulder_roll.urdf.xacro" />
+	<xacro:include filename="$(find irl_common_description)/urdf/reddy_arm/shoulder_pitch.urdf.xacro" />
+	<xacro:include filename="$(find irl_common_description)/urdf/reddy_arm/elbow_pitch.urdf.xacro" />
+	<xacro:include filename="$(find irl_common_description)/urdf/reddy_arm/forearm.urdf.xacro" />
+	<xacro:include filename="$(find irl_common_description)/urdf/reddy_arm/hand.urdf.xacro" />
 	<xacro:macro name="reddy_arm" params="name reflect parent offset_x offset_y offset_z">
 		<xacro:reddy_arm_shoulder_roll

File: robot_models/irl_common_description/urdf/reddy_arm/elbow_pitch.urdf.xacro (robot description, xacro)
@@ -4,5 +4,5 @@
        xmlns:interface="http://playerstage.sourceforge.net/gazebo/xmlschema/#interface"
        xmlns:xacro="http://ros.org/wiki/xacro">
-	<include filename="$(find irl_common_description)/urdf/reddy_arm/arm.transmission.xacro" />
+	<xacro:include filename="$(find irl_common_description)/urdf/reddy_arm/arm.transmission.xacro" />
 	<xacro:macro name="reddy_arm_elbow_pitch" params="name reflect parent">
 		<link name="${name}_box">

File: robot_models/irl_common_description/urdf/reddy_arm/forearm.urdf.xacro (robot description, xacro)
@@ -4,5 +4,5 @@
        xmlns:interface="http://playerstage.sourceforge.net/gazebo/xmlschema/#interface"
        xmlns:xacro="http://ros.org/wiki/xacro">
-	<include filename="$(find irl_common_description)/urdf/common_geometry.xacro" />
+	<xacro:include filename="$(find irl_common_description)/urdf/common_geometry.xacro" />
 	<xacro:macro name="forearm" params="name reflect parent">
 		<xacro:simple_cylinder

File: robot_models/irl_common_description/urdf/reddy_arm/hand.urdf.xacro (robot description, xacro)
@@ -4,5 +4,5 @@
        xmlns:interface="http://playerstage.sourceforge.net/gazebo/xmlschema/#interface"
        xmlns:xacro="http://ros.org/wiki/xacro">
-	<include filename="$(find irl_common_description)/urdf/common_geometry.xacro" />
+	<xacro:include filename="$(find irl_common_description)/urdf/common_geometry.xacro" />
 	<xacro:macro name="hand" params="name reflect parent">
 		<xacro:simple_sphere

File: robot_models/irl_common_description/urdf/reddy_arm/shoulder_pitch.urdf.xacro (robot description, xacro)
@@ -4,5 +4,5 @@
        xmlns:interface="http://playerstage.sourceforge.net/gazebo/xmlschema/#interface"
        xmlns:xacro="http://ros.org/wiki/xacro">
-	<include filename="$(find irl_common_description)/urdf/reddy_arm/arm.transmission.xacro" />
+	<xacro:include filename="$(find irl_common_description)/urdf/reddy_arm/arm.transmission.xacro" />
 	<xacro:macro name="reddy_arm_shoulder_pitch" params="name reflect parent">
 		<joint name="${name}_fixed_1_joint" type="fixed">
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
Commit message: Updates to transmission definitions for the arms and grippers.

File: robot_models/irl_common_description/urdf/actuators/DEA.urdf.xacro (robot description, xacro)
@@ -54,9 +54,13 @@
 		<link name="${name}_end_frame" />
 		<!-- Transmission for the actuator -->
-		<transmission type="pr2_mechanism_model/SimpleTransmission"
-			name="$name}_transmission">
-			<actuator name="${name}_motor"/>
-			<joint name="${name}_rotor_joint"/>
-			<mechanicalReduction>1.0</mechanicalReduction>
+        <transmission name="${name}_transmission">
+            <type>transmission_interface/SimpleTransmission</type>
+			<joint name="${name}_rotor_joint">
+              <hardwareInterface>hardware_interface/EffortJointInterface</hardwareInterface>
+            </joint>
+			<actuator name="${name}_motor">
+              <hardwareInterface>hardware_interface/EffortJointInterface</hardwareInterface>
+			  <mechanicalReduction>1.0</mechanicalReduction>
+            </actuator>
 		</transmission>
 	</xacro:macro>

File: robot_models/irl_common_description/urdf/jn0_arm/forearm/forearm.transmission.xacro (robot description, xacro)
@@ -3,7 +3,12 @@
 	<xacro:macro name="johnny_0_forearm_transmission" params="side">
 		<!-- Elbow tilt -->
-		<transmission type="pr2_mechanism_model/SimpleTransmission" name="${side}_elbow_tilt_trans">
-			<actuator name="${side}_elbow_tilt_motor" />
-			<joint name="${side}_elbow_tilt_joint" />
+		<transmission name="${side}_elbow_tilt_trans">
+            <type>hardware_interface/SimpleTransmission</type>
+            <actuator name="${side}_elbow_tilt_motor">
+              <hardwareInterface>hardware_interface/EffortJointInterface</hardwareInterface>
+            </actuator>
+			<joint name="${side}_elbow_tilt_joint">
+              <hardwareInterface>hardware_interface/EffortJointInterface</hardwareInterface>
+            </joint>
 			<mechanicalReduction>1.0</mechanicalReduction>
 		</transmission>

File: robot_models/irl_common_description/urdf/jn0_arm/gripper/gripper.transmission.xacro (robot description, xacro)
@@ -3,13 +3,23 @@
 	<xacro:macro name="johnny_0_gripper_transmission" params="side">
 		<!-- Gripper up transmission -->
-		<transmission type="pr2_mechanism_model/SimpleTransmission" name="${side}_gripper_up_trans">
-			<actuator name="${side}_gripper_up_motor" />
-			<joint name="${side}_gripper_up_joint" />
+		<transmission name="${side}_gripper_up_trans">
+            <type>hardware_interface/SimpleTransmission</type>
+			<actuator name="${side}_gripper_up_motor">
+              <hardwareInterface>hardware_interface/EffortJointInterface</hardwareInterface>
+            </actuator>
+			<joint name="${side}_gripper_up_joint">
+              <hardwareInterface>hardware_interface/EffortJointInterface</hardwareInterface>
+            </joint>
 			<mechanicalReduction>1.0</mechanicalReduction>
 		</transmission>
 		<!-- Gripper down transmission -->
-		<transmission type="pr2_mechanism_model/SimpleTransmission" name="${side}_gripper_down_trans">
-			<actuator name="${side}_gripper_down_motor" />
-			<joint name="${side}_gripper_down_joint" />
+		<transmission name="${side}_gripper_down_trans">
+            <type>hardware_interface/SimpleTransmission</type>
+			<actuator name="${side}_gripper_down_motor">
+              <hardwareInterface>hardware_interface/EffortJointInterface</hardwareInterface>
+            </actuator>
+			<joint name="${side}_gripper_down_joint">
+              <hardwareInterface>hardware_interface/EffortJointInterface</hardwareInterface>
+            </joint>
 			<mechanicalReduction>1.0</mechanicalReduction>
 		</transmission>

File: robot_models/irl_common_description/urdf/jn0_arm/shoulder/shoulder.transmission.xacro (robot description, xacro)
@@ -3,13 +3,23 @@
 	<xacro:macro name="johnny_0_shoulder_transmission" params="reflect side">
 		<!-- Shoulder pan -->
-		<transmission type="pr2_mechanism_model/SimpleTransmission" name="${side}_shoulder_pan_trans">
-			<actuator name="${side}_shoulder_pan_motor" />
-			<joint name="${side}_shoulder_pan_joint" />
+		<transmission name="${side}_shoulder_pan_trans">
+            <type>hardware_interface/SimpleTransmission</type>
+			<actuator name="${side}_shoulder_pan_motor">
+              <hardwareInterface>hardware_interface/EffortJointInterface</hardwareInterface>
+            </actuator>
+			<joint name="${side}_shoulder_pan_joint">
+              <hardwareInterface>hardware_interface/EffortJointInterface</hardwareInterface>
+            </joint>
 			<mechanicalReduction>1.0</mechanicalReduction>
 		</transmission>
 		<!-- Shoulder tilt -->
-		<transmission type="pr2_mechanism_model/SimpleTransmission" name="${side}_shoulder_tilt_trans">
-			<actuator name="${side}_shoulder_tilt_motor" />
-			<joint name="${side}_shoulder_tilt_joint" />
+		<transmission name="${side}_shoulder_tilt_trans">
+            <type>hardware_interface/SimpleTransmission</type>
+			<actuator name="${side}_shoulder_tilt_motor">
+              <hardwareInterface>hardware_interface/EffortJointInterface</hardwareInterface>
+            </actuator>
+			<joint name="${side}_shoulder_tilt_joint">
+              <hardwareInterface>hardware_interface/EffortJointInterface</hardwareInterface>
+            </joint>
 			<mechanicalReduction>${reflect}</mechanicalReduction>
 		</transmission>

File: robot_models/irl_common_description/urdf/jn0_arm/upper_arm/upper_arm.transmission.xacro (robot description, xacro)
@@ -3,7 +3,12 @@
 	<xacro:macro name="johnny_0_upper_arm_transmission" params="side reflect">
 		<!-- Shoulder roll -->
-		<transmission type="pr2_mechanism_model/SimpleTransmission" name="${side}_shoulder_roll_trans">
-			<actuator name="${side}_shoulder_roll_motor" />
-			<joint name="${side}_shoulder_roll_joint" />
+		<transmission name="${side}_shoulder_roll_trans">
+            <type>hardware_interface/SimpleTransmission</type>
+			<actuator name="${side}_shoulder_roll_motor">
+              <hardwareInterface>hardware_interface/EffortJointInterface</hardwareInterface>
+            </actuator>
+			<joint name="${side}_shoulder_roll_joint">
+              <hardwareInterface>hardware_interface/EffortJointInterface</hardwareInterface>
+            </joint>
 			<mechanicalReduction>${reflect * -1.0}</mechanicalReduction>
 		</transmission>
