Commit message: Higher velocity limits in PTU.

File: robot_models/irl_common_description/urdf/actuators/irl_ptu.urdf.xacro (robot description, xacro)
@@ -25,5 +25,5 @@
 			<origin xyz="0 0 0.041" rpy="0 0 0" />
 			<axis xyz="0 0 1" rpy="0 0 0"/>
-            <limit effort="100" velocity="0.1" lower="${-M_PI/2}" upper="${M_PI/2}" />
+            <limit effort="100" velocity="2.0" lower="${-M_PI/2}" upper="${M_PI/2}" />
 		</joint>
         <xacro:simple_box
@@ -41,5 +41,5 @@
             <origin xyz="0.013 0 0.025" rpy="0 0 0" />
 			<axis xyz="0 1 0" rpy="0 0 0"/>
-			<limit effort="100" velocity="0.1" lower="-0.170" upper="0.7854" />
+			<limit effort="100" velocity="2.0" lower="-0.170" upper="0.7854" />
 		</joint>
         <xacro:simple_box
