Commit message: Copied PID values from old setup, fixed inertia matrices for the grippers, which fixed the stability issues.

File: robot_models/irl_common_description/urdf/az3_base/base.gazebo.xacro (robot description, xacro)
@@ -3,5 +3,5 @@
   <xacro:macro name="az3_base_gazebo" params="name">
     <gazebo reference="${name}_link">
-      <selfCollide>true</selfCollide>
+      <selfCollide>false</selfCollide>
 	  <!-- No bumper -->
       <!--sensor:contact name="${name}_contact_sensor">

File: robot_models/irl_common_description/urdf/jn0_arm/forearm/forearm.urdf.xacro (robot description, xacro)
@@ -18,7 +18,6 @@
 			<child link="${side}_forearm_link"/>
 			<!-- This parameters have to be modified -->
-			<limit effort="30" velocity="2.0" lower="${-43*M_PI/180}" upper="${80*M_PI/180}" />
-			<!--limit effort="30" velocity="2.0" lower="${-M_PI/2}" upper="${M_PI/2}" /-->
-			<!--safety_controller k_position="20" k_velocity="10" soft_lower_limit="${-43*M_PI/180}" soft_upper_limit="${80*M_PI/180}"  /-->
+			<limit effort="10" velocity="1.0" lower="${-43*M_PI/180}" upper="${70*M_PI/180}" />
+            <dynamics damping="0.1"/>
 		</joint>
 		<link name="${side}_forearm_link">

File: robot_models/irl_common_description/urdf/jn0_arm/gripper/gripper.urdf.xacro (robot description, xacro)
@@ -26,10 +26,7 @@
 				<mass value="0.21180172" />
 				<origin xyz="0.05877696 0.00139214 -0.00602003" rpy="0 0 0"/>
-				<inertia  ixx="0" ixy="0"  ixz="0"
-					iyy="0" iyz="0"
-					izz="0" />
-				<!--inertia  	ixx="0.00003889" 	ixy="0.00000916"  	ixz="-0.00003123"
-										iyy="0.00026591" 	iyz="0.00000146"
-														izz="0.00026384" /-->
+				<inertia  	ixx="0.00003889"    ixy="0.00000916"    ixz="-0.00003123"
+							                    iyy="0.00026591"    iyz="0.00000146"
+												                    izz="0.00026384" />
 			</inertial>
 			<visual>
@@ -63,10 +60,7 @@
 				<mass value="0.19772070" />
 				<origin xyz="0.06212355 0.00111307 0.00727599" rpy="0 0 0"/>
-				<inertia  ixx="0" ixy="0"  ixz="0"
-					iyy="0" iyz="0"
-					izz="0" />
-				<!--inertia  	ixx="0.00003272" 	ixy="0.00001291"  	ixz="0.00001859"
-										iyy="0.00022630" 	iyz="-0.00000033"
-														izz="0.00022754" /-->
+				<inertia  	ixx="0.00003889"    ixy="0.00000916"    ixz="-0.00003123"
+							                    iyy="0.00026591"    iyz="0.00000146"
+												                    izz="0.00026384" />
 			</inertial>
 			<visual>

File: robot_models/irl_common_description/urdf/jn0_arm/shoulder/shoulder.gazebo.xacro (robot description, xacro)
@@ -3,6 +3,5 @@
 	<xacro:macro name="johnny_0_shoulder_gazebo" params="name">
 		<gazebo reference="${name}_link">
-			<selfCollide>true</selfCollide>
-			<material value="PR2/Green" />
+			<selfCollide>false</selfCollide>
 		</gazebo>
 	</xacro:macro>

File: robot_models/irl_common_description/urdf/jn0_arm/shoulder/shoulder.urdf.xacro (robot description, xacro)
@@ -46,5 +46,6 @@
 			<child link="${side}_shoulder_pan_link"/>
 			<!-- This parameters have to be modified -->
-			<limit effort="30" velocity="2.0" lower="${-M_PI/2}" upper="${M_PI/2}" />
+			<limit effort="10" velocity="2.0" lower="${-M_PI/2}" upper="${M_PI/2}" />
+            <dynamics damping="0.1"/>
 			<!--safety_controller k_position="100" k_velocity="10" soft_lower_limit="${-M_PI/2+0.15}" soft_upper_limit="${M_PI/2-0.15}"  /-->
 		</joint>
@@ -73,6 +74,4 @@
 		<!-- Shoulder revolute joint - axis 2 : tilt -->
 		<joint name="${side}_shoulder_tilt_joint" type="revolute">
-		<!--joint name="${side}_shoulder_tilt_joint" type="continuous"-->
-		<!--joint name="${side}_shoulder_tilt_joint" type="fixed"-->
 			<axis xyz="0 0 1" />
 			<origin xyz="0 ${reflect*0.09471141} 0" rpy="${-M_PI/2} 0 0"/>
@@ -80,7 +79,6 @@
 			<child link="${side}_shoulder_tilt_link"/>
 			<!-- This parameters have to be modified -->
-			<!--limit effort="30" velocity="2.0" lower="${-M_PI/2}" upper="${M_PI}" /-->
-			<limit effort="30" velocity="2.0" lower="${-M_PI}" upper="${M_PI/2}" />
-			<!--safety_controller k_position="100" k_velocity="10" soft_lower_limit="${-M_PI/2}" soft_upper_limit="${M_PI}"/-->
+			<limit effort="20" velocity="1.0" lower="${-M_PI}" upper="${M_PI/2}" />
+            <dynamics damping="0.1"/>
 		</joint>
 		<!-- Shoulder link -->

File: robot_models/irl_common_description/urdf/jn0_arm/upper_arm/upper_arm.urdf.xacro (robot description, xacro)
@@ -11,6 +11,4 @@
 		<!-- Shoulder revolute joint - axis 3 : roll -->
 		<joint name="${side}_shoulder_roll_joint" type="revolute">
-		<!--joint name="${side}_shoulder_roll_joint" type="continuous"-->
-		<!--joint name="${side}_shoulder_roll_joint" type="fixed"-->
 			<axis xyz="0 0 1"/>
 			<xacro:insert_block name="origin" />
@@ -18,7 +16,6 @@
 			<child link="${side}_upper_arm_link"/>
 			<!-- This parameters have to be modified -->
-			<limit effort="30" velocity="2.0" lower="${-M_PI/2}" upper="${M_PI/2}"/>
-			<!-- limit effort="30" velocity="2.0" lower="${-3*M_PI/4}" upper="${3*M_PI/4}" /-->
-			<!--safety_controller k_position="100" k_velocity="2" soft_lower_limit="${-M_PI/2}" soft_upper_limit="${M_PI/2}"  /-->
+			<limit effort="10" velocity="2.0" lower="${-M_PI/2}" upper="${M_PI/2}"/>
+            <dynamics damping="0.1"/>
 		</joint>
 		<!-- Upper arm link -->
